Commit message: create collision objects, rotation and scale params for create_cube(), reset cursor rotation

File: puzzles/simple_two_cubes/urdf/simple_two_cubes.urdf (robot description, URDF)
Before this commit: robot simple_two_cubes, 2 links, 1 joints
Links:
- link base_link: geometry collision box size=2.0 2.0 2.0; visual box size=2.0 2.0 2.0
- link link1: geometry collision box size=2.0 4.0 2.0; visual box size=2.0 4.0 2.0
Joints:
- joint link1: origin xyz=0 0 2.0 rpy=0 0 0 -> xyz=0 0 2.0 rpy=0 0 0.7854
