Commit message: minor cosmetic changes, merged two for loops into one

File: puzzles/simple_sliders/urdf/simple_sliders.urdf (robot description, URDF)
Before this commit: robot simple_sliders, 6 links, 5 joints
Joints:
- joint link0: limit lower=0 upper=2.0 effort=0 velocity=0 -> lower=0 upper=1.0 effort=0 velocity=0
- joint link1: limit lower=0 upper=2.0 effort=0 velocity=0 -> lower=0 upper=1.0 effort=0 velocity=0
- joint link2: limit lower=0 upper=2.0 effort=0 velocity=0 -> lower=0 upper=1.0 effort=0 velocity=0
- joint link3: limit lower=0 upper=2.0 effort=0 velocity=0 -> lower=0 upper=1.0 effort=0 velocity=0
- joint link4: limit lower=0 upper=2.0 effort=0 velocity=0 -> lower=0 upper=1.0 effort=0 velocity=0

Commit message: 4 spaces instead of tab indent, added python subscript to solve the created urdf with pybullet ompl

File: puzzles/simple_sliders/urdf/simple_sliders.urdf (robot description, URDF)
Before this commit: robot simple_sliders, 6 links, 5 joints
Links:
- removed link link2
- removed link link3
- removed link link4
Joints:
- removed joint link2
- removed joint link3
- removed joint link4

Commit message: divide scaling factors by 2 because blender measures object size differently (divided by 2) compared to urdf

File: puzzles/simple_sliders/urdf/simple_sliders.urdf (robot description, URDF)
Before this commit: robot simple_sliders, 3 links, 2 joints
Links:
- link base_link: geometry collision box size=16.0 16.0 0.1; visual box size=16.0 16.0 0.1
- link link0: geometry collision box size=0.1 0.1 1.8; visual box size=0.1 0.1 1.8
- link link1: geometry collision box size=0.1 0.1 1.8; visual box size=0.1 0.1 1.8

Commit message: small fix: some numbers were incorrect due to the added division by 2

File: puzzles/simple_sliders/urdf/simple_sliders.urdf (robot description, URDF)
Before this commit: robot simple_sliders, 3 links, 2 joints
Links:
- link base_link: geometry collision box size=16.0 16.0 0.2; visual box size=16.0 16.0 0.2
- link link0: geometry collision box size=0.2 0.2 1.6; visual box size=0.2 0.2 1.6
- link link1: geometry collision box size=0.2 0.2 1.6; visual box size=0.2 0.2 1.6

Commit message: docstrings added, improved (class) structure

File: puzzles/simple_sliders/urdf/simple_sliders.urdf (robot description, URDF)
Before this commit: robot simple_sliders, 3 links, 2 joints
Links:
- added link link2, mass 0.001; collision box size=0.2 0.2 1.6; visual box size=0.2 0.2 1.6
Joints:
- added joint link2: type prismatic, parent base_link, child link2, origin xyz=1.0 -1.0 0.1 rpy=1.5708 0 0, axis 0 0 1.0, limit lower=0 upper=1.0 effort=0 velocity=0

Commit message: moved implementation of simple sliders to World

File: puzzles/simple_sliders/urdf/simple_sliders.urdf (robot description, URDF)
Before this commit: robot simple_sliders, 4 links, 3 joints
Links:
- removed link link2
Joints:
- removed joint link2
