Commit message: feat: choose exact solution and planner in test_with_pybullet_ompl()

File: puzzles/sampleworld/urdf/sampleworld.urdf (robot description, URDF)
Before this commit: robot sampleworld, 6 links, 5 joints
Links:
- link link1: geometry collision box size=3.0 1.0 1.0; visual box size=3.0 1.0 1.0
- link link2: geometry collision box size=1.0 1.0 2.0; visual box size=1.0 1.0 2.0
Joints:
- joint link1: limit lower=0 upper=1.0 effort=0 velocity=0 -> lower=0 upper=2.31933 effort=0 velocity=0; origin xyz=-2.10514 0.09608 0.5 rpy=-1.5708 0 -0.42202 -> xyz=-2.75846 -1.50998 0.5 rpy=0 0 -2.43302; type prismatic -> revolute
- joint link2: limit lower=0 upper=2.98164 effort=0 velocity=0 -> lower=0 upper=1.0 effort=0 velocity=0; origin xyz=-0.56079 3.01274 0.5 rpy=0 0 -0.48141 -> xyz=-2.81847 1.89345 0.5 rpy=-1.5708 0 -2.8865; type revolute -> prismatic
- joint link3: limit lower=0 upper=3.06268 effort=0 velocity=0 -> lower=0 upper=1.70019 effort=0 velocity=0; origin xyz=3.11277 4.96317 0.5 rpy=0 0 -0.65949 -> xyz=-0.99083 3.25291 0.5 rpy=0 0 -0.52187
- joint link4: origin xyz=5.59595 6.18261 0.5 rpy=-1.5708 0 0.51756 -> xyz=1.62317 3.35612 0.5 rpy=-1.5708 0 -2.00692

Commit message: feat: complete sampleworld

File: puzzles/sampleworld/urdf/sampleworld.urdf (robot description, URDF)
Before this commit: robot sampleworld, 6 links, 5 joints
Links:
- removed link link3
- removed link link4
- link link0: geometry collision box size=1.0 1.0 2.0; visual box size=1.0 1.0 2.0
- link link2: geometry collision box size=3.0 1.0 1.0; visual box size=3.0 1.0 1.0
Joints:
- removed joint link3
- removed joint link4
- joint link0: limit lower=0 upper=2.23143 effort=0 velocity=0 -> lower=0 upper=2.02255 effort=0 velocity=0; origin xyz=0 0 0.5 rpy=0 0 -0.97753 -> xyz=0 0 0.5 rpy=-1.5708 0 2.64253; type revolute -> prismatic
- joint link1: limit lower=0 upper=2.31933 effort=0 velocity=0 -> lower=0 upper=2.8855 effort=0 velocity=0; origin xyz=-2.75846 -1.50998 0.5 rpy=0 0 -2.43302 -> xyz=0.02182 -2.76373 0.5 rpy=0 0 -1.68642
- joint link2: limit lower=0 upper=1.0 effort=0 velocity=0 -> lower=0 upper=1.59781 effort=0 velocity=0; origin xyz=-2.81847 1.89345 0.5 rpy=-1.5708 0 -2.8865 -> xyz=2.09437 -3.70985 0.5 rpy=0 0 2.57551; type prismatic -> revolute

Commit message: feat: use goal SPACE instead of goal STATE
The goal space allows any position within the joint bounds, except for joint0: it must be moved to its limit.

File: puzzles/sampleworld/urdf/sampleworld.urdf (robot description, URDF)
Before this commit: robot sampleworld, 4 links, 3 joints
Joints:
- joint link1: limit lower=0 upper=2.8855 effort=0 velocity=0 -> lower=-3.05772 upper=0 effort=0 velocity=0; origin xyz=0.02182 -2.76373 0.5 rpy=0 0 -1.68642 -> xyz=-2.39635 -2.12185 0.5 rpy=0 0 -2.92672
- joint link2: limit lower=0 upper=1.59781 effort=0 velocity=0 -> lower=0 upper=2.20328 effort=0 velocity=0; origin xyz=2.09437 -3.70985 0.5 rpy=0 0 2.57551 -> xyz=-5.15238 -1.03587 0.5 rpy=0 0 0.26392

Commit message: feat: test_with_pybullet_ompl() now really takes a goal SPACE

File: puzzles/sampleworld/urdf/sampleworld.urdf (robot description, URDF)
Before this commit: robot sampleworld, 4 links, 3 joints
Links:
- link base_link: geometry collision box size=32.0 32.0 0.2; visual box size=32.0 32.0 0.2

Commit message: refactor: simplify sample_joint() by creating a separate function sample_first_joint() only for the first joint

File: puzzles/sampleworld/urdf/sampleworld.urdf (robot description, URDF)
Before this commit: robot sampleworld, 4 links, 3 joints
Links:
- link link0: geometry collision box size=3.0 1.0 1.0; visual box size=3.0 1.0 1.0
- link link2: geometry collision box size=1.0 1.0 2.0; visual box size=1.0 1.0 2.0
Joints:
- joint link0: limit lower=0 upper=2.02255 effort=0 velocity=0 -> lower=-1.82033 upper=0 effort=0 velocity=0; origin xyz=0 0 0.5 rpy=-1.5708 0 2.64253 -> xyz=0 0 0.5 rpy=0 0 -0.97753; type prismatic -> revolute
- joint link1: limit lower=-3.05772 upper=0 effort=0 velocity=0 -> lower=-2.79898 upper=0 effort=0 velocity=0; origin xyz=-2.39635 -2.12185 0.5 rpy=0 0 -2.92672 -> xyz=-2.51733 -1.07967 0.5 rpy=0 0 -3.0917
- joint link2: limit lower=0 upper=2.20328 effort=0 velocity=0 -> lower=0 upper=1.44092 effort=0 velocity=0; origin xyz=-5.15238 -1.03587 0.5 rpy=0 0 0.26392 -> xyz=-0.44686 -2.62146 0.5 rpy=-1.5708 0 -1.6871; type revolute -> prismatic
