Commit message: refactor: separate module calc for math functions

File: puzzles/my_custom_urdf/urdf/my_custom_urdf.urdf (robot description, URDF)
Before this commit: robot my_custom_urdf, 3 links, 2 joints
Links:
- added link link2, mass 0.001; collision box size=0.2 0.2 0.2; visual box size=0.2 0.2 0.2
- added link link3, mass 0.001; collision box size=0.2 0.2 0.2; visual box size=0.2 0.2 0.2
- link link0: geometry collision box size=2.0 0.2 4.0; visual box size=2.0 0.2 4.0
- link link1: geometry collision box size=1.0 1.0 4.0; visual box size=1.0 1.0 4.0
Joints:
- added joint link2: type prismatic, parent base_link, child link2, origin xyz=0 -4.0 0.1 rpy=0 0 0, axis 0 0 1.0, limit lower=0 upper=0 effort=0 velocity=0
- added joint link3: type prismatic, parent base_link, child link3, origin xyz=2.0 -3.4641 0.1 rpy=0 0 0.5236, axis 0 0 1.0, limit lower=0 upper=0 effort=0 velocity=0
- joint link0: limit lower=0 upper=2.0 effort=0 velocity=0 -> lower=-0.7854 upper=0.7854 effort=0 velocity=0; origin xyz=0 0 0.5 rpy=1.5708 0 0 -> xyz=0 4.0 2.0 rpy=0 0 0; type prismatic -> revolute
- joint link1: limit lower=-0.7854 upper=0.7854 effort=0 velocity=0 -> lower=0 upper=2.0 effort=0 velocity=0; origin xyz=0 4.0 2.0 rpy=0 0 0 -> xyz=0 0 0.5 rpy=1.5708 0 0.5236; type revolute -> prismatic

Commit message: refactor: improve performance with calculate_next_start_point() - to get a more accurate estimate location of the best sampling area - by tweaking some sampling parameters - and by reducing radians() calls

File: puzzles/my_custom_urdf/urdf/my_custom_urdf.urdf (robot description, URDF)
Before this commit: robot my_custom_urdf, 5 links, 4 joints
Joints:
- joint link0: origin xyz=0 4.0 2.0 rpy=0 0 0 -> xyz=0 5.0 2.0 rpy=0 0 0
- joint link1: origin xyz=0 0 0.5 rpy=1.5708 0 0.5236 -> xyz=0 0 0.5 rpy=-1.5708 0 0.5236
- joint link2: origin xyz=0 -4.0 0.1 rpy=0 0 0 -> xyz=0 4.0 0.1 rpy=0 0 0
- joint link3: origin xyz=2.0 -3.4641 0.1 rpy=0 0 0.5236 -> xyz=-2.0 3.4641 0.1 rpy=0 0 0.5236

File: puzzles/sampleworld/urdf/sampleworld.urdf (robot description, URDF)
Before this commit: robot sampleworld, 4 links, 3 joints
Joints:
- joint link1: limit lower=-2.79898 upper=0 effort=0 velocity=0 -> lower=0 upper=1.58552 effort=0 velocity=0; origin xyz=-2.51733 -1.07967 0.5 rpy=0 0 -3.0917 -> xyz=1.89729 1.60702 0.5 rpy=0 0 -2.61769
- joint link2: limit lower=0 upper=1.44092 effort=0 velocity=0 -> lower=0 upper=3.81949 effort=0 velocity=0; origin xyz=-0.44686 -2.62146 0.5 rpy=-1.5708 0 -1.6871 -> xyz=2.7436 -0.22319 0.5 rpy=-1.5708 0 -2.39786

Commit message: fix: correct values of calc.RAD180 and RAD360 and remove radians() calls completely (for improved performance)

File: puzzles/my_custom_urdf/urdf/my_custom_urdf.urdf (robot description, URDF)
Before this commit: robot my_custom_urdf, 5 links, 4 joints
Joints:
- joint link1: origin xyz=0 0 0.5 rpy=-1.5708 0 0.5236 -> xyz=0 0 0.5 rpy=-1.5708 0 0.7854
- joint link3: origin xyz=-2.0 3.4641 0.1 rpy=0 0 0.5236 -> xyz=-2.82843 2.82843 0.1 rpy=0 0 0.7854
