Commit message: implemented create_gridworld_puzzle() (only for prismatic joints, yet)

File: puzzles/gridworld/urdf/gridworld.urdf (robot description, URDF)
Before this commit: robot gridworld, 3 links, 2 joints
Links:
- added link link2, mass 0.001; collision box size=0.8 0.8 1.8; visual box size=0.8 0.8 1.8
- added link link3, mass 0.001; collision box size=0.8 0.8 1.8; visual box size=0.8 0.8 1.8
- link link1: geometry collision box size=0.8 0.8 1.8; visual box size=0.8 0.8 1.8
Joints:
- added joint link2: type prismatic, parent base_link, child link2, origin xyz=-2.0 2.5 0.4 rpy=-1.5708 0 0, axis 0 0 1.0, limit lower=0 upper=1.0 effort=0 velocity=0
- added joint link3: type prismatic, parent base_link, child link3, origin xyz=-1.5 4.0 0.4 rpy=0 1.5708 0, axis 0 0 1.0, limit lower=0 upper=1.0 effort=0 velocity=0
- joint link0: origin xyz=0 0.5 0.4 rpy=-1.5708 0 0 -> xyz=-0.5 0 0.4 rpy=0 -1.5708 0
- joint link1: limit lower=0 upper=1.5708 effort=0 velocity=0 -> lower=0 upper=1.0 effort=0 velocity=0; origin xyz=-0.5 2.0 0.9 rpy=0 0 0 -> xyz=-2.0 0.5 0.4 rpy=-1.5708 0 0; type revolute -> prismatic

Commit message: seed()

File: puzzles/gridworld/urdf/gridworld.urdf (robot description, URDF)
Before this commit: robot gridworld, 5 links, 4 joints
Joints:
- joint link0: origin xyz=-0.5 0 0.4 rpy=0 -1.5708 0 -> xyz=0 -0.5 0.4 rpy=1.5708 0 0
- joint link1: origin xyz=-2.0 0.5 0.4 rpy=-1.5708 0 0 -> xyz=-0.5 -2.0 0.4 rpy=0 -1.5708 0
- joint link2: origin xyz=-2.0 2.5 0.4 rpy=-1.5708 0 0 -> xyz=-2.5 -2.0 0.4 rpy=0 -1.5708 0
- joint link3: origin xyz=-1.5 4.0 0.4 rpy=0 1.5708 0 -> xyz=-4.0 -1.5 0.4 rpy=-1.5708 0 0

Commit message: create_gridworld_puzzle() done incl revolute joints
goal_state is now an attribute of World

File: puzzles/gridworld/urdf/gridworld.urdf (robot description, URDF)
Before this commit: robot gridworld, 5 links, 4 joints
Links:
- added link link4, mass 0.001; collision box size=0.8 0.8 1.8; visual box size=0.8 0.8 1.8
- added link link5, mass 0.001; collision box size=0.8 0.8 1.8; visual box size=0.8 0.8 1.8
- added link link6, mass 0.001; collision box size=0.8 0.8 1.8; visual box size=0.8 0.8 1.8
- link link0: geometry collision box size=1.8 0.1 1.8; visual box size=1.8 0.1 1.8
- link link1: geometry collision box size=1.8 0.1 1.8; visual box size=1.8 0.1 1.8
- link link3: geometry collision box size=1.8 0.1 1.8; visual box size=1.8 0.1 1.8
Joints:
- added joint link4: type prismatic, parent base_link, child link4, origin xyz=-0.5 -4.0 0.4 rpy=0 1.5708 0, axis 0 0 1.0, limit lower=0 upper=1.0 effort=0 velocity=0
- added joint link5: type prismatic, parent base_link, child link5, origin xyz=1.0 -4.5 0.4 rpy=1.5708 0 0, axis 0 0 1.0, limit lower=0 upper=1.0 effort=0 velocity=0
- added joint link6: type prismatic, parent base_link, child link6, origin xyz=1.5 -6.0 0.4 rpy=0 1.5708 0, axis 0 0 1.0, limit lower=0 upper=1.0 effort=0 velocity=0
- joint link0: limit lower=0 upper=1.0 effort=0 velocity=0 -> lower=0 upper=1.5708 effort=0 velocity=0; origin xyz=0 -0.5 0.4 rpy=1.5708 0 0 -> xyz=-0.5 0 0.9 rpy=0 0 0; type prismatic -> revolute
- joint link1: limit lower=0 upper=1.0 effort=0 velocity=0 -> lower=-1.5708 upper=0 effort=0 velocity=0; origin xyz=-0.5 -2.0 0.4 rpy=0 -1.5708 0 -> xyz=-1.0 -1.5 0.9 rpy=0 0 1.5708; type prismatic -> revolute
- joint link2: origin xyz=-2.5 -2.0 0.4 rpy=0 -1.5708 0 -> xyz=-2.0 -2.5 0.4 rpy=1.5708 0 0
- joint link3: limit lower=0 upper=1.0 effort=0 velocity=0 -> lower=-1.5708 upper=0 effort=0 velocity=0; origin xyz=-4.0 -1.5 0.4 rpy=-1.5708 0 0 -> xyz=-2.0 -4.5 0.9 rpy=0 0 1.5708; type prismatic -> revolute

Commit message: fix: adequate box size for revolute joints -> better gridworld puzzles
feat: also print created sequence to console (minor change)

File: puzzles/gridworld/urdf/gridworld.urdf (robot description, URDF)
Before this commit: robot gridworld, 8 links, 7 joints
Links:
- removed link link4
- removed link link5
- removed link link6
- link link0: geometry collision box size=0.9 0.9 1.9; visual box size=0.9 0.9 1.9
- link link1: geometry collision box size=2.9 0.9 0.9; visual box size=2.9 0.9 0.9
- link link2: geometry collision box size=0.9 0.9 1.9; visual box size=0.9 0.9 1.9
- link link3: geometry collision box size=2.9 0.9 0.9; visual box size=2.9 0.9 0.9
Joints:
- removed joint link4
- removed joint link5
- removed joint link6
- joint link0: limit lower=0 upper=1.5708 effort=0 velocity=0 -> lower=0 upper=1.0 effort=0 velocity=0; origin xyz=-0.5 0 0.9 rpy=0 0 0 -> xyz=0.5 0 0.45 rpy=0 1.5708 0; type revolute -> prismatic
- joint link1: origin xyz=-1.0 -1.5 0.9 rpy=0 0 1.5708 -> xyz=2.0 -1.0 0.45 rpy=0 0 1.5708
- joint link2: origin xyz=-2.0 -2.5 0.4 rpy=1.5708 0 0 -> xyz=3.0 0.5 0.45 rpy=-1.5708 0 0
- joint link3: limit lower=-1.5708 upper=0 effort=0 velocity=0 -> lower=0 upper=1.5708 effort=0 velocity=0; origin xyz=-2.0 -4.5 0.9 rpy=0 0 1.5708 -> xyz=2.0 2.0 0.45 rpy=0 0 0

Commit message: feat: move start_point from (0, 0) to (0.5, 0.5) to align boxes better in rviz

File: puzzles/gridworld/urdf/gridworld.urdf (robot description, URDF)
Before this commit: robot gridworld, 5 links, 4 joints
Joints:
- joint link0: origin xyz=0.5 0 0.45 rpy=0 1.5708 0 -> xyz=1.0 0.5 0.45 rpy=0 1.5708 0
- joint link1: origin xyz=2.0 -1.0 0.45 rpy=0 0 1.5708 -> xyz=2.5 -0.5 0.45 rpy=0 0 1.5708
- joint link2: origin xyz=3.0 0.5 0.45 rpy=-1.5708 0 0 -> xyz=3.5 1.0 0.45 rpy=-1.5708 0 0
- joint link3: origin xyz=2.0 2.0 0.45 rpy=0 0 0 -> xyz=2.5 2.5 0.45 rpy=0 0 0

Commit message: feat: degree_of_branching can be set in config
this new parameter can increase the complexity of the puzzle without increasing the DOFs

start_point is now a queue of start_points

File: puzzles/gridworld/urdf/gridworld.urdf (robot description, URDF)
Before this commit: robot gridworld, 5 links, 4 joints
Links:
- added link link4, mass 0.001; collision box size=0.9 0.9 1.9; visual box size=0.9 0.9 1.9
- link link0: geometry collision box size=2.9 0.9 0.9; visual box size=2.9 0.9 0.9
- link link2: geometry collision box size=2.9 0.9 0.9; visual box size=2.9 0.9 0.9
- link link3: geometry collision box size=0.9 0.9 1.9; visual box size=0.9 0.9 1.9
Joints:
- added joint link4: type prismatic, parent base_link, child link4, origin xyz=-3.5 1.0 0.45 rpy=-1.5708 0 0, axis 0 0 1.0, limit lower=0 upper=1.0 effort=0 velocity=0
- joint link0: limit lower=0 upper=1.0 effort=0 velocity=0 -> lower=0 upper=1.5708 effort=0 velocity=0; origin xyz=1.0 0.5 0.45 rpy=0 1.5708 0 -> xyz=-0.5 0.5 0.45 rpy=0 0 0; type prismatic -> revolute
- joint link1: origin xyz=2.5 -0.5 0.45 rpy=0 0 1.5708 -> xyz=-2.5 -0.5 0.45 rpy=0 0 0
- joint link2: limit lower=0 upper=1.0 effort=0 velocity=0 -> lower=-1.5708 upper=0 effort=0 velocity=0; origin xyz=3.5 1.0 0.45 rpy=-1.5708 0 0 -> xyz=1.5 1.5 0.45 rpy=0 0 0; type prismatic -> revolute
- joint link3: limit lower=0 upper=1.5708 effort=0 velocity=0 -> lower=0 upper=1.0 effort=0 velocity=0; origin xyz=2.5 2.5 0.45 rpy=0 0 0 -> xyz=-1.5 -2.0 0.45 rpy=1.5708 0 0; type revolute -> prismatic

Commit message: refactor: make name update of world possible and move sampler attributes floor_size, allow_clockwise and attempts

File: puzzles/gridworld/urdf/gridworld.urdf (robot description, URDF)
Before this commit: robot gridworld, 6 links, 5 joints
Links:
- removed link link3
- removed link link4
- link base_link: geometry collision box size=32.0 32.0 0.2; visual box size=32.0 32.0 0.2
- link link2: geometry collision box size=0.9 0.9 1.9; visual box size=0.9 0.9 1.9
Joints:
- removed joint link3
- removed joint link4
- joint link2: limit lower=-1.5708 upper=0 effort=0 velocity=0 -> lower=0 upper=1.0 effort=0 velocity=0; origin xyz=1.5 1.5 0.45 rpy=0 0 0 -> xyz=1.0 1.5 0.45 rpy=0 1.5708 0; type revolute -> prismatic

File: puzzles/simple_sliders/urdf/simple_sliders.urdf (robot description, URDF)
Before this commit: robot simple_sliders, 3 links, 2 joints
Links:
- removed link link1
- link base_link: geometry collision box size=32.0 32.0 0.2; visual box size=32.0 32.0 0.2
Joints:
- removed joint link1

Commit message: chore (minor): nicer examples (2 prismatic joints)

File: puzzles/gridworld/urdf/gridworld.urdf (robot description, URDF)
Before this commit: robot gridworld, 4 links, 3 joints
Links:
- added link link3, mass 0.001; collision box size=0.9 0.9 1.9; visual box size=0.9 0.9 1.9
Joints:
- added joint link3: type prismatic, parent base_link, child link3, origin xyz=-1.5 -2.0 0.45 rpy=1.5708 0 0, axis 0 0 1.0, limit lower=0 upper=1.0 effort=0 velocity=0

File: puzzles/sampleworld/urdf/sampleworld.urdf (robot description, URDF)
Before this commit: robot sampleworld, 4 links, 3 joints
Links:
- added link link3, mass 0.001; collision box size=1.0 1.0 2.0; visual box size=1.0 1.0 2.0
Joints:
- added joint link3: type prismatic, parent base_link, child link3, origin xyz=3.51572 -2.56209 0.5 rpy=-1.5708 0 -2.44487, axis 0 0 1.0, limit lower=0 upper=3.93321 effort=0 velocity=0

File: puzzles/simple_sliders/urdf/simple_sliders.urdf (robot description, URDF)
Before this commit: robot simple_sliders, 2 links, 1 joints
Links:
- added link link1, mass 0.001; collision box size=0.2 0.2 1.6; visual box size=0.2 0.2 1.6
Joints:
- added joint link1: type prismatic, parent base_link, child link1, origin xyz=0 -1.0 0.1 rpy=0 1.5708 0, axis 0 0 1.0, limit lower=0 upper=1.0 effort=0 velocity=0
