Commit message: feat: meshes

File: puzzles/continuous_space/urdf/unnamed.urdf (robot description, URDF)
Before this commit: robot unnamed, 2 links, 1 joints
Links:
- link link_cog: geometry collision mesh filename=file:///home/userone/ba/puzzle-generator/puzzles/continuous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 scale=1.0 1.0 1.0; visual mesh filename=file:///home/userone/ba/puzzle-generator/puzzles/continuous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 scale=1.0 1.0 1.0

File: puzzles/my_custom/urdf/my_custom.urdf (robot description, URDF)
Before this commit: robot my_custom, 5 links, 4 joints
Links:
- added link link4, mass 0.001; collision mesh filename=file:///home/userone/ba/puzzle-generator/puzzles/my_custom/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 scale=1.0 1.0 1.0; visual mesh filename=file:///home/userone/ba/puzzle-generator/puzzles/my_custom/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 scale=0.5 0.5 0.5
- link base_link: geometry collision box size=32.0 32.0 0.2; visual box size=32.0 32.0 0.2
Joints:
- added joint link4: type revolute, parent base_link, child link4, origin xyz=0 -5.0 0.5 rpy=0 0 0, axis 0 0 1.0, limit lower=-0.7854 upper=0.7854 effort=0 velocity=0
