Commit message: chore (minor): rename files and folders

File: puzzles/continuous_space/urdf/continuous_space.urdf (robot description, URDF)
Before this commit: robot gridworld, 5 links, 4 joints
Links:
- link link0: geometry collision box size=3.0 1.0 1.0; visual box size=3.0 1.0 1.0
- link link1: geometry collision box size=3.0 1.0 1.0; visual box size=3.0 1.0 1.0
- link link2: geometry collision box size=1.0 1.0 2.0; visual box size=1.0 1.0 2.0
- link link3: geometry collision box size=1.0 1.0 2.0; visual box size=1.0 1.0 2.0
Joints:
- joint link0: limit lower=0 upper=1.5708 effort=0 velocity=0 -> lower=-1.82033 upper=0 effort=0 velocity=0; origin xyz=-0.5 0.5 0.45 rpy=0 0 0 -> xyz=0 0 0.5 rpy=0 0 -0.97753
- joint link1: limit lower=-1.5708 upper=0 effort=0 velocity=0 -> lower=0 upper=1.58552 effort=0 velocity=0; origin xyz=-2.5 -0.5 0.45 rpy=0 0 0 -> xyz=1.89729 1.60702 0.5 rpy=0 0 -2.61769
- joint link2: limit lower=0 upper=1.0 effort=0 velocity=0 -> lower=0 upper=3.81949 effort=0 velocity=0; origin xyz=1.0 1.5 0.45 rpy=0 1.5708 0 -> xyz=2.7436 -0.22319 0.5 rpy=-1.5708 0 -2.39786
- joint link3: limit lower=0 upper=1.0 effort=0 velocity=0 -> lower=0 upper=3.93321 effort=0 velocity=0; origin xyz=-1.5 -2.0 0.45 rpy=1.5708 0 0 -> xyz=3.51572 -2.56209 0.5 rpy=-1.5708 0 -2.44487

File: puzzles/grid_world/urdf/grid_world.urdf (robot description, URDF)
Before this commit: robot my_custom_urdf, 5 links, 4 joints
Links:
- link base_link: geometry collision box size=32.0 32.0 0.2; visual box size=32.0 32.0 0.2
- link link0: geometry collision box size=2.9 0.9 0.9; visual box size=2.9 0.9 0.9
- link link1: geometry collision box size=2.9 0.9 0.9; visual box size=2.9 0.9 0.9
- link link2: geometry collision box size=0.9 0.9 1.9; visual box size=0.9 0.9 1.9
- link link3: geometry collision box size=0.9 0.9 1.9; visual box size=0.9 0.9 1.9
Joints:
- joint link0: limit lower=-0.7854 upper=0.7854 effort=0 velocity=0 -> lower=0 upper=1.5708 effort=0 velocity=0; origin xyz=0 5.0 2.0 rpy=0 0 0 -> xyz=-0.5 0.5 0.45 rpy=0 0 0
- joint link1: limit lower=0 upper=2.0 effort=0 velocity=0 -> lower=-1.5708 upper=0 effort=0 velocity=0; origin xyz=0 0 0.5 rpy=-1.5708 0 0.7854 -> xyz=-2.5 -0.5 0.45 rpy=0 0 0; type prismatic -> revolute
- joint link2: limit lower=0 upper=0 effort=0 velocity=0 -> lower=0 upper=1.0 effort=0 velocity=0; origin xyz=0 4.0 0.1 rpy=0 0 0 -> xyz=1.0 1.5 0.45 rpy=0 1.5708 0
- joint link3: limit lower=0 upper=0 effort=0 velocity=0 -> lower=0 upper=1.0 effort=0 velocity=0; origin xyz=-2.82843 2.82843 0.1 rpy=0 0 0.7854 -> xyz=-1.5 -2.0 0.45 rpy=1.5708 0 0

File: puzzles/my_custom/urdf/my_custom.urdf (robot description, URDF)
Before this commit: robot sampleworld, 5 links, 4 joints
Links:
- link base_link: geometry collision box size=0 0 0.2; visual box size=0 0 0.2
- link link0: geometry collision box size=2.0 0.2 4.0; visual box size=2.0 0.2 4.0
- link link1: geometry collision box size=1.0 1.0 4.0; visual box size=1.0 1.0 4.0
- link link2: geometry collision box size=0.2 0.2 0.2; visual box size=0.2 0.2 0.2
- link link3: geometry collision box size=0.2 0.2 0.2; visual box size=0.2 0.2 0.2
Joints:
- joint link0: limit lower=-1.82033 upper=0 effort=0 velocity=0 -> lower=-0.7854 upper=0.7854 effort=0 velocity=0; origin xyz=0 0 0.5 rpy=0 0 -0.97753 -> xyz=0 5.0 2.0 rpy=0 0 0
- joint link1: limit lower=0 upper=1.58552 effort=0 velocity=0 -> lower=0 upper=2.0 effort=0 velocity=0; origin xyz=1.89729 1.60702 0.5 rpy=0 0 -2.61769 -> xyz=0 0 0.5 rpy=-1.5708 0 0.7854; type revolute -> prismatic
- joint link2: limit lower=0 upper=3.81949 effort=0 velocity=0 -> lower=0 upper=0 effort=0 velocity=0; origin xyz=2.7436 -0.22319 0.5 rpy=-1.5708 0 -2.39786 -> xyz=0 4.0 0.1 rpy=0 0 0
- joint link3: limit lower=0 upper=3.93321 effort=0 velocity=0 -> lower=0 upper=0 effort=0 velocity=0; origin xyz=3.51572 -2.56209 0.5 rpy=-1.5708 0 -2.44487 -> xyz=-2.82843 2.82843 0.1 rpy=0 0 0.7854

Commit message: fix: consider floor_thickness when placing objects

File: puzzles/continuous_space/urdf/continuous_space.urdf (robot description, URDF)
Before this commit: robot continuous_space, 5 links, 4 joints
Joints:
- joint link0: origin xyz=0 0 0.5 rpy=0 0 -0.97753 -> xyz=0 0 0.6 rpy=0 0 -0.97753
- joint link1: origin xyz=1.89729 1.60702 0.5 rpy=0 0 -2.61769 -> xyz=1.89729 1.60702 0.6 rpy=0 0 -2.61769
- joint link2: origin xyz=2.7436 -0.22319 0.5 rpy=-1.5708 0 -2.39786 -> xyz=2.7436 -0.22319 0.6 rpy=-1.5708 0 -2.39786
- joint link3: origin xyz=3.51572 -2.56209 0.5 rpy=-1.5708 0 -2.44487 -> xyz=3.51572 -2.56209 0.6 rpy=-1.5708 0 -2.44487

File: puzzles/grid_world/urdf/grid_world.urdf (robot description, URDF)
Before this commit: robot grid_world, 5 links, 4 joints
Joints:
- joint link0: origin xyz=-0.5 0.5 0.45 rpy=0 0 0 -> xyz=-0.5 0.5 0.55 rpy=0 0 0
- joint link1: origin xyz=-2.5 -0.5 0.45 rpy=0 0 0 -> xyz=-2.5 -0.5 0.55 rpy=0 0 0
- joint link2: origin xyz=1.0 1.5 0.45 rpy=0 1.5708 0 -> xyz=1.0 1.5 0.55 rpy=0 1.5708 0
- joint link3: origin xyz=-1.5 -2.0 0.45 rpy=1.5708 0 0 -> xyz=-1.5 -2.0 0.55 rpy=1.5708 0 0

File: puzzles/simple_sliders/urdf/simple_sliders.urdf (robot description, URDF)
Before this commit: robot simple_sliders, 3 links, 2 joints
Joints:
- joint link0: origin xyz=0 0 0.1 rpy=1.5708 0 0 -> xyz=0 0 0.2 rpy=1.5708 0 0
- joint link1: origin xyz=0 -1.0 0.1 rpy=0 1.5708 0 -> xyz=0 -1.0 0.2 rpy=0 1.5708 0

Commit message: chore: make goal green and any other link red

File: puzzles/continuous_space/urdf/continuous_space.urdf (robot description, URDF)
Before this commit: robot continuous_space, 5 links, 4 joints
Links:
- removed link link0
- removed link link1
- removed link link2
- removed link link3
- added link link_0, mass 0.001; collision box size=3.0 1.0 1.0; visual box size=3.0 1.0 1.0
- added link link_1, mass 0.001; collision box size=3.0 1.0 1.0; visual box size=3.0 1.0 1.0
- added link link_2, mass 0.001; collision box size=1.0 1.0 2.0; visual box size=1.0 1.0 2.0
- added link link_3, mass 0.001; collision box size=1.0 1.0 2.0; visual box size=1.0 1.0 2.0
Joints:
- removed joint link0
- removed joint link1
- removed joint link2
- removed joint link3
- added joint link_0: type revolute, parent base_link, child link_0, origin xyz=0 0 0.6 rpy=0 0 -0.97753, axis 0 0 1.0, limit lower=-1.82033 upper=0 effort=0 velocity=0
- added joint link_1: type revolute, parent base_link, child link_1, origin xyz=1.89729 1.60702 0.6 rpy=0 0 -2.61769, axis 0 0 1.0, limit lower=0 upper=1.58552 effort=0 velocity=0
- added joint link_2: type prismatic, parent base_link, child link_2, origin xyz=2.7436 -0.22319 0.6 rpy=-1.5708 0 -2.39786, axis 0 0 1.0, limit lower=0 upper=3.81949 effort=0 velocity=0
- added joint link_3: type prismatic, parent base_link, child link_3, origin xyz=6.16197 -1.43395 0.6 rpy=-1.5708 0 -0.61471, axis 0 0 1.0, limit lower=0 upper=3.45966 effort=0 velocity=0

File: puzzles/grid_world/urdf/grid_world.urdf (robot description, URDF)
Before this commit: robot grid_world, 5 links, 4 joints
Links:
- removed link link0
- removed link link1
- removed link link2
- removed link link3
- added link link_0, mass 0.001; collision box size=2.9 0.9 0.9; visual box size=2.9 0.9 0.9
- added link link_1, mass 0.001; collision box size=2.9 0.9 0.9; visual box size=2.9 0.9 0.9
- added link link_2, mass 0.001; collision box size=0.9 0.9 1.9; visual box size=0.9 0.9 1.9
- added link link_3, mass 0.001; collision box size=0.9 0.9 1.9; visual box size=0.9 0.9 1.9
Joints:
- removed joint link0
- removed joint link1
- removed joint link2
- removed joint link3
- added joint link_0: type revolute, parent base_link, child link_0, origin xyz=-0.5 0.5 0.55 rpy=0 0 0, axis 0 0 1.0, limit lower=0 upper=1.5708 effort=0 velocity=0
- added joint link_1: type revolute, parent base_link, child link_1, origin xyz=-2.5 -0.5 0.55 rpy=0 0 0, axis 0 0 1.0, limit lower=-1.5708 upper=0 effort=0 velocity=0
- added joint link_2: type prismatic, parent base_link, child link_2, origin xyz=1.0 1.5 0.55 rpy=0 1.5708 0, axis 0 0 1.0, limit lower=0 upper=1.0 effort=0 velocity=0
- added joint link_3: type prismatic, parent base_link, child link_3, origin xyz=-1.5 -2.0 0.55 rpy=1.5708 0 0, axis 0 0 1.0, limit lower=0 upper=1.0 effort=0 velocity=0

File: puzzles/lockbox2017/urdf/lockbox2017.urdf (robot description, URDF)
Before this commit: robot lockbox2017, 6 links, 5 joints
Links:
- removed link link0
- removed link link1
- removed link link2
- removed link link3
- removed link link4
- added link link_0, mass 0.001; collision box size=3.6 0.8 1.0; visual box size=3.6 0.8 1.0
- added link link_1, mass 0.001; collision box size=0.8 1.0 3.6; visual box size=0.8 1.0 3.6
- added link link_2, mass 0.001; collision mesh filename=file:///home/userone/ba/puzzle-generator/puzzles/lockbox201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 scale=1.0 1.0 1.0; visual mesh filename=file:///home/userone/ba/puzzle-generator/puzzles/lockbox201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 scale=1.0 1.0 1.0
- added link link_3, mass 0.001; collision box size=0.8 1.0 3.6; visual box size=0.8 1.0 3.6
- added link link_4, mass 0.001; collision box size=3.6 0.8 1.0; visual box size=3.6 0.8 1.0
Joints:
- removed joint link0
- removed joint link1
- removed joint link2
- removed joint link3
- removed joint link4
- added joint link_0: type revolute, parent base_link, child link_0, origin xyz=-6.0 -1.0 0.6 rpy=0 0 0, axis 0 0 1.0, limit lower=0 upper=1.5708 effort=0 velocity=0
- added joint link_1: type prismatic, parent base_link, child link_1, origin xyz=-4.0 0 0.6 rpy=-1.5708 0 -1.5708, axis 0 0 1.0, limit lower=0 upper=2.0 effort=0 velocity=0
- added joint link_2: type revolute, parent base_link, child link_2, origin xyz=0 0 0.6 rpy=0 0 1.5708, axis 0 0 1.0, limit lower=-3.14159 upper=3.14159 effort=0 velocity=0
- added joint link_3: type prismatic, parent base_link, child link_3, origin xyz=0 2.0 0.6 rpy=-1.5708 0 0, axis 0 0 1.0, limit lower=0 upper=2.0 effort=0 velocity=0
- added joint link_4: type revolute, parent base_link, child link_4, origin xyz=-1.0 5.0 0.6 rpy=0 0 0, axis 0 0 1.0, limit lower=0 upper=1.5708 effort=0 velocity=0

File: puzzles/simple_sliders/urdf/simple_sliders.urdf (robot description, URDF)
Before this commit: robot simple_sliders, 3 links, 2 joints
Links:
- removed link link0
- removed link link1
- added link link_0, mass 0.001; collision box size=0.2 0.2 1.6; visual box size=0.2 0.2 1.6
- added link link_1, mass 0.001; collision box size=0.2 0.2 1.6; visual box size=0.2 0.2 1.6
Joints:
- removed joint link0
- removed joint link1
- added joint link_0: type prismatic, parent base_link, child link_0, origin xyz=0 0 0.2 rpy=1.5708 0 0, axis 0 0 1.0, limit lower=0 upper=1.0 effort=0 velocity=0
- added joint link_1: type prismatic, parent base_link, child link_1, origin xyz=0 -1.0 0.2 rpy=0 1.5708 0, axis 0 0 1.0, limit lower=0 upper=1.0 effort=0 velocity=0

Commit message: chore (minor): update continuous_space.urdf

File: puzzles/continuous_space/urdf/continuous_space.urdf (robot description, URDF)
Before this commit: robot continuous_space, 5 links, 4 joints
Joints:
- joint link_3: limit lower=0 upper=3.45966 effort=0 velocity=0 -> lower=0 upper=3.93321 effort=0 velocity=0; origin xyz=6.16197 -1.43395 0.6 rpy=-1.5708 0 -0.61471 -> xyz=3.51572 -2.56209 0.6 rpy=-1.5708 0 -2.44487
