Commit message: feat: create_handle_automatically(), add hinge for revolute joints

File: puzzles/continuous_space/urdf/continuous_space.urdf (robot description, URDF)
Before this commit: robot continuous_space, 5 links, 4 joints
Links:
- added link link_handle_knob_0, mass 0.001; collision box size=0.05 0.05 0.2; visual box size=0.05 0.05 0.2
- added link link_handle_knob_1, mass 0.001; collision box size=0.05 0.05 0.2; visual box size=0.05 0.05 0.2
- added link link_handle_knob_2, mass 0.001; collision box size=0.05 0.05 0.2; visual box size=0.05 0.05 0.2
- added link link_handle_knob_3, mass 0.001; collision box size=0.05 0.05 0.2; visual box size=0.05 0.05 0.2
- added link link_handle_shaft_0, mass 0.001; collision cylinder length=1.0 radius=0.1; visual cylinder length=1.0 radius=0.1
- added link link_handle_shaft_1, mass 0.001; collision cylinder length=1.0 radius=0.1; visual cylinder length=1.0 radius=0.1
- added link link_handle_shaft_2, mass 0.001; collision box size=0.2 0.2 1.0; visual box size=0.2 0.2 1.0
- added link link_handle_shaft_3, mass 0.001; collision box size=0.2 0.2 1.0; visual box size=0.2 0.2 1.0
- added link link_hinge_0, mass 0.001; collision cylinder length=1.1 radius=0.05; visual cylinder length=1.1 radius=0.05
- added link link_hinge_1, mass 0.001; collision cylinder length=1.1 radius=0.05; visual cylinder length=1.1 radius=0.05
Joints:
- added joint link_handle_knob_0: type fixed, parent link_handle_shaft_0, child link_handle_knob_0, origin xyz=0 0 0.6 rpy=0 0 0
- added joint link_handle_knob_1: type fixed, parent link_handle_shaft_1, child link_handle_knob_1, origin xyz=0 0 0.6 rpy=0 0 0
- added joint link_handle_knob_2: type fixed, parent link_handle_shaft_2, child link_handle_knob_2, origin xyz=0 0 0.6 rpy=0 0 0
- added joint link_handle_knob_3: type fixed, parent link_handle_shaft_3, child link_handle_knob_3, origin xyz=0 0 0.6 rpy=0 0 0
- added joint link_handle_shaft_0: type fixed, parent link_0, child link_handle_shaft_0, origin xyz=1.125 0 1.0 rpy=0 0 0
- added joint link_handle_shaft_1: type fixed, parent link_1, child link_handle_shaft_1, origin xyz=1.125 0 1.0 rpy=0 0 0
- added joint link_handle_shaft_2: type fixed, parent link_2, child link_handle_shaft_2, origin xyz=0 -1.0 0 rpy=1.5708 0 0
- added joint link_handle_shaft_3: type fixed, parent link_3, child link_handle_shaft_3, origin xyz=0 -1.0 0 rpy=1.5708 0 0
- added joint link_hinge_0: type fixed, parent link_0, child link_hinge_0, origin xyz=0 0 0 rpy=0 0 0
- added joint link_hinge_1: type fixed, parent link_1, child link_hinge_1, origin xyz=0 0 0 rpy=0 0 0
- joint link_3: limit lower=0 upper=3.93321 effort=0 velocity=0 -> lower=0 upper=2.2014 effort=0 velocity=0; origin xyz=3.51572 -2.56209 0.6 rpy=-1.5708 0 -2.44487 -> xyz=5.40311 -1.16809 0.6 rpy=-1.5708 0 -1.98559

File: puzzles/grid_world/urdf/grid_world.urdf (robot description, URDF)
Before this commit: robot grid_world, 5 links, 4 joints
Links:
- added link link_handle_knob_0, mass 0.001; collision box size=0.05 0.05 0.2; visual box size=0.05 0.05 0.2
- added link link_handle_knob_1, mass 0.001; collision box size=0.05 0.05 0.2; visual box size=0.05 0.05 0.2
- added link link_handle_knob_2, mass 0.001; collision box size=0.05 0.05 0.2; visual box size=0.05 0.05 0.2
- added link link_handle_knob_3, mass 0.001; collision box size=0.05 0.05 0.2; visual box size=0.05 0.05 0.2
- added link link_handle_shaft_0, mass 0.001; collision cylinder length=1.0 radius=0.1; visual cylinder length=1.0 radius=0.1
- added link link_handle_shaft_1, mass 0.001; collision cylinder length=1.0 radius=0.1; visual cylinder length=1.0 radius=0.1
- added link link_handle_shaft_2, mass 0.001; collision box size=0.2 0.2 1.0; visual box size=0.2 0.2 1.0
- added link link_handle_shaft_3, mass 0.001; collision box size=0.2 0.2 1.0; visual box size=0.2 0.2 1.0
- added link link_hinge_0, mass 0.001; collision cylinder length=1.0 radius=0.05; visual cylinder length=1.0 radius=0.05
- added link link_hinge_1, mass 0.001; collision cylinder length=1.0 radius=0.05; visual cylinder length=1.0 radius=0.05
Joints:
- added joint link_handle_knob_0: type fixed, parent link_handle_shaft_0, child link_handle_knob_0, origin xyz=0 0 0.6 rpy=0 0 0
- added joint link_handle_knob_1: type fixed, parent link_handle_shaft_1, child link_handle_knob_1, origin xyz=0 0 0.6 rpy=0 0 0
- added joint link_handle_knob_2: type fixed, parent link_handle_shaft_2, child link_handle_knob_2, origin xyz=0 0 0.6 rpy=0 0 0
- added joint link_handle_knob_3: type fixed, parent link_handle_shaft_3, child link_handle_knob_3, origin xyz=0 0 0.6 rpy=0 0 0
- added joint link_handle_shaft_0: type fixed, parent link_0, child link_handle_shaft_0, origin xyz=1.0875 0 0.95 rpy=0 0 0
- added joint link_handle_shaft_1: type fixed, parent link_1, child link_handle_shaft_1, origin xyz=1.0875 0 0.95 rpy=0 0 0
- added joint link_handle_shaft_2: type fixed, parent link_2, child link_handle_shaft_2, origin xyz=-0.95 0 0 rpy=0 -1.5708 0
- added joint link_handle_shaft_3: type fixed, parent link_3, child link_handle_shaft_3, origin xyz=0 0.95 0 rpy=-1.5708 0 0
- added joint link_hinge_0: type fixed, parent link_0, child link_hinge_0, origin xyz=0 0 0 rpy=0 0 0
- added joint link_hinge_1: type fixed, parent link_1, child link_hinge_1, origin xyz=0 0 0 rpy=0 0 0

File: puzzles/lockbox2017/urdf/lockbox2017.urdf (robot description, URDF)
Before this commit: robot lockbox2017, 12 links, 11 joints
Links:
- removed link link_door_handle_1
- removed link link_door_handle_5
- removed link link_door_panel_1
- removed link link_door_panel_5
- removed link link_handle_2
- removed link link_handle_4
- added link link_door_handle_0, mass 0.001; collision box size=0.2 0.05 0.2; visual box size=0.2 0.05 0.2
- added link link_door_handle_4, mass 0.001; collision box size=0.2 0.05 0.2; visual box size=0.2 0.05 0.2
- added link link_door_panel_0, mass 0.001; collision box size=2.0 0.2 2.0; visual box size=2.0 0.2 2.0
- added link link_door_panel_4, mass 0.001; collision box size=4.0 0.2 2.0; visual box size=4.0 0.2 2.0
- added link link_handle_knob_1, mass 0.001; collision box size=0.05 0.05 0.2; visual box size=0.05 0.05 0.2
- added link link_handle_knob_2, mass 0.001; collision box size=0.05 0.05 0.2; visual box size=0.05 0.05 0.2
- added link link_handle_knob_3, mass 0.001; collision box size=0.05 0.05 0.2; visual box size=0.05 0.05 0.2
- added link link_handle_shaft_1, mass 0.001; collision box size=0.2 0.2 1.0; visual box size=0.2 0.2 1.0
- added link link_handle_shaft_2, mass 0.001; collision cylinder length=1.0 radius=0.1; visual cylinder length=1.0 radius=0.1
- added link link_handle_shaft_3, mass 0.001; collision box size=0.2 0.2 1.0; visual box size=0.2 0.2 1.0
- added link link_hinge_0, mass 0.001; collision cylinder length=2.1 radius=0.05; visual cylinder length=2.1 radius=0.05
- added link link_hinge_2, mass 0.001; collision cylinder length=1.1 radius=0.05; visual cylinder length=1.1 radius=0.05
- added link link_hinge_4, mass 0.001; collision cylinder length=2.1 radius=0.05; visual cylinder length=2.1 radius=0.05
Joints:
- removed joint link_door_handle_1
- removed joint link_door_handle_5
- removed joint link_door_panel_1
- removed joint link_door_panel_5
- removed joint link_handle_2
- removed joint link_handle_4
- added joint link_door_handle_0: type fixed, parent link_door_0, child link_door_handle_0, origin xyz=1.5 0 1.1 rpy=0 0 0
- added joint link_door_handle_4: type fixed, parent link_door_4, child link_door_handle_4, origin xyz=3.0 0 1.1 rpy=0 0 0
- added joint link_door_panel_0: type fixed, parent link_door_0, child link_door_panel_0, origin xyz=1.0 0 0 rpy=0 0 0
- added joint link_door_panel_4: type fixed, parent link_door_4, child link_door_panel_4, origin xyz=2.0 0 0 rpy=0 0 0
- added joint link_handle_knob_1: type fixed, parent link_handle_shaft_1, child link_handle_knob_1, origin xyz=0 0 0.6 rpy=0 0 0
- added joint link_handle_knob_2: type fixed, parent link_handle_shaft_2, child link_handle_knob_2, origin xyz=0 0 0.6 rpy=0 0 0
- added joint link_handle_knob_3: type fixed, parent link_handle_shaft_3, child link_handle_knob_3, origin xyz=0 0 0.6 rpy=0 0 0
- added joint link_handle_shaft_1: type fixed, parent link_1, child link_handle_shaft_1, origin xyz=0 -1.0 0 rpy=1.5708 0 0
- added joint link_handle_shaft_2: type fixed, parent link_2, child link_handle_shaft_2, origin xyz=0 1.5 1.0 rpy=0 0 0
- added joint link_handle_shaft_3: type fixed, parent link_3, child link_handle_shaft_3, origin xyz=0 -1.0 0 rpy=1.5708 0 0
- added joint link_hinge_0: type fixed, parent link_door_0, child link_hinge_0, origin xyz=0 0 0 rpy=0 0 0
- added joint link_hinge_2: type fixed, parent link_2, child link_hinge_2, origin xyz=0 0 0 rpy=0 0 0
- added joint link_hinge_4: type fixed, parent link_door_4, child link_hinge_4, origin xyz=0 0 0 rpy=0 0 0

File: puzzles/my_custom/urdf/my_custom.urdf (robot description, URDF)
Before this commit: robot my_custom, 11 links, 10 joints
Links:
- removed link link_door_handle1_2
- removed link link_door_handle2_2
- removed link link_door_handle_1
- removed link link_door_panel_2
- added link link_door_handle1_1, mass 0.001; collision box size=0.05 0.2 0.2; visual box size=0.05 0.2 0.2
- added link link_door_handle2_1, mass 0.001; collision box size=0.05 0.2 0.2; visual box size=0.05 0.2 0.2
- added link link_door_handle_0, mass 0.001; collision box size=0.2 0.05 0.2; visual box size=0.2 0.05 0.2
- added link link_door_panel_0, mass 0.001; collision box size=2.0 0.2 4.0; visual box size=2.0 0.2 4.0
- added link link_handle_knob_2, mass 0.001; collision box size=0.05 0.05 0.2; visual box size=0.05 0.05 0.2
- added link link_handle_knob_3, mass 0.001; collision box size=0.05 0.05 0.2; visual box size=0.05 0.05 0.2
- added link link_handle_knob_4, mass 0.001; collision box size=0.05 0.05 0.2; visual box size=0.05 0.05 0.2
- added link link_handle_shaft_2, mass 0.001; collision cylinder length=1.0 radius=0.1; visual cylinder length=1.0 radius=0.1
- added link link_handle_shaft_3, mass 0.001; collision box size=0.2 0.2 1.0; visual box size=0.2 0.2 1.0
- added link link_handle_shaft_4, mass 0.001; collision cylinder length=1.0 radius=0.1; visual cylinder length=1.0 radius=0.1
- added link link_hinge_0, mass 0.001; collision cylinder length=4.1 radius=0.05; visual cylinder length=4.1 radius=0.05
- added link link_hinge_1, mass 0.001; collision cylinder length=4.1 radius=0.05; visual cylinder length=4.1 radius=0.05
- added link link_hinge_2, mass 0.001; collision cylinder length=2.1 radius=0.05; visual cylinder length=2.1 radius=0.05
- added link link_hinge_4, mass 0.001; collision cylinder length=1.1 radius=0.05; visual cylinder length=1.1 radius=0.05
- link link_2: geometry collision cylinder length=2.0 radius=1.0; visual cylinder length=2.0 radius=1.0
Joints:
- removed joint link_door_handle1_2
- removed joint link_door_handle2_2
- removed joint link_door_handle_1
- removed joint link_door_panel_2
- added joint link_door_handle1_1: type fixed, parent link_door_1, child link_door_handle1_1, origin xyz=1.5 0.2 0 rpy=0 0 0
- added joint link_door_handle2_1: type fixed, parent link_door_1, child link_door_handle2_1, origin xyz=1.5 -0.2 0 rpy=0 0 0
- added joint link_door_handle_0: type fixed, parent link_door_0, child link_door_handle_0, origin xyz=1.5 0 2.1 rpy=0 0 0
- added joint link_door_panel_0: type fixed, parent link_door_0, child link_door_panel_0, origin xyz=1.0 0 0 rpy=0 0 0
- added joint link_handle_knob_2: type fixed, parent link_handle_shaft_2, child link_handle_knob_2, origin xyz=0 0 0.6 rpy=0 0 0
- added joint link_handle_knob_3: type fixed, parent link_handle_shaft_3, child link_handle_knob_3, origin xyz=0 0 0.6 rpy=0 0 0
- added joint link_handle_knob_4: type fixed, parent link_handle_shaft_4, child link_handle_knob_4, origin xyz=0 0 0.6 rpy=0 0 0
- added joint link_handle_shaft_2: type fixed, parent link_2, child link_handle_shaft_2, origin xyz=0 0.75 1.5 rpy=0 0 0
- added joint link_handle_shaft_3: type fixed, parent link_3, child link_handle_shaft_3, origin xyz=0 -1.0 0 rpy=1.5708 0 0
- added joint link_handle_shaft_4: type fixed, parent link_4, child link_handle_shaft_4, origin xyz=0 1.5 1.0 rpy=0 0 0
- added joint link_hinge_0: type fixed, parent link_door_0, child link_hinge_0, origin xyz=0 0 0 rpy=0 0 0
- added joint link_hinge_1: type fixed, parent link_door_1, child link_hinge_1, origin xyz=0 0 0 rpy=0 0 0
- added joint link_hinge_2: type fixed, parent link_2, child link_hinge_2, origin xyz=0 0 0 rpy=0 0 0
- added joint link_hinge_4: type fixed, parent link_4, child link_hinge_4, origin xyz=0 0 0 rpy=0 0 0
- joint link_door_panel_1: parent link_door_0 -> link_door_1

File: puzzles/simple_sliders/urdf/simple_sliders.urdf (robot description, URDF)
Before this commit: robot simple_sliders, 3 links, 2 joints
Links:
- added link link_handle_knob_0, mass 0.001; collision box size=0.05 0.05 0.2; visual box size=0.05 0.05 0.2
- added link link_handle_knob_1, mass 0.001; collision box size=0.05 0.05 0.2; visual box size=0.05 0.05 0.2
- added link link_handle_shaft_0, mass 0.001; collision box size=0.2 0.2 1.0; visual box size=0.2 0.2 1.0
- added link link_handle_shaft_1, mass 0.001; collision box size=0.2 0.2 1.0; visual box size=0.2 0.2 1.0
Joints:
- added joint link_handle_knob_0: type fixed, parent link_handle_shaft_0, child link_handle_knob_0, origin xyz=0 0 0.6 rpy=0 0 0
- added joint link_handle_knob_1: type fixed, parent link_handle_shaft_1, child link_handle_knob_1, origin xyz=0 0 0.6 rpy=0 0 0
- added joint link_handle_shaft_0: type fixed, parent link_0, child link_handle_shaft_0, origin xyz=0 0.6 0 rpy=-1.5708 0 0
- added joint link_handle_shaft_1: type fixed, parent link_1, child link_handle_shaft_1, origin xyz=-0.6 0 0 rpy=0 -1.5708 0

Commit message: feat: create_goal_duplicate() create a semitransparent link to indicate goal position of goal joint

File: puzzles/continuous_space/urdf/continuous_space.urdf (robot description, URDF)
Before this commit: robot continuous_space, 15 links, 14 joints
Links:
- added link goal, mass 0.001; visual box size=3.0 1.0 1.0
- added link link_handle_knob_0.001, mass 0.001; visual box size=0.05 0.05 0.2
- added link link_handle_shaft_0.001, mass 0.001; visual cylinder length=1.0 radius=0.1
- added link link_hinge_0.001, mass 0.001; visual cylinder length=1.1 radius=0.05
- link link_hinge_0: geometry visual cylinder length=1.1 radius=0.05
- link link_hinge_1: geometry visual cylinder length=1.1 radius=0.05
Joints:
- added joint goal: type fixed, parent base_link, child goal, origin xyz=0 0 0.6 rpy=0 0 -2.79785, limit effort=0 velocity=0
- added joint link_handle_knob_0.001: type fixed, parent link_handle_shaft_0.001, child link_handle_knob_0.001, origin xyz=0 0 0.6 rpy=0 0 0
- added joint link_handle_shaft_0.001: type fixed, parent goal, child link_handle_shaft_0.001, origin xyz=1.125 0 1.0 rpy=0 0 0
- added joint link_hinge_0.001: type fixed, parent goal, child link_hinge_0.001, origin xyz=0 0 0 rpy=0 0 0
- joint link_3: limit lower=0 upper=2.2014 effort=0 velocity=0 -> lower=0 upper=3.93321 effort=0 velocity=0; origin xyz=5.40311 -1.16809 0.6 rpy=-1.5708 0 -1.98559 -> xyz=3.51572 -2.56209 0.6 rpy=-1.5708 0 -2.44487

File: puzzles/grid_world/urdf/grid_world.urdf (robot description, URDF)
Before this commit: robot grid_world, 15 links, 14 joints
Links:
- added link goal, mass 0.001; visual box size=2.9 0.9 0.9
- added link link_handle_knob_0.001, mass 0.001; visual box size=0.05 0.05 0.2
- added link link_handle_shaft_0.001, mass 0.001; visual cylinder length=1.0 radius=0.1
- added link link_hinge_0.001, mass 0.001; visual cylinder length=1.0 radius=0.05
- link link_hinge_0: geometry visual cylinder length=1.0 radius=0.05
- link link_hinge_1: geometry visual cylinder length=1.0 radius=0.05
Joints:
- added joint goal: type fixed, parent base_link, child goal, origin xyz=-0.5 0.5 0.55 rpy=0 0 1.5707, limit effort=0 velocity=0
- added joint link_handle_knob_0.001: type fixed, parent link_handle_shaft_0.001, child link_handle_knob_0.001, origin xyz=0 0 0.6 rpy=0 0 0
- added joint link_handle_shaft_0.001: type fixed, parent goal, child link_handle_shaft_0.001, origin xyz=1.0875 0 0.95 rpy=0 0 0
- added joint link_hinge_0.001: type fixed, parent goal, child link_hinge_0.001, origin xyz=0 0 0 rpy=0 0 0

File: puzzles/lockbox2017/urdf/lockbox2017.urdf (robot description, URDF)
Before this commit: robot lockbox2017, 19 links, 18 joints
Links:
- removed link link_door_0
- removed link link_door_4
- added link goal, mass 0.001; visual cylinder length=2.0 radius=0.2
- added link link_0, mass 0.001; collision cylinder length=2.0 radius=0.2; visual cylinder length=2.0 radius=0.2
- added link link_4, mass 0.001; collision cylinder length=2.0 radius=0.2; visual cylinder length=2.0 radius=0.2
- added link link_door_handle_0.001, mass 0.001; visual box size=0.2 0.05 0.2
- added link link_door_panel_0.001, mass 0.001; visual box size=2.0 0.2 2.0
- added link link_hinge_0.001, mass 0.001; visual cylinder length=2.1 radius=0.05
- link link_hinge_0: geometry visual cylinder length=2.1 radius=0.05
- link link_hinge_2: geometry visual cylinder length=1.1 radius=0.05
- link link_hinge_4: geometry visual cylinder length=2.1 radius=0.05
Joints:
- removed joint link_door_0
- removed joint link_door_4
- added joint goal: type fixed, parent base_link, child goal, origin xyz=-6.0 -1.0 1.1 rpy=0 0 1.5708, limit effort=0 velocity=0
- added joint link_0: type revolute, parent base_link, child link_0, origin xyz=-6.0 -1.0 1.1 rpy=0 0 0, axis 0 0 1.0, limit lower=0 upper=1.5708 effort=0 velocity=0
- added joint link_4: type revolute, parent base_link, child link_4, origin xyz=-2.0 4.0 1.1 rpy=0 0 0, axis 0 0 1.0, limit lower=0 upper=1.5708 effort=0 velocity=0
- added joint link_door_handle_0.001: type fixed, parent goal, child link_door_handle_0.001, origin xyz=1.5 0 1.1 rpy=0 0 0
- added joint link_door_panel_0.001: type fixed, parent goal, child link_door_panel_0.001, origin xyz=1.0 0 0 rpy=0 0 0
- added joint link_hinge_0.001: type fixed, parent goal, child link_hinge_0.001, origin xyz=0 0 0 rpy=0 0 0
- joint link_door_handle_0: parent link_door_0 -> link_0
- joint link_door_handle_4: parent link_door_4 -> link_4
- joint link_door_panel_0: parent link_door_0 -> link_0
- joint link_door_panel_4: parent link_door_4 -> link_4
- joint link_hinge_0: parent link_door_0 -> link_0
- joint link_hinge_4: parent link_door_4 -> link_4

File: puzzles/lockbox_random/urdf/lockbox_random.urdf (robot description, URDF)
Before this commit: robot lockbox_random, 18 links, 17 joints
Links:
- added link goal, mass 0.001; visual box size=1.0 0.6 1.9
- added link link_handle_knob_0.001, mass 0.001; visual box size=0.05 0.05 0.2
- added link link_handle_shaft_0.001, mass 0.001; visual box size=0.2 0.2 1.0
- link link_hinge_1: geometry visual cylinder length=1.1 radius=0.05
- link link_hinge_3: geometry visual cylinder length=1.1 radius=0.05
Joints:
- added joint goal: type fixed, parent base_link, child goal, origin xyz=-1.0 0.5 0.6 rpy=0 1.5708 0, limit effort=0 velocity=0
- added joint link_handle_knob_0.001: type fixed, parent link_handle_shaft_0.001, child link_handle_knob_0.001, origin xyz=0 0 0.6 rpy=0 0 0
- added joint link_handle_shaft_0.001: type fixed, parent goal, child link_handle_shaft_0.001, origin xyz=-1.0 0 0 rpy=0 -1.5708 0

File: puzzles/simple_sliders/urdf/simple_sliders.urdf (robot description, URDF)
Before this commit: robot simple_sliders, 7 links, 6 joints
Links:
- added link goal, mass 0.001; visual box size=0.2 0.2 1.6
- added link link_handle_knob_0.001, mass 0.001; visual box size=0.05 0.05 0.2
- added link link_handle_shaft_0.001, mass 0.001; visual box size=0.2 0.2 1.0
Joints:
- added joint goal: type fixed, parent base_link, child goal, origin xyz=0 -1.0 0.2 rpy=1.5708 0 0, limit effort=0 velocity=0
- added joint link_handle_knob_0.001: type fixed, parent link_handle_shaft_0.001, child link_handle_knob_0.001, origin xyz=0 0 0.6 rpy=0 0 0
- added joint link_handle_shaft_0.001: type fixed, parent goal, child link_handle_shaft_0.001, origin xyz=0 0.6 0 rpy=-1.5708 0 0

Commit message: feat: allow both absolute and relative paths

File: puzzles/continuous_space/urdf/continuous_space.urdf (robot description, URDF)
Before this commit: robot continuous_space, 19 links, 18 joints
Joints:
- joint link_3: limit lower=0 upper=3.93321 effort=0 velocity=0 -> lower=0 upper=2.2014 effort=0 velocity=0; origin xyz=3.51572 -2.56209 0.6 rpy=-1.5708 0 -2.44487 -> xyz=5.40311 -1.16809 0.6 rpy=-1.5708 0 -1.98559
