Commit message: feat: name links automatically according to pattern: link_x_joint_y

File: puzzles/continuous_space/urdf/continuous_space.urdf (robot description, URDF)
Before this commit: robot continuous_space, 19 links, 18 joints
Links:
- removed link link_0
- removed link link_1
- removed link link_2
- removed link link_3
- removed link link_handle_knob_0
- removed link link_handle_knob_0.001
- removed link link_handle_knob_1
- removed link link_handle_knob_2
- removed link link_handle_knob_3
- removed link link_handle_shaft_0
- removed link link_handle_shaft_0.001
- removed link link_handle_shaft_1
- removed link link_handle_shaft_2
- removed link link_handle_shaft_3
- removed link link_hinge_0
- removed link link_hinge_0.001
- removed link link_hinge_1
- added link link_0_fixed_joint_1_handle_shaft, mass 0.001; collision cylinder length=1.0 radius=0.1; visual cylinder length=1.0 radius=0.1
- added link link_0_fixed_joint_1_handle_shaft.001, mass 0.001; visual cylinder length=1.0 radius=0.1
- added link link_0_fixed_joint_2_handle_knob, mass 0.001; collision box size=0.05 0.05 0.2; visual box size=0.05 0.05 0.2
- added link link_0_fixed_joint_2_handle_knob.001, mass 0.001; visual box size=0.05 0.05 0.2
- added link link_0_fixed_joint_3_hinge, mass 0.001; visual cylinder length=1.1 radius=0.05
- added link link_0_fixed_joint_3_hinge.001, mass 0.001; visual cylinder length=1.1 radius=0.05
- added link link_0_joint_0, mass 0.001; collision box size=3.0 1.0 1.0; visual box size=3.0 1.0 1.0
- added link link_1_fixed_joint_1_handle_shaft, mass 0.001; collision cylinder length=1.0 radius=0.1; visual cylinder length=1.0 radius=0.1
- added link link_1_fixed_joint_2_handle_knob, mass 0.001; collision box size=0.05 0.05 0.2; visual box size=0.05 0.05 0.2
- added link link_1_fixed_joint_3_hinge, mass 0.001; visual cylinder length=1.1 radius=0.05
- added link link_1_joint_0, mass 0.001; collision box size=3.0 1.0 1.0; visual box size=3.0 1.0 1.0
- added link link_2_fixed_joint_1_handle_shaft, mass 0.001; collision box size=0.2 0.2 1.0; visual box size=0.2 0.2 1.0
- added link link_2_fixed_joint_2_handle_knob, mass 0.001; collision box size=0.05 0.05 0.2; visual box size=0.05 0.05 0.2
- added link link_2_joint_0, mass 0.001; collision box size=1.0 1.0 2.0; visual box size=1.0 1.0 2.0
- added link link_3_fixed_joint_1_handle_shaft, mass 0.001; collision box size=0.2 0.2 1.0; visual box size=0.2 0.2 1.0
- added link link_3_fixed_joint_2_handle_knob, mass 0.001; collision box size=0.05 0.05 0.2; visual box size=0.05 0.05 0.2
- added link link_3_joint_0, mass 0.001; collision box size=1.0 1.0 2.0; visual box size=1.0 1.0 2.0
Joints:
- removed joint link_0
- removed joint link_1
- removed joint link_2
- removed joint link_3
- removed joint link_handle_knob_0
- removed joint link_handle_knob_0.001
- removed joint link_handle_knob_1
- removed joint link_handle_knob_2
- removed joint link_handle_knob_3
- removed joint link_handle_shaft_0
- removed joint link_handle_shaft_0.001
- removed joint link_handle_shaft_1
- removed joint link_handle_shaft_2
- removed joint link_handle_shaft_3
- removed joint link_hinge_0
- removed joint link_hinge_0.001
- removed joint link_hinge_1
- added joint link_0_fixed_joint_1_handle_shaft: type fixed, parent link_0_joint_0, child link_0_fixed_joint_1_handle_shaft, origin xyz=1.125 0 1.0 rpy=0 0 0
- added joint link_0_fixed_joint_1_handle_shaft.001: type fixed, parent goal, child link_0_fixed_joint_1_handle_shaft.001, origin xyz=1.125 0 1.0 rpy=0 0 0
- added joint link_0_fixed_joint_2_handle_knob: type fixed, parent link_0_fixed_joint_1_handle_shaft, child link_0_fixed_joint_2_handle_knob, origin xyz=0 0 0.6 rpy=0 0 0
- added joint link_0_fixed_joint_2_handle_knob.001: type fixed, parent link_0_fixed_joint_1_handle_shaft.001, child link_0_fixed_joint_2_handle_knob.001, origin xyz=0 0 0.6 rpy=0 0 0
- added joint link_0_fixed_joint_3_hinge: type fixed, parent link_0_joint_0, child link_0_fixed_joint_3_hinge, origin xyz=0 0 0 rpy=0 0 0
- added joint link_0_fixed_joint_3_hinge.001: type fixed, parent goal, child link_0_fixed_joint_3_hinge.001, origin xyz=0 0 0 rpy=0 0 0
- added joint link_0_joint_0: type revolute, parent base_link, child link_0_joint_0, origin xyz=0 0 0.6 rpy=0 0 -0.97753, axis 0 0 1.0, limit lower=-1.82033 upper=0 effort=0 velocity=0
- added joint link_1_fixed_joint_1_handle_shaft: type fixed, parent link_1_joint_0, child link_1_fixed_joint_1_handle_shaft, origin xyz=1.125 0 1.0 rpy=0 0 0
- added joint link_1_fixed_joint_2_handle_knob: type fixed, parent link_1_fixed_joint_1_handle_shaft, child link_1_fixed_joint_2_handle_knob, origin xyz=0 0 0.6 rpy=0 0 0
- added joint link_1_fixed_joint_3_hinge: type fixed, parent link_1_joint_0, child link_1_fixed_joint_3_hinge, origin xyz=0 0 0 rpy=0 0 0
- added joint link_1_joint_0: type revolute, parent base_link, child link_1_joint_0, origin xyz=1.89729 1.60702 0.6 rpy=0 0 -2.61769, axis 0 0 1.0, limit lower=0 upper=1.58552 effort=0 velocity=0
- added joint link_2_fixed_joint_1_handle_shaft: type fixed, parent link_2_joint_0, child link_2_fixed_joint_1_handle_shaft, origin xyz=0 -1.0 0 rpy=1.5708 0 0
- added joint link_2_fixed_joint_2_handle_knob: type fixed, parent link_2_fixed_joint_1_handle_shaft, child link_2_fixed_joint_2_handle_knob, origin xyz=0 0 0.6 rpy=0 0 0
- added joint link_2_joint_0: type prismatic, parent base_link, child link_2_joint_0, origin xyz=2.7436 -0.22319 0.6 rpy=-1.5708 0 -2.39786, axis 0 0 1.0, limit lower=0 upper=3.81949 effort=0 velocity=0
- added joint link_3_fixed_joint_1_handle_shaft: type fixed, parent link_3_joint_0, child link_3_fixed_joint_1_handle_shaft, origin xyz=0 -1.0 0 rpy=1.5708 0 0
- added joint link_3_fixed_joint_2_handle_knob: type fixed, parent link_3_fixed_joint_1_handle_shaft, child link_3_fixed_joint_2_handle_knob, origin xyz=0 0 0.6 rpy=0 0 0
- added joint link_3_joint_0: type prismatic, parent base_link, child link_3_joint_0, origin xyz=3.51572 -2.56209 0.6 rpy=-1.5708 0 -2.44487, axis 0 0 1.0, limit lower=0 upper=3.93321 effort=0 velocity=0

File: puzzles/grid_world/urdf/grid_world.urdf (robot description, URDF)
Before this commit: robot grid_world, 19 links, 18 joints
Links:
- removed link link_0
- removed link link_1
- removed link link_2
- removed link link_3
- removed link link_handle_knob_0
- removed link link_handle_knob_0.001
- removed link link_handle_knob_1
- removed link link_handle_knob_2
- removed link link_handle_knob_3
- removed link link_handle_shaft_0
- removed link link_handle_shaft_0.001
- removed link link_handle_shaft_1
- removed link link_handle_shaft_2
- removed link link_handle_shaft_3
- removed link link_hinge_0
- removed link link_hinge_0.001
- removed link link_hinge_1
- added link link_0_fixed_joint_1_handle_shaft, mass 0.001; collision cylinder length=1.0 radius=0.1; visual cylinder length=1.0 radius=0.1
- added link link_0_fixed_joint_1_handle_shaft.001, mass 0.001; visual cylinder length=1.0 radius=0.1
- added link link_0_fixed_joint_2_handle_knob, mass 0.001; collision box size=0.05 0.05 0.2; visual box size=0.05 0.05 0.2
- added link link_0_fixed_joint_2_handle_knob.001, mass 0.001; visual box size=0.05 0.05 0.2
- added link link_0_fixed_joint_3_hinge, mass 0.001; visual cylinder length=1.0 radius=0.05
- added link link_0_fixed_joint_3_hinge.001, mass 0.001; visual cylinder length=1.0 radius=0.05
- added link link_0_joint_0, mass 0.001; collision box size=2.9 0.9 0.9; visual box size=2.9 0.9 0.9
- added link link_1_fixed_joint_1_handle_shaft, mass 0.001; collision cylinder length=1.0 radius=0.1; visual cylinder length=1.0 radius=0.1
- added link link_1_fixed_joint_2_handle_knob, mass 0.001; collision box size=0.05 0.05 0.2; visual box size=0.05 0.05 0.2
- added link link_1_fixed_joint_3_hinge, mass 0.001; visual cylinder length=1.0 radius=0.05
- added link link_1_joint_0, mass 0.001; collision box size=2.9 0.9 0.9; visual box size=2.9 0.9 0.9
- added link link_2_fixed_joint_1_handle_shaft, mass 0.001; collision box size=0.2 0.2 1.0; visual box size=0.2 0.2 1.0
- added link link_2_fixed_joint_2_handle_knob, mass 0.001; collision box size=0.05 0.05 0.2; visual box size=0.05 0.05 0.2
- added link link_2_joint_0, mass 0.001; collision box size=0.9 0.9 1.9; visual box size=0.9 0.9 1.9
- added link link_3_fixed_joint_1_handle_shaft, mass 0.001; collision box size=0.2 0.2 1.0; visual box size=0.2 0.2 1.0
- added link link_3_fixed_joint_2_handle_knob, mass 0.001; collision box size=0.05 0.05 0.2; visual box size=0.05 0.05 0.2
- added link link_3_joint_0, mass 0.001; collision box size=0.9 0.9 1.9; visual box size=0.9 0.9 1.9
Joints:
- removed joint link_0
- removed joint link_1
- removed joint link_2
- removed joint link_3
- removed joint link_handle_knob_0
- removed joint link_handle_knob_0.001
- removed joint link_handle_knob_1
- removed joint link_handle_knob_2
- removed joint link_handle_knob_3
- removed joint link_handle_shaft_0
- removed joint link_handle_shaft_0.001
- removed joint link_handle_shaft_1
- removed joint link_handle_shaft_2
- removed joint link_handle_shaft_3
- removed joint link_hinge_0
- removed joint link_hinge_0.001
- removed joint link_hinge_1
- added joint link_0_fixed_joint_1_handle_shaft: type fixed, parent link_0_joint_0, child link_0_fixed_joint_1_handle_shaft, origin xyz=1.0875 0 0.95 rpy=0 0 0
- added joint link_0_fixed_joint_1_handle_shaft.001: type fixed, parent goal, child link_0_fixed_joint_1_handle_shaft.001, origin xyz=1.0875 0 0.95 rpy=0 0 0
- added joint link_0_fixed_joint_2_handle_knob: type fixed, parent link_0_fixed_joint_1_handle_shaft, child link_0_fixed_joint_2_handle_knob, origin xyz=0 0 0.6 rpy=0 0 0
- added joint link_0_fixed_joint_2_handle_knob.001: type fixed, parent link_0_fixed_joint_1_handle_shaft.001, child link_0_fixed_joint_2_handle_knob.001, origin xyz=0 0 0.6 rpy=0 0 0
- added joint link_0_fixed_joint_3_hinge: type fixed, parent link_0_joint_0, child link_0_fixed_joint_3_hinge, origin xyz=0 0 0 rpy=0 0 0
- added joint link_0_fixed_joint_3_hinge.001: type fixed, parent goal, child link_0_fixed_joint_3_hinge.001, origin xyz=0 0 0 rpy=0 0 0
- added joint link_0_joint_0: type revolute, parent base_link, child link_0_joint_0, origin xyz=-0.5 0.5 0.55 rpy=0 0 0, axis 0 0 1.0, limit lower=0 upper=1.5708 effort=0 velocity=0
- added joint link_1_fixed_joint_1_handle_shaft: type fixed, parent link_1_joint_0, child link_1_fixed_joint_1_handle_shaft, origin xyz=1.0875 0 0.95 rpy=0 0 0
- added joint link_1_fixed_joint_2_handle_knob: type fixed, parent link_1_fixed_joint_1_handle_shaft, child link_1_fixed_joint_2_handle_knob, origin xyz=0 0 0.6 rpy=0 0 0
- added joint link_1_fixed_joint_3_hinge: type fixed, parent link_1_joint_0, child link_1_fixed_joint_3_hinge, origin xyz=0 0 0 rpy=0 0 0
- added joint link_1_joint_0: type revolute, parent base_link, child link_1_joint_0, origin xyz=-2.5 -0.5 0.55 rpy=0 0 0, axis 0 0 1.0, limit lower=-1.5708 upper=0 effort=0 velocity=0
- added joint link_2_fixed_joint_1_handle_shaft: type fixed, parent link_2_joint_0, child link_2_fixed_joint_1_handle_shaft, origin xyz=-0.95 0 0 rpy=0 -1.5708 0
- added joint link_2_fixed_joint_2_handle_knob: type fixed, parent link_2_fixed_joint_1_handle_shaft, child link_2_fixed_joint_2_handle_knob, origin xyz=0 0 0.6 rpy=0 0 0
- added joint link_2_joint_0: type prismatic, parent base_link, child link_2_joint_0, origin xyz=1.0 1.5 0.55 rpy=0 1.5708 0, axis 0 0 1.0, limit lower=0 upper=1.0 effort=0 velocity=0
- added joint link_3_fixed_joint_1_handle_shaft: type fixed, parent link_3_joint_0, child link_3_fixed_joint_1_handle_shaft, origin xyz=0 0.95 0 rpy=-1.5708 0 0
- added joint link_3_fixed_joint_2_handle_knob: type fixed, parent link_3_fixed_joint_1_handle_shaft, child link_3_fixed_joint_2_handle_knob, origin xyz=0 0 0.6 rpy=0 0 0
- added joint link_3_joint_0: type prismatic, parent base_link, child link_3_joint_0, origin xyz=-1.5 -2.0 0.55 rpy=1.5708 0 0, axis 0 0 1.0, limit lower=0 upper=1.0 effort=0 velocity=0

File: puzzles/lockbox2017/urdf/lockbox2017.urdf (robot description, URDF)
Before this commit: robot lockbox2017, 23 links, 22 joints
Links:
- removed link link_0
- removed link link_1
- removed link link_2
- removed link link_3
- removed link link_4
- removed link link_door_handle_0
- removed link link_door_handle_0.001
- removed link link_door_handle_4
- removed link link_door_panel_0
- removed link link_door_panel_0.001
- removed link link_door_panel_4
- removed link link_handle_knob_1
- removed link link_handle_knob_2
- removed link link_handle_knob_3
- removed link link_handle_shaft_1
- removed link link_handle_shaft_2
- removed link link_handle_shaft_3
- removed link link_hinge_0
- removed link link_hinge_0.001
- removed link link_hinge_2
- removed link link_hinge_4
- added link link_0_fixed_joint_1_hinge, mass 0.001; visual cylinder length=2.1 radius=0.05
- added link link_0_fixed_joint_1_hinge.001, mass 0.001; visual cylinder length=2.1 radius=0.05
- added link link_0_fixed_joint_2_door_panel, mass 0.001; collision box size=2.0 0.2 2.0; visual box size=2.0 0.2 2.0
- added link link_0_fixed_joint_2_door_panel.001, mass 0.001; visual box size=2.0 0.2 2.0
- added link link_0_fixed_joint_3_door_handle, mass 0.001; collision box size=0.2 0.05 0.2; visual box size=0.2 0.05 0.2
- added link link_0_fixed_joint_3_door_handle.001, mass 0.001; visual box size=0.2 0.05 0.2
- added link link_0_joint_0, mass 0.001; collision cylinder length=2.0 radius=0.2; visual cylinder length=2.0 radius=0.2
- added link link_1_fixed_joint_1_handle_shaft, mass 0.001; collision box size=0.2 0.2 1.0; visual box size=0.2 0.2 1.0
- added link link_1_fixed_joint_2_handle_knob, mass 0.001; collision box size=0.05 0.05 0.2; visual box size=0.05 0.05 0.2
- added link link_1_joint_0, mass 0.001; collision box size=0.8 1.0 3.6; visual box size=0.8 1.0 3.6
- added link link_2_fixed_joint_1_handle_shaft, mass 0.001; collision cylinder length=1.0 radius=0.1; visual cylinder length=1.0 radius=0.1
- added link link_2_fixed_joint_2_handle_knob, mass 0.001; collision box size=0.05 0.05 0.2; visual box size=0.05 0.05 0.2
- added link link_2_fixed_joint_3_hinge, mass 0.001; visual cylinder length=1.1 radius=0.05
- added link link_2_joint_0, mass 0.001; collision mesh filename=file:///home/userone/ba/puzzle-generator/puzzles/lockbox201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 scale=1.0 1.0 1.0; visual mesh filename=file:///home/userone/ba/puzzle-generator/puzzles/lockbox201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 scale=1.0 1.0 1.0
- added link link_3_fixed_joint_1_handle_shaft, mass 0.001; collision box size=0.2 0.2 1.0; visual box size=0.2 0.2 1.0
- added link link_3_fixed_joint_2_handle_knob, mass 0.001; collision box size=0.05 0.05 0.2; visual box size=0.05 0.05 0.2
- added link link_3_joint_0, mass 0.001; collision box size=0.8 1.0 3.6; visual box size=0.8 1.0 3.6
- added link link_4_fixed_joint_1_hinge, mass 0.001; visual cylinder length=2.1 radius=0.05
- added link link_4_fixed_joint_2_door_panel, mass 0.001; collision box size=4.0 0.2 2.0; visual box size=4.0 0.2 2.0
- added link link_4_fixed_joint_3_door_handle, mass 0.001; collision box size=0.2 0.05 0.2; visual box size=0.2 0.05 0.2
- added link link_4_joint_0, mass 0.001; collision cylinder length=2.0 radius=0.2; visual cylinder length=2.0 radius=0.2
Joints:
- removed joint link_0
- removed joint link_1
- removed joint link_2
- removed joint link_3
- removed joint link_4
- removed joint link_door_handle_0
- removed joint link_door_handle_0.001
- removed joint link_door_handle_4
- removed joint link_door_panel_0
- removed joint link_door_panel_0.001
- removed joint link_door_panel_4
- removed joint link_handle_knob_1
- removed joint link_handle_knob_2
- removed joint link_handle_knob_3
- removed joint link_handle_shaft_1
- removed joint link_handle_shaft_2
- removed joint link_handle_shaft_3
- removed joint link_hinge_0
- removed joint link_hinge_0.001
- removed joint link_hinge_2
- removed joint link_hinge_4
- added joint link_0_fixed_joint_1_hinge: type fixed, parent link_0_joint_0, child link_0_fixed_joint_1_hinge, origin xyz=0 0 0 rpy=0 0 0
- added joint link_0_fixed_joint_1_hinge.001: type fixed, parent goal, child link_0_fixed_joint_1_hinge.001, origin xyz=0 0 0 rpy=0 0 0
- added joint link_0_fixed_joint_2_door_panel: type fixed, parent link_0_joint_0, child link_0_fixed_joint_2_door_panel, origin xyz=1.0 0 0 rpy=0 0 0
- added joint link_0_fixed_joint_2_door_panel.001: type fixed, parent goal, child link_0_fixed_joint_2_door_panel.001, origin xyz=1.0 0 0 rpy=0 0 0
- added joint link_0_fixed_joint_3_door_handle: type fixed, parent link_0_joint_0, child link_0_fixed_joint_3_door_handle, origin xyz=1.5 0 1.1 rpy=0 0 0
- added joint link_0_fixed_joint_3_door_handle.001: type fixed, parent goal, child link_0_fixed_joint_3_door_handle.001, origin xyz=1.5 0 1.1 rpy=0 0 0
- added joint link_0_joint_0: type revolute, parent base_link, child link_0_joint_0, origin xyz=-6.0 -1.0 1.1 rpy=0 0 0, axis 0 0 1.0, limit lower=0 upper=1.5708 effort=0 velocity=0
- added joint link_1_fixed_joint_1_handle_shaft: type fixed, parent link_1_joint_0, child link_1_fixed_joint_1_handle_shaft, origin xyz=0 -1.0 0 rpy=1.5708 0 0
- added joint link_1_fixed_joint_2_handle_knob: type fixed, parent link_1_fixed_joint_1_handle_shaft, child link_1_fixed_joint_2_handle_knob, origin xyz=0 0 0.6 rpy=0 0 0
- added joint link_1_joint_0: type prismatic, parent base_link, child link_1_joint_0, origin xyz=-4.0 0 0.6 rpy=-1.5708 0 -1.5708, axis 0 0 1.0, limit lower=0 upper=2.0 effort=0 velocity=0
- added joint link_2_fixed_joint_1_handle_shaft: type fixed, parent link_2_joint_0, child link_2_fixed_joint_1_handle_shaft, origin xyz=0 1.5 1.0 rpy=0 0 0
- added joint link_2_fixed_joint_2_handle_knob: type fixed, parent link_2_fixed_joint_1_handle_shaft, child link_2_fixed_joint_2_handle_knob, origin xyz=0 0 0.6 rpy=0 0 0
- added joint link_2_fixed_joint_3_hinge: type fixed, parent link_2_joint_0, child link_2_fixed_joint_3_hinge, origin xyz=0 0 0 rpy=0 0 0
- added joint link_2_joint_0: type revolute, parent base_link, child link_2_joint_0, origin xyz=0 0 0.6 rpy=0 0 1.5708, axis 0 0 1.0, limit lower=0 upper=1.5708 effort=0 velocity=0
- added joint link_3_fixed_joint_1_handle_shaft: type fixed, parent link_3_joint_0, child link_3_fixed_joint_1_handle_shaft, origin xyz=0 -1.0 0 rpy=1.5708 0 0
- added joint link_3_fixed_joint_2_handle_knob: type fixed, parent link_3_fixed_joint_1_handle_shaft, child link_3_fixed_joint_2_handle_knob, origin xyz=0 0 0.6 rpy=0 0 0
- added joint link_3_joint_0: type prismatic, parent base_link, child link_3_joint_0, origin xyz=0 2.0 0.6 rpy=-1.5708 0 0, axis 0 0 1.0, limit lower=0 upper=2.0 effort=0 velocity=0
- added joint link_4_fixed_joint_1_hinge: type fixed, parent link_4_joint_0, child link_4_fixed_joint_1_hinge, origin xyz=0 0 0 rpy=0 0 0
- added joint link_4_fixed_joint_2_door_panel: type fixed, parent link_4_joint_0, child link_4_fixed_joint_2_door_panel, origin xyz=2.0 0 0 rpy=0 0 0
- added joint link_4_fixed_joint_3_door_handle: type fixed, parent link_4_joint_0, child link_4_fixed_joint_3_door_handle, origin xyz=3.0 0 1.1 rpy=0 0 0
- added joint link_4_joint_0: type revolute, parent base_link, child link_4_joint_0, origin xyz=-2.0 4.0 1.1 rpy=0 0 0, axis 0 0 1.0, limit lower=0 upper=1.5708 effort=0 velocity=0
