Commit message: feat: name links automatically according to pattern: link_x_joint_y

File: puzzles/lockbox_random/urdf/lockbox_random.urdf (robot description, URDF)
Before this commit: robot lockbox_random, 21 links, 20 joints
Links:
- removed link link_0
- removed link link_1
- removed link link_2
- removed link link_3
- removed link link_4
- removed link link_handle_knob_0
- removed link link_handle_knob_0.001
- removed link link_handle_knob_1
- removed link link_handle_knob_2
- removed link link_handle_knob_3
- removed link link_handle_knob_4
- removed link link_handle_shaft_0
- removed link link_handle_shaft_0.001
- removed link link_handle_shaft_1
- removed link link_handle_shaft_2
- removed link link_handle_shaft_3
- removed link link_handle_shaft_4
- removed link link_hinge_1
- removed link link_hinge_3
- added link link_0_fixed_joint_1_handle_shaft, mass 0.001; collision box size=0.2 0.2 1.0; visual box size=0.2 0.2 1.0
- added link link_0_fixed_joint_1_handle_shaft.001, mass 0.001; visual box size=0.2 0.2 1.0
- added link link_0_fixed_joint_2_handle_knob, mass 0.001; collision box size=0.05 0.05 0.2; visual box size=0.05 0.05 0.2
- added link link_0_fixed_joint_2_handle_knob.001, mass 0.001; visual box size=0.05 0.05 0.2
- added link link_0_joint_0, mass 0.001; collision box size=1.0 0.6 1.9; visual box size=1.0 0.6 1.9
- added link link_1_fixed_joint_1_handle_shaft, mass 0.001; collision cylinder length=1.0 radius=0.1; visual cylinder length=1.0 radius=0.1
- added link link_1_fixed_joint_2_handle_knob, mass 0.001; collision box size=0.05 0.05 0.2; visual box size=0.05 0.05 0.2
- added link link_1_fixed_joint_3_hinge, mass 0.001; visual cylinder length=1.1 radius=0.05
- added link link_1_joint_0, mass 0.001; collision mesh filename=file:///home/userone/ba/puzzle-generator/puzzles/lockbox_ra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 scale=1.0 1.0 1.0; visual mesh filename=file:///home/userone/ba/puzzle-generator/puzzles/lockbox_ra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 scale=1.0 1.0 1.0
- added link link_2_fixed_joint_1_handle_shaft, mass 0.001; collision box size=0.2 0.2 1.0; visual box size=0.2 0.2 1.0
- added link link_2_fixed_joint_2_handle_knob, mass 0.001; collision box size=0.05 0.05 0.2; visual box size=0.05 0.05 0.2
- added link link_2_joint_0, mass 0.001; collision box size=1.0 0.6 1.9; visual box size=1.0 0.6 1.9
- added link link_3_fixed_joint_1_handle_shaft, mass 0.001; collision cylinder length=1.0 radius=0.1; visual cylinder length=1.0 radius=0.1
- added link link_3_fixed_joint_2_handle_knob, mass 0.001; collision box size=0.05 0.05 0.2; visual box size=0.05 0.05 0.2
- added link link_3_fixed_joint_3_hinge, mass 0.001; visual cylinder length=1.1 radius=0.05
- added link link_3_joint_0, mass 0.001; collision mesh filename=file:///home/userone/ba/puzzle-generator/puzzles/lockbox_ra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 scale=1.0 1.0 1.0; visual mesh filename=file:///home/userone/ba/puzzle-generator/puzzles/lockbox_ra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 scale=1.0 1.0 1.0
- added link link_4_fixed_joint_1_handle_shaft, mass 0.001; collision box size=0.2 0.2 1.0; visual box size=0.2 0.2 1.0
- added link link_4_fixed_joint_2_handle_knob, mass 0.001; collision box size=0.05 0.05 0.2; visual box size=0.05 0.05 0.2
- added link link_4_joint_0, mass 0.001; collision box size=1.0 0.6 1.9; visual box size=1.0 0.6 1.9
Joints:
- removed joint link_0
- removed joint link_1
- removed joint link_2
- removed joint link_3
- removed joint link_4
- removed joint link_handle_knob_0
- removed joint link_handle_knob_0.001
- removed joint link_handle_knob_1
- removed joint link_handle_knob_2
- removed joint link_handle_knob_3
- removed joint link_handle_knob_4
- removed joint link_handle_shaft_0
- removed joint link_handle_shaft_0.001
- removed joint link_handle_shaft_1
- removed joint link_handle_shaft_2
- removed joint link_handle_shaft_3
- removed joint link_handle_shaft_4
- removed joint link_hinge_1
- removed joint link_hinge_3
- added joint link_0_fixed_joint_1_handle_shaft: type fixed, parent link_0_joint_0, child link_0_fixed_joint_1_handle_shaft, origin xyz=-1.0 0 0 rpy=0 -1.5708 0
- added joint link_0_fixed_joint_1_handle_shaft.001: type fixed, parent goal, child link_0_fixed_joint_1_handle_shaft.001, origin xyz=-1.0 0 0 rpy=0 -1.5708 0
- added joint link_0_fixed_joint_2_handle_knob: type fixed, parent link_0_fixed_joint_1_handle_shaft, child link_0_fixed_joint_2_handle_knob, origin xyz=0 0 0.6 rpy=0 0 0
- added joint link_0_fixed_joint_2_handle_knob.001: type fixed, parent link_0_fixed_joint_1_handle_shaft.001, child link_0_fixed_joint_2_handle_knob.001, origin xyz=0 0 0.6 rpy=0 0 0
- added joint link_0_joint_0: type prismatic, parent base_link, child link_0_joint_0, origin xyz=-2.0 0.5 0.6 rpy=0 1.5708 0, axis 0 0 1.0, limit lower=0 upper=1.0 effort=0 velocity=0
- added joint link_1_fixed_joint_1_handle_shaft: type fixed, parent link_1_joint_0, child link_1_fixed_joint_1_handle_shaft, origin xyz=0 1.125 1.0 rpy=0 0 0
- added joint link_1_fixed_joint_2_handle_knob: type fixed, parent link_1_fixed_joint_1_handle_shaft, child link_1_fixed_joint_2_handle_knob, origin xyz=0 0 0.6 rpy=0 0 0
- added joint link_1_fixed_joint_3_hinge: type fixed, parent link_1_joint_0, child link_1_fixed_joint_3_hinge, origin xyz=0 0 0 rpy=0 0 0
- added joint link_1_joint_0: type revolute, parent base_link, child link_1_joint_0, origin xyz=0.5 0.5 0.6 rpy=0 0 1.5708, axis 0 0 1.0, limit lower=-3.14159 upper=3.14159 effort=0 velocity=0
- added joint link_2_fixed_joint_1_handle_shaft: type fixed, parent link_2_joint_0, child link_2_fixed_joint_1_handle_shaft, origin xyz=-1.0 0 0 rpy=0 -1.5708 0
- added joint link_2_fixed_joint_2_handle_knob: type fixed, parent link_2_fixed_joint_1_handle_shaft, child link_2_fixed_joint_2_handle_knob, origin xyz=0 0 0.6 rpy=0 0 0
- added joint link_2_joint_0: type prismatic, parent base_link, child link_2_joint_0, origin xyz=0.5 2.0 0.6 rpy=-1.5708 1.5708 0, axis 0 0 1.0, limit lower=0 upper=1.0 effort=0 velocity=0
- added joint link_3_fixed_joint_1_handle_shaft: type fixed, parent link_3_joint_0, child link_3_fixed_joint_1_handle_shaft, origin xyz=0 1.125 1.0 rpy=0 0 0
- added joint link_3_fixed_joint_2_handle_knob: type fixed, parent link_3_fixed_joint_1_handle_shaft, child link_3_fixed_joint_2_handle_knob, origin xyz=0 0 0.6 rpy=0 0 0
- added joint link_3_fixed_joint_3_hinge: type fixed, parent link_3_joint_0, child link_3_fixed_joint_3_hinge, origin xyz=0 0 0 rpy=0 0 0
- added joint link_3_joint_0: type revolute, parent base_link, child link_3_joint_0, origin xyz=0.5 4.5 0.6 rpy=0 0 -3.14159, axis 0 0 1.0, limit lower=-3.14159 upper=3.14159 effort=0 velocity=0
- added joint link_4_fixed_joint_1_handle_shaft: type fixed, parent link_4_joint_0, child link_4_fixed_joint_1_handle_shaft, origin xyz=-1.0 0 0 rpy=0 -1.5708 0
- added joint link_4_fixed_joint_2_handle_knob: type fixed, parent link_4_fixed_joint_1_handle_shaft, child link_4_fixed_joint_2_handle_knob, origin xyz=0 0 0.6 rpy=0 0 0
- added joint link_4_joint_0: type prismatic, parent base_link, child link_4_joint_0, origin xyz=-1.0 4.5 0.6 rpy=3.14159 1.5708 0, axis 0 0 1.0, limit lower=0 upper=1.0 effort=0 velocity=0

File: puzzles/my_custom/urdf/my_custom.urdf (robot description, URDF)
Before this commit: robot my_custom, 21 links, 20 joints
Links:
- removed link link_0
- removed link link_1
- removed link link_2
- removed link link_3
- removed link link_4
- removed link link_door_handle1_1
- removed link link_door_handle2_1
- removed link link_door_handle_0
- removed link link_door_panel_0
- removed link link_door_panel_1
- removed link link_handle_knob_2
- removed link link_handle_knob_3
- removed link link_handle_knob_4
- removed link link_handle_shaft_2
- removed link link_handle_shaft_3
- removed link link_handle_shaft_4
- removed link link_hinge_0
- removed link link_hinge_1
- removed link link_hinge_2
- removed link link_hinge_4
- added link link_0_fixed_joint_3_hinge, mass 0.001; visual cylinder length=1.1 radius=0.05
- added link link_0_joint_0, mass 0.001; visual box size=0 0 0
- added link link_0_joint_1, mass 0.001; visual box size=0 0 0
- added link link_0_joint_2, mass 0.001; collision box size=1.0 1.0 1.0; visual box size=1.0 1.0 1.0
Joints:
- removed joint link_0
- removed joint link_1
- removed joint link_2
- removed joint link_3
- removed joint link_4
- removed joint link_door_handle1_1
- removed joint link_door_handle2_1
- removed joint link_door_handle_0
- removed joint link_door_panel_0
- removed joint link_door_panel_1
- removed joint link_handle_knob_2
- removed joint link_handle_knob_3
- removed joint link_handle_knob_4
- removed joint link_handle_shaft_2
- removed joint link_handle_shaft_3
- removed joint link_handle_shaft_4
- removed joint link_hinge_0
- removed joint link_hinge_1
- removed joint link_hinge_2
- removed joint link_hinge_4
- added joint link_0_fixed_joint_3_hinge: type fixed, parent link_0_joint_2, child link_0_fixed_joint_3_hinge, origin xyz=0 0 0 rpy=0 0 0
- added joint link_0_joint_0: type prismatic, parent base_link, child link_0_joint_0, origin xyz=0 0 0.6 rpy=0 0 0, axis 1.0 0 0, limit lower=0 upper=2.0 effort=0 velocity=0
- added joint link_0_joint_1: type prismatic, parent link_0_joint_0, child link_0_joint_1, origin xyz=0 0 0 rpy=0 0 0, axis 0 1.0 0, limit lower=0 upper=2.0 effort=0 velocity=0
- added joint link_0_joint_2: type revolute, parent link_0_joint_1, child link_0_joint_2, origin xyz=0 0 0 rpy=0 0 0, axis 0 0 1.0, limit lower=0 upper=2.0 effort=0 velocity=0

File: puzzles/simple_sliders/urdf/simple_sliders.urdf (robot description, URDF)
Before this commit: robot simple_sliders, 10 links, 9 joints
Links:
- removed link link_0
- removed link link_1
- removed link link_handle_knob_0
- removed link link_handle_knob_0.001
- removed link link_handle_knob_1
- removed link link_handle_shaft_0
- removed link link_handle_shaft_0.001
- removed link link_handle_shaft_1
- added link link_0_fixed_joint_1_handle_shaft, mass 0.001; collision box size=0.2 0.2 1.0; visual box size=0.2 0.2 1.0
- added link link_0_fixed_joint_1_handle_shaft.001, mass 0.001; visual box size=0.2 0.2 1.0
- added link link_0_fixed_joint_2_handle_knob, mass 0.001; collision box size=0.05 0.05 0.2; visual box size=0.05 0.05 0.2
- added link link_0_fixed_joint_2_handle_knob.001, mass 0.001; visual box size=0.05 0.05 0.2
- added link link_0_joint_0, mass 0.001; collision box size=0.2 0.2 1.6; visual box size=0.2 0.2 1.6
- added link link_1_fixed_joint_1_handle_shaft, mass 0.001; collision box size=0.2 0.2 1.0; visual box size=0.2 0.2 1.0
- added link link_1_fixed_joint_2_handle_knob, mass 0.001; collision box size=0.05 0.05 0.2; visual box size=0.05 0.05 0.2
- added link link_1_joint_0, mass 0.001; collision box size=0.2 0.2 1.6; visual box size=0.2 0.2 1.6
Joints:
- removed joint link_0
- removed joint link_1
- removed joint link_handle_knob_0
- removed joint link_handle_knob_0.001
- removed joint link_handle_knob_1
- removed joint link_handle_shaft_0
- removed joint link_handle_shaft_0.001
- removed joint link_handle_shaft_1
- added joint link_0_fixed_joint_1_handle_shaft: type fixed, parent link_0_joint_0, child link_0_fixed_joint_1_handle_shaft, origin xyz=0 0.6 0 rpy=-1.5708 0 0
- added joint link_0_fixed_joint_1_handle_shaft.001: type fixed, parent goal, child link_0_fixed_joint_1_handle_shaft.001, origin xyz=0 0.6 0 rpy=-1.5708 0 0
- added joint link_0_fixed_joint_2_handle_knob: type fixed, parent link_0_fixed_joint_1_handle_shaft, child link_0_fixed_joint_2_handle_knob, origin xyz=0 0 0.6 rpy=0 0 0
- added joint link_0_fixed_joint_2_handle_knob.001: type fixed, parent link_0_fixed_joint_1_handle_shaft.001, child link_0_fixed_joint_2_handle_knob.001, origin xyz=0 0 0.6 rpy=0 0 0
- added joint link_0_joint_0: type prismatic, parent base_link, child link_0_joint_0, origin xyz=0 0 0.2 rpy=1.5708 0 0, axis 0 0 1.0, limit lower=0 upper=1.0 effort=0 velocity=0
- added joint link_1_fixed_joint_1_handle_shaft: type fixed, parent link_1_joint_0, child link_1_fixed_joint_1_handle_shaft, origin xyz=-0.6 0 0 rpy=0 -1.5708 0
- added joint link_1_fixed_joint_2_handle_knob: type fixed, parent link_1_fixed_joint_1_handle_shaft, child link_1_fixed_joint_2_handle_knob, origin xyz=0 0 0.6 rpy=0 0 0
- added joint link_1_joint_0: type prismatic, parent base_link, child link_1_joint_0, origin xyz=0 -1.0 0.2 rpy=0 1.5708 0, axis 0 0 1.0, limit lower=0 upper=1.0 effort=0 velocity=0

Commit message: feat (minor): add "create_handle" to sampler_config

File: puzzles/continuous_space/urdf/continuous_space.urdf (robot description, URDF)
Before this commit: robot continuous_space, 19 links, 18 joints
Joints:
- joint link_3_joint_0: limit lower=0 upper=3.93321 effort=0 velocity=0 -> lower=0 upper=2.2014 effort=0 velocity=0; origin xyz=3.51572 -2.56209 0.6 rpy=-1.5708 0 -2.44487 -> xyz=5.40311 -1.16809 0.6 rpy=-1.5708 0 -1.98559

File: puzzles/simple_sliders/urdf/simple_sliders.urdf (robot description, URDF)
Before this commit: robot simple_sliders, 10 links, 9 joints
Links:
- removed link link_0_fixed_joint_1_handle_shaft
- removed link link_0_fixed_joint_1_handle_shaft.001
- removed link link_0_fixed_joint_2_handle_knob
- removed link link_0_fixed_joint_2_handle_knob.001
- removed link link_1_fixed_joint_1_handle_shaft
- removed link link_1_fixed_joint_2_handle_knob
- added link link_2_joint_0, mass 0.001; collision box size=0.2 0.2 1.6; visual box size=0.2 0.2 1.6
- added link link_3_joint_0, mass 0.001; collision box size=0.2 0.2 1.6; visual box size=0.2 0.2 1.6
Joints:
- removed joint link_0_fixed_joint_1_handle_shaft
- removed joint link_0_fixed_joint_1_handle_shaft.001
- removed joint link_0_fixed_joint_2_handle_knob
- removed joint link_0_fixed_joint_2_handle_knob.001
- removed joint link_1_fixed_joint_1_handle_shaft
- removed joint link_1_fixed_joint_2_handle_knob
- added joint link_2_joint_0: type prismatic, parent base_link, child link_2_joint_0, origin xyz=1.0 -1.0 0.2 rpy=1.5708 0 0, axis 0 0 1.0, limit lower=0 upper=1.0 effort=0 velocity=0
- added joint link_3_joint_0: type prismatic, parent base_link, child link_3_joint_0, origin xyz=1.0 -2.0 0.2 rpy=0 1.5708 0, axis 0 0 1.0, limit lower=0 upper=1.0 effort=0 velocity=0

Commit message: fix: round to avoid numbers with more than 5 decimals

File: puzzles/continuous_space/urdf/continuous_space.urdf (robot description, URDF)
Before this commit: robot continuous_space, 19 links, 18 joints
Joints:
- joint goal: origin xyz=0 0 0.6 rpy=0 0 -2.79785 -> xyz=0 0 0.6 rpy=0 0 -2.79786
- joint link_1_joint_0: origin xyz=1.89729 1.60702 0.6 rpy=0 0 -2.61769 -> xyz=1.89728 1.60703 0.6 rpy=0 0 -2.61769
- joint link_2_joint_0: origin xyz=2.7436 -0.22319 0.6 rpy=-1.5708 0 -2.39786 -> xyz=2.7436 -0.22317 0.6 rpy=-1.5708 0 -2.39786
- joint link_3_joint_0: limit lower=0 upper=2.2014 effort=0 velocity=0 -> lower=0 upper=3.93321 effort=0 velocity=0; origin xyz=5.40311 -1.16809 0.6 rpy=-1.5708 0 -1.98559 -> xyz=3.51572 -2.56206 0.6 rpy=-1.5708 0 -2.44487

File: puzzles/grid_world/urdf/grid_world.urdf (robot description, URDF)
Before this commit: robot grid_world, 19 links, 18 joints
Joints:
- joint goal: origin xyz=-0.5 0.5 0.55 rpy=0 0 1.5707 -> xyz=-0.5 0.5 0.55 rpy=0 0 1.5708

File: puzzles/lockbox_random/urdf/lockbox_random.urdf (robot description, URDF)
Before this commit: robot lockbox_random, 21 links, 20 joints
Joints:
- joint link_2_fixed_joint_1_handle_shaft: origin xyz=-1.0 0 0 rpy=0 -1.5708 0 -> xyz=-1.0 0 0 rpy=-0.06577 -1.5708 0.06577
- joint link_2_joint_0: origin xyz=0.5 2.0 0.6 rpy=-1.5708 1.5708 0 -> xyz=0.5 2.0 0.6 rpy=0 1.5708 1.5708
- joint link_3_joint_0: origin xyz=0.5 4.5 0.6 rpy=0 0 -3.14159 -> xyz=0.5 4.5 0.6 rpy=0 0 3.14159
- joint link_4_fixed_joint_1_handle_shaft: origin xyz=-1.0 0 0 rpy=0 -1.5708 0 -> xyz=-1.0 0 0 rpy=-0.01294 -1.5708 0.01294
- joint link_4_joint_0: origin xyz=-1.0 4.5 0.6 rpy=3.14159 1.5708 0 -> xyz=-1.0 4.5 0.6 rpy=-3.14159 1.57079 0

Commit message: fix: remove useless visuals (size = 0)

File: puzzles/continuous_space/urdf/continuous_space.urdf (robot description, URDF)
Before this commit: robot continuous_space, 19 links, 18 joints
Joints:
- joint link_3_joint_0: limit lower=0 upper=3.93321 effort=0 velocity=0 -> lower=0 upper=2.2014 effort=0 velocity=0; origin xyz=3.51572 -2.56206 0.6 rpy=-1.5708 0 -2.44487 -> xyz=5.40312 -1.16807 0.6 rpy=-1.5708 0 -1.98559

File: puzzles/escape_room/urdf/escape_room.urdf (robot description, URDF)
Before this commit: robot escape_room, 17 links, 16 joints
Links:
- link goal: geometry 
- link link_0_joint_0: geometry 
- link link_0_joint_1: geometry 
- link link_0_joint_1.001: geometry 
