Commit message: chore (minor): update output files according to recent changes (link_size_reduction)

File: puzzles/continuous_space/urdf/continuous_space.urdf (robot description, URDF)
Before this commit: robot continuous_space, 19 links, 18 joints
Links:
- link base_link: geometry collision box size=31.999 31.999 0.199; visual box size=31.999 31.999 0.199
- link goal: geometry visual box size=2.999 0.999 0.999
- link link_0_fixed_joint_1_handle_shaft: geometry collision cylinder length=0.999 radius=0.0995; visual cylinder length=0.999 radius=0.0995
- link link_0_fixed_joint_1_handle_shaft.001: geometry visual cylinder length=0.999 radius=0.0995
- link link_0_fixed_joint_2_handle_knob: geometry collision box size=0.049 0.049 0.199; visual box size=0.049 0.049 0.199
- link link_0_fixed_joint_2_handle_knob.001: geometry visual box size=0.049 0.049 0.199
- link link_0_fixed_joint_3_hinge: geometry visual cylinder length=1.099 radius=0.0495
- link link_0_fixed_joint_3_hinge.001: geometry visual cylinder length=1.099 radius=0.0495
- link link_0_joint_0: geometry collision box size=2.999 0.999 0.999; visual box size=2.999 0.999 0.999
- link link_1_fixed_joint_1_handle_shaft: geometry collision cylinder length=0.999 radius=0.0995; visual cylinder length=0.999 radius=0.0995
- link link_1_fixed_joint_2_handle_knob: geometry collision box size=0.049 0.049 0.199; visual box size=0.049 0.049 0.199
- link link_1_fixed_joint_3_hinge: geometry visual cylinder length=1.099 radius=0.0495
- link link_1_joint_0: geometry collision box size=2.999 0.999 0.999; visual box size=2.999 0.999 0.999
- link link_2_fixed_joint_1_handle_shaft: geometry collision box size=0.199 0.199 0.999; visual box size=0.199 0.199 0.999
- link link_2_fixed_joint_2_handle_knob: geometry collision box size=0.049 0.049 0.199; visual box size=0.049 0.049 0.199
- link link_2_joint_0: geometry collision box size=0.999 0.999 1.999; visual box size=0.999 0.999 1.999
- link link_3_fixed_joint_1_handle_shaft: geometry collision box size=0.199 0.199 0.999; visual box size=0.199 0.199 0.999
- link link_3_fixed_joint_2_handle_knob: geometry collision box size=0.049 0.049 0.199; visual box size=0.049 0.049 0.199
- link link_3_joint_0: geometry collision box size=0.999 0.999 1.999; visual box size=0.999 0.999 1.999
Joints:
- joint link_3_joint_0: limit lower=0 upper=2.2014 effort=0 velocity=0 -> lower=0 upper=3.93321 effort=0 velocity=0; origin xyz=5.40312 -1.16807 0.6 rpy=-1.5708 0 -1.98559 -> xyz=3.51572 -2.56206 0.6 rpy=-1.5708 0 -2.44487

File: puzzles/escape_room/urdf/escape_room.urdf (robot description, URDF)
Before this commit: robot escape_room, 17 links, 16 joints
Links:
- link base_link: geometry collision box size=31.999 31.999 0.199; visual box size=31.999 31.999 0.199
- link link_0_fixed_joint_3_hinge: geometry visual cylinder length=1.099 radius=0.0495
- link link_0_fixed_joint_3_hinge.001: geometry visual cylinder length=1.099 radius=0.0495
- link link_1_fixed_joint_1_hinge: geometry visual cylinder length=1.099 radius=0.0495
- link link_1_fixed_joint_2_door_panel: geometry collision box size=1.999 0.199 0.999; visual box size=1.999 0.199 0.999
- link link_1_fixed_joint_3_door_handle1: geometry collision box size=0.049 0.199 0.199; visual box size=0.049 0.199 0.199
- link link_1_fixed_joint_4_door_handle2: geometry collision box size=0.049 0.199 0.199; visual box size=0.049 0.199 0.199
- link link_1_joint_0: geometry collision cylinder length=0.999 radius=0.1995; visual cylinder length=0.999 radius=0.1995
- link link_2_fixed_joint_0_wall1: geometry collision box size=3.999 0.199 0.999; visual box size=3.999 0.199 0.999
- link link_2_fixed_joint_0_wall2: geometry collision box size=3.999 0.199 0.999; visual box size=3.999 0.199 0.999
- link link_2_fixed_joint_0_wall3: geometry collision box size=0.199 1.999 0.999; visual box size=0.199 1.999 0.999

File: puzzles/grid_world/urdf/grid_world.urdf (robot description, URDF)
Before this commit: robot grid_world, 19 links, 18 joints
Links:
- link base_link: geometry collision box size=31.999 31.999 0.199; visual box size=31.999 31.999 0.199
- link goal: geometry visual box size=2.899 0.899 0.899
- link link_0_fixed_joint_1_handle_shaft: geometry collision cylinder length=0.999 radius=0.0995; visual cylinder length=0.999 radius=0.0995
- link link_0_fixed_joint_1_handle_shaft.001: geometry visual cylinder length=0.999 radius=0.0995
- link link_0_fixed_joint_2_handle_knob: geometry collision box size=0.049 0.049 0.199; visual box size=0.049 0.049 0.199
- link link_0_fixed_joint_2_handle_knob.001: geometry visual box size=0.049 0.049 0.199
- link link_0_fixed_joint_3_hinge: geometry visual cylinder length=0.999 radius=0.0495
- link link_0_fixed_joint_3_hinge.001: geometry visual cylinder length=0.999 radius=0.0495
- link link_0_joint_0: geometry collision box size=2.899 0.899 0.899; visual box size=2.899 0.899 0.899
- link link_1_fixed_joint_1_handle_shaft: geometry collision cylinder length=0.999 radius=0.0995; visual cylinder length=0.999 radius=0.0995
- link link_1_fixed_joint_2_handle_knob: geometry collision box size=0.049 0.049 0.199; visual box size=0.049 0.049 0.199
- link link_1_fixed_joint_3_hinge: geometry visual cylinder length=0.999 radius=0.0495
- link link_1_joint_0: geometry collision box size=2.899 0.899 0.899; visual box size=2.899 0.899 0.899
- link link_2_fixed_joint_1_handle_shaft: geometry collision box size=0.199 0.199 0.999; visual box size=0.199 0.199 0.999
- link link_2_fixed_joint_2_handle_knob: geometry collision box size=0.049 0.049 0.199; visual box size=0.049 0.049 0.199
- link link_2_joint_0: geometry collision box size=0.899 0.899 1.899; visual box size=0.899 0.899 1.899
- link link_3_fixed_joint_1_handle_shaft: geometry collision box size=0.199 0.199 0.999; visual box size=0.199 0.199 0.999
- link link_3_fixed_joint_2_handle_knob: geometry collision box size=0.049 0.049 0.199; visual box size=0.049 0.049 0.199
- link link_3_joint_0: geometry collision box size=0.899 0.899 1.899; visual box size=0.899 0.899 1.899

File: puzzles/lockbox2017/urdf/lockbox2017.urdf (robot description, URDF)
Before this commit: robot lockbox2017, 23 links, 22 joints
Links:
- link base_link: geometry collision box size=31.999 31.999 0.199; visual box size=31.999 31.999 0.199
- link goal: geometry visual cylinder length=1.999 radius=0.1995
- link link_0_fixed_joint_1_hinge: geometry visual cylinder length=2.099 radius=0.0495
- link link_0_fixed_joint_1_hinge.001: geometry visual cylinder length=2.099 radius=0.0495
- link link_0_fixed_joint_2_door_panel: geometry collision box size=1.999 0.199 1.999; visual box size=1.999 0.199 1.999
- link link_0_fixed_joint_2_door_panel.001: geometry visual box size=1.999 0.199 1.999
- link link_0_fixed_joint_3_door_handle: geometry collision box size=0.199 0.049 0.199; visual box size=0.199 0.049 0.199
- link link_0_fixed_joint_3_door_handle.001: geometry visual box size=0.199 0.049 0.199
- link link_0_joint_0: geometry collision cylinder length=1.999 radius=0.1995; visual cylinder length=1.999 radius=0.1995
- link link_1_fixed_joint_1_handle_shaft: geometry collision box size=0.199 0.199 0.999; visual box size=0.199 0.199 0.999
- link link_1_fixed_joint_2_handle_knob: geometry collision box size=0.049 0.049 0.199; visual box size=0.049 0.049 0.199
- link link_1_joint_0: geometry collision box size=0.799 0.999 3.599; visual box size=0.799 0.999 3.599
- link link_2_fixed_joint_1_handle_shaft: geometry collision cylinder length=0.999 radius=0.0995; visual cylinder length=0.999 radius=0.0995
- link link_2_fixed_joint_2_handle_knob: geometry collision box size=0.049 0.049 0.199; visual box size=0.049 0.049 0.199
- link link_2_fixed_joint_3_hinge: geometry visual cylinder length=1.099 radius=0.0495
- link link_3_fixed_joint_1_handle_shaft: geometry collision box size=0.199 0.199 0.999; visual box size=0.199 0.199 0.999
- link link_3_fixed_joint_2_handle_knob: geometry collision box size=0.049 0.049 0.199; visual box size=0.049 0.049 0.199
- link link_3_joint_0: geometry collision box size=0.799 0.999 3.599; visual box size=0.799 0.999 3.599
- link link_4_fixed_joint_1_hinge: geometry visual cylinder length=2.099 radius=0.0495
- link link_4_fixed_joint_2_door_panel: geometry collision box size=3.999 0.199 1.999; visual box size=3.999 0.199 1.999
- link link_4_fixed_joint_3_door_handle: geometry collision box size=0.199 0.049 0.199; visual box size=0.199 0.049 0.199
- link link_4_joint_0: geometry collision cylinder length=1.999 radius=0.1995; visual cylinder length=1.999 radius=0.1995

File: puzzles/lockbox_random/urdf/lockbox_random.urdf (robot description, URDF)
Before this commit: robot lockbox_random, 21 links, 20 joints
Links:
- link base_link: geometry collision box size=31.999 31.999 0.199; visual box size=31.999 31.999 0.199
- link goal: geometry visual box size=0.999 0.199 1.899
- link link_0_fixed_joint_1_handle_shaft: geometry collision box size=0.199 0.199 0.999; visual box size=0.199 0.199 0.999
- link link_0_fixed_joint_1_handle_shaft.001: geometry visual box size=0.199 0.199 0.999
- link link_0_fixed_joint_2_handle_knob: geometry collision box size=0.049 0.049 0.199; visual box size=0.049 0.049 0.199
- link link_0_fixed_joint_2_handle_knob.001: geometry visual box size=0.049 0.049 0.199
- link link_0_joint_0: geometry collision box size=0.999 0.199 1.899; visual box size=0.999 0.199 1.899
- link link_1_fixed_joint_1_handle_shaft: geometry collision cylinder length=0.999 radius=0.0995; visual cylinder length=0.999 radius=0.0995
- link link_1_fixed_joint_2_handle_knob: geometry collision box size=0.049 0.049 0.199; visual box size=0.049 0.049 0.199
- link link_1_fixed_joint_3_hinge: geometry visual cylinder length=1.099 radius=0.0495
- link link_2_fixed_joint_1_handle_shaft: geometry collision box size=0.199 0.199 0.999; visual box size=0.199 0.199 0.999
- link link_2_fixed_joint_2_handle_knob: geometry collision box size=0.049 0.049 0.199; visual box size=0.049 0.049 0.199
- link link_2_joint_0: geometry collision box size=0.999 0.199 1.899; visual box size=0.999 0.199 1.899
- link link_3_fixed_joint_1_handle_shaft: geometry collision cylinder length=0.999 radius=0.0995; visual cylinder length=0.999 radius=0.0995
- link link_3_fixed_joint_2_handle_knob: geometry collision box size=0.049 0.049 0.199; visual box size=0.049 0.049 0.199
- link link_3_fixed_joint_3_hinge: geometry visual cylinder length=1.099 radius=0.0495
- link link_4_fixed_joint_1_handle_shaft: geometry collision box size=0.199 0.199 0.999; visual box size=0.199 0.199 0.999
- link link_4_fixed_joint_2_handle_knob: geometry collision box size=0.049 0.049 0.199; visual box size=0.049 0.049 0.199
- link link_4_joint_0: geometry collision box size=0.999 0.199 1.899; visual box size=0.999 0.199 1.899

File: puzzles/move_twice/urdf/move_twice.urdf (robot description, URDF)
Before this commit: robot move_twice, 14 links, 13 joints
Links:
- link base_link: geometry collision box size=31.999 31.999 0.199; visual box size=31.999 31.999 0.199
- link link_0_fixed_joint_3_hinge: geometry visual cylinder length=1.099 radius=0.0495
- link link_0_fixed_joint_3_hinge.001: geometry visual cylinder length=1.099 radius=0.0495
- link link_1_fixed_joint_0_wall_back: geometry collision box size=0.199 5.999 0.999; visual box size=0.199 5.999 0.999
- link link_1_fixed_joint_0_wall_left: geometry collision box size=3.999 0.199 0.999; visual box size=3.999 0.199 0.999
- link link_1_fixed_joint_0_wall_mid: geometry collision box size=3.999 0.199 0.999; visual box size=3.999 0.199 0.999
- link link_1_fixed_joint_0_wall_right: geometry collision box size=3.999 0.199 0.999; visual box size=3.999 0.199 0.999
- link link_1_joint_0: geometry collision box size=0.199 5.999 0.999; visual box size=0.199 5.999 0.999
Joints:
- joint goal: origin xyz=0 3.0 0.6 rpy=0 0 1.5708 -> xyz=4.0 0 0.6 rpy=0 0 0
- joint link_1_joint_0: limit lower=-2.0 upper=2.0 effort=0 velocity=0 -> lower=-3.0 upper=3.0 effort=0 velocity=0

File: puzzles/simple_sliders/urdf/simple_sliders.urdf (robot description, URDF)
Before this commit: robot simple_sliders, 6 links, 5 joints
Links:
- link base_link: geometry collision box size=31.999 31.999 0.199; visual box size=31.999 31.999 0.199
- link goal: geometry visual box size=0.199 0.199 1.599
- link link_0_joint_0: geometry collision box size=0.199 0.199 1.599; visual box size=0.199 0.199 1.599
- link link_1_joint_0: geometry collision box size=0.199 0.199 1.599; visual box size=0.199 0.199 1.599
- link link_2_joint_0: geometry collision box size=0.199 0.199 1.599; visual box size=0.199 0.199 1.599
- link link_3_joint_0: geometry collision box size=0.199 0.199 1.599; visual box size=0.199 0.199 1.599
