Commit message: chore: name links from leaf to root

File: puzzles/continuous_space/urdf/continuous_space.urdf (robot description, URDF)
Before this commit: robot continuous_space, 19 links, 18 joints
Links:
- removed link link_0_fixed_joint_1_handle_shaft
- removed link link_0_fixed_joint_1_handle_shaft.001
- removed link link_0_fixed_joint_2_handle_knob
- removed link link_0_fixed_joint_2_handle_knob.001
- removed link link_0_fixed_joint_3_hinge
- removed link link_0_fixed_joint_3_hinge.001
- removed link link_1_fixed_joint_1_handle_shaft
- removed link link_1_fixed_joint_2_handle_knob
- removed link link_1_fixed_joint_3_hinge
- removed link link_2_fixed_joint_1_handle_shaft
- removed link link_2_fixed_joint_2_handle_knob
- removed link link_3_fixed_joint_1_handle_shaft
- removed link link_3_fixed_joint_2_handle_knob
- added link link_19_fixed_handle_shaft, mass 0.001; collision cylinder length=0.999 radius=0.0995; visual cylinder length=0.999 radius=0.0995
- added link link_19_fixed_handle_shaft.001, mass 0.001; visual cylinder length=0.999 radius=0.0995
- added link link_20_fixed_handle_knob, mass 0.001; collision box size=0.049 0.049 0.199; visual box size=0.049 0.049 0.199
- added link link_20_fixed_handle_knob.001, mass 0.001; visual box size=0.049 0.049 0.199
- added link link_21_fixed_hinge, mass 0.001; visual cylinder length=1.099 radius=0.0495
- added link link_21_fixed_hinge.001, mass 0.001; visual cylinder length=1.099 radius=0.0495
- added link link_27_fixed_handle_shaft, mass 0.001; collision cylinder length=0.999 radius=0.0995; visual cylinder length=0.999 radius=0.0995
- added link link_28_fixed_handle_knob, mass 0.001; collision box size=0.049 0.049 0.199; visual box size=0.049 0.049 0.199
- added link link_29_fixed_hinge, mass 0.001; visual cylinder length=1.099 radius=0.0495
- added link link_31_fixed_handle_shaft, mass 0.001; collision box size=0.199 0.199 0.999; visual box size=0.199 0.199 0.999
- added link link_32_fixed_handle_knob, mass 0.001; collision box size=0.049 0.049 0.199; visual box size=0.049 0.049 0.199
- added link link_37_fixed_handle_shaft, mass 0.001; collision box size=0.199 0.199 0.999; visual box size=0.199 0.199 0.999
- added link link_38_fixed_handle_knob, mass 0.001; collision box size=0.049 0.049 0.199; visual box size=0.049 0.049 0.199
Joints:
- removed joint link_0_fixed_joint_1_handle_shaft
- removed joint link_0_fixed_joint_1_handle_shaft.001
- removed joint link_0_fixed_joint_2_handle_knob
- removed joint link_0_fixed_joint_2_handle_knob.001
- removed joint link_0_fixed_joint_3_hinge
- removed joint link_0_fixed_joint_3_hinge.001
- removed joint link_1_fixed_joint_1_handle_shaft
- removed joint link_1_fixed_joint_2_handle_knob
- removed joint link_1_fixed_joint_3_hinge
- removed joint link_2_fixed_joint_1_handle_shaft
- removed joint link_2_fixed_joint_2_handle_knob
- removed joint link_3_fixed_joint_1_handle_shaft
- removed joint link_3_fixed_joint_2_handle_knob
- added joint link_19_fixed_handle_shaft: type fixed, parent link_0_joint_0, child link_19_fixed_handle_shaft, origin xyz=1.125 0 1.0 rpy=0 0 0
- added joint link_19_fixed_handle_shaft.001: type fixed, parent goal, child link_19_fixed_handle_shaft.001, origin xyz=1.125 0 1.0 rpy=0 0 0
- added joint link_20_fixed_handle_knob: type fixed, parent link_19_fixed_handle_shaft, child link_20_fixed_handle_knob, origin xyz=0 0 0.6 rpy=0 0 0
- added joint link_20_fixed_handle_knob.001: type fixed, parent link_19_fixed_handle_shaft.001, child link_20_fixed_handle_knob.001, origin xyz=0 0 0.6 rpy=0 0 0
- added joint link_21_fixed_hinge: type fixed, parent link_0_joint_0, child link_21_fixed_hinge, origin xyz=0 0 0 rpy=0 0 0
- added joint link_21_fixed_hinge.001: type fixed, parent goal, child link_21_fixed_hinge.001, origin xyz=0 0 0 rpy=0 0 0
- added joint link_27_fixed_handle_shaft: type fixed, parent link_1_joint_0, child link_27_fixed_handle_shaft, origin xyz=1.125 0 1.0 rpy=0 0 0
- added joint link_28_fixed_handle_knob: type fixed, parent link_27_fixed_handle_shaft, child link_28_fixed_handle_knob, origin xyz=0 0 0.6 rpy=0 0 0
- added joint link_29_fixed_hinge: type fixed, parent link_1_joint_0, child link_29_fixed_hinge, origin xyz=0 0 0 rpy=0 0 0
- added joint link_31_fixed_handle_shaft: type fixed, parent link_2_joint_0, child link_31_fixed_handle_shaft, origin xyz=0 -1.0 0 rpy=1.5708 0 0
- added joint link_32_fixed_handle_knob: type fixed, parent link_31_fixed_handle_shaft, child link_32_fixed_handle_knob, origin xyz=0 0 0.6 rpy=0 0 0
- added joint link_37_fixed_handle_shaft: type fixed, parent link_3_joint_0, child link_37_fixed_handle_shaft, origin xyz=0 -1.0 0 rpy=1.5708 0 0
- added joint link_38_fixed_handle_knob: type fixed, parent link_37_fixed_handle_shaft, child link_38_fixed_handle_knob, origin xyz=0 0 0.6 rpy=0 0 0
- joint link_3_joint_0: limit lower=0 upper=3.93321 effort=0 velocity=0 -> lower=0 upper=2.2014 effort=0 velocity=0; origin xyz=3.51572 -2.56206 0.6 rpy=-1.5708 0 -2.44487 -> xyz=5.40312 -1.16807 0.6 rpy=-1.5708 0 -1.98559

File: puzzles/escape_room/urdf/escape_room.urdf (robot description, URDF)
Before this commit: robot escape_room, 17 links, 16 joints
Links:
- removed link link_0_fixed_joint_3_hinge
- removed link link_0_fixed_joint_3_hinge.001
- removed link link_0_joint_2.001
- removed link link_1_fixed_joint_1_hinge
- removed link link_1_fixed_joint_2_door_panel
- removed link link_1_fixed_joint_3_door_handle1
- removed link link_1_fixed_joint_4_door_handle2
- removed link link_2_fixed_joint_0_wall1
- removed link link_2_fixed_joint_0_wall2
- removed link link_2_fixed_joint_0_wall3
- added link link_0_joint_0.001, mass 0.001; visual mesh filename=file:///home/userone/ba/puzzle-generator/puzzles/escape_roo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 scale=1.0 1.0 1.0
- added link link_77_fixed_hinge, mass 0.001; visual cylinder length=1.099 radius=0.0495
- added link link_77_fixed_hinge.001, mass 0.001; visual cylinder length=1.099 radius=0.0495
- added link link_79_fixed_hinge, mass 0.001; visual cylinder length=1.099 radius=0.0495
- added link link_80_fixed_door_panel, mass 0.001; collision box size=1.999 0.199 0.999; visual box size=1.999 0.199 0.999
- added link link_81_fixed_door_handle1, mass 0.001; collision box size=0.049 0.199 0.199; visual box size=0.049 0.199 0.199
- added link link_82_fixed_door_handle2, mass 0.001; collision box size=0.049 0.199 0.199; visual box size=0.049 0.199 0.199
- added link link_83_fixed_wall1, mass 0.001; collision box size=3.999 0.199 0.999; visual box size=3.999 0.199 0.999
- added link link_84_fixed_wall2, mass 0.001; collision box size=3.999 0.199 0.999; visual box size=3.999 0.199 0.999
- added link link_85_fixed_wall3, mass 0.001; collision box size=0.199 1.999 0.999; visual box size=0.199 1.999 0.999
- link link_0_joint_0: geometry collision mesh filename=file:///home/userone/ba/puzzle-generator/puzzles/escape_roo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 scale=1.0 1.0 1.0; visual mesh filename=file:///home/userone/ba/puzzle-generator/puzzles/escape_roo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 scale=1.0 1.0 1.0
- link link_0_joint_2: geometry 
Joints:
- removed joint link_0_fixed_joint_3_hinge
- removed joint link_0_fixed_joint_3_hinge.001
- removed joint link_0_joint_2.001
- removed joint link_1_fixed_joint_1_hinge
- removed joint link_1_fixed_joint_2_door_panel
- removed joint link_1_fixed_joint_3_door_handle1
- removed joint link_1_fixed_joint_4_door_handle2
- removed joint link_2_fixed_joint_0_wall1
- removed joint link_2_fixed_joint_0_wall2
- removed joint link_2_fixed_joint_0_wall3
- added joint link_0_joint_0.001: type fixed, parent link_0_joint_1.001, child link_0_joint_0.001, origin xyz=0 0 0 rpy=0 0 0, limit effort=0 velocity=0
- added joint link_77_fixed_hinge: type fixed, parent link_0_joint_0, child link_77_fixed_hinge, origin xyz=0 0 0 rpy=0 0 0
- added joint link_77_fixed_hinge.001: type fixed, parent link_0_joint_0.001, child link_77_fixed_hinge.001, origin xyz=0 0 0 rpy=0 0 0
- added joint link_79_fixed_hinge: type fixed, parent link_1_joint_0, child link_79_fixed_hinge, origin xyz=0 0 0 rpy=0 0 0
- added joint link_80_fixed_door_panel: type fixed, parent link_1_joint_0, child link_80_fixed_door_panel, origin xyz=1.0 0 0 rpy=0 0 0
- added joint link_81_fixed_door_handle1: type fixed, parent link_1_joint_0, child link_81_fixed_door_handle1, origin xyz=1.5 0.2 0 rpy=0 0 0
- added joint link_82_fixed_door_handle2: type fixed, parent link_1_joint_0, child link_82_fixed_door_handle2, origin xyz=1.5 -0.2 0 rpy=0 0 0
- added joint link_83_fixed_wall1: type fixed, parent base_link, child link_83_fixed_wall1, origin xyz=0 -1.4 0.6 rpy=0 0 0
- added joint link_84_fixed_wall2: type fixed, parent base_link, child link_84_fixed_wall2, origin xyz=0 1.4 0.6 rpy=0 0 0
- added joint link_85_fixed_wall3: type fixed, parent base_link, child link_85_fixed_wall3, origin xyz=-2.0 0 0.6 rpy=0 0 0
- joint link_0_joint_0: axis 1.0 0 0 -> 0 0 1.0; limit lower=-16.0 upper=16.0 effort=0 velocity=0 -> lower=-3.14159 upper=3.14159 effort=0 velocity=0; origin xyz=0 0 0.6 rpy=0 0 0 -> xyz=0 0 0 rpy=0 0 0; parent base_link -> link_0_joint_1; type prismatic -> revolute
- joint link_0_joint_1: parent link_0_joint_0 -> link_0_joint_2
- joint link_0_joint_2: axis 0 0 1.0 -> 1.0 0 0; limit lower=-3.14159 upper=3.14159 effort=0 velocity=0 -> lower=-16.0 upper=16.0 effort=0 velocity=0; origin xyz=0 0 0 rpy=0 0 0 -> xyz=0 0 0.6 rpy=0 0 0; parent link_0_joint_1 -> base_link; type revolute -> prismatic

File: puzzles/grid_world/urdf/grid_world.urdf (robot description, URDF)
Before this commit: robot grid_world, 19 links, 18 joints
Links:
- removed link link_0_fixed_joint_1_handle_shaft
- removed link link_0_fixed_joint_1_handle_shaft.001
- removed link link_0_fixed_joint_2_handle_knob
- removed link link_0_fixed_joint_2_handle_knob.001
- removed link link_0_fixed_joint_3_hinge
- removed link link_0_fixed_joint_3_hinge.001
- removed link link_1_fixed_joint_1_handle_shaft
- removed link link_1_fixed_joint_2_handle_knob
- removed link link_1_fixed_joint_3_hinge
- removed link link_2_fixed_joint_1_handle_shaft
- removed link link_2_fixed_joint_2_handle_knob
- removed link link_3_fixed_joint_1_handle_shaft
- removed link link_3_fixed_joint_2_handle_knob
- added link link_10_fixed_handle_knob, mass 0.001; collision box size=0.049 0.049 0.199; visual box size=0.049 0.049 0.199
- added link link_11_fixed_hinge, mass 0.001; visual cylinder length=0.999 radius=0.0495
- added link link_13_fixed_handle_shaft, mass 0.001; collision box size=0.199 0.199 0.999; visual box size=0.199 0.199 0.999
- added link link_14_fixed_handle_knob, mass 0.001; collision box size=0.049 0.049 0.199; visual box size=0.049 0.049 0.199
- added link link_16_fixed_handle_shaft, mass 0.001; collision box size=0.199 0.199 0.999; visual box size=0.199 0.199 0.999
- added link link_17_fixed_handle_knob, mass 0.001; collision box size=0.049 0.049 0.199; visual box size=0.049 0.049 0.199
- added link link_5_fixed_handle_shaft, mass 0.001; collision cylinder length=0.999 radius=0.0995; visual cylinder length=0.999 radius=0.0995
- added link link_5_fixed_handle_shaft.001, mass 0.001; visual cylinder length=0.999 radius=0.0995
- added link link_6_fixed_handle_knob, mass 0.001; collision box size=0.049 0.049 0.199; visual box size=0.049 0.049 0.199
- added link link_6_fixed_handle_knob.001, mass 0.001; visual box size=0.049 0.049 0.199
- added link link_7_fixed_hinge, mass 0.001; visual cylinder length=0.999 radius=0.0495
- added link link_7_fixed_hinge.001, mass 0.001; visual cylinder length=0.999 radius=0.0495
- added link link_9_fixed_handle_shaft, mass 0.001; collision cylinder length=0.999 radius=0.0995; visual cylinder length=0.999 radius=0.0995
Joints:
- removed joint link_0_fixed_joint_1_handle_shaft
- removed joint link_0_fixed_joint_1_handle_shaft.001
- removed joint link_0_fixed_joint_2_handle_knob
- removed joint link_0_fixed_joint_2_handle_knob.001
- removed joint link_0_fixed_joint_3_hinge
- removed joint link_0_fixed_joint_3_hinge.001
- removed joint link_1_fixed_joint_1_handle_shaft
- removed joint link_1_fixed_joint_2_handle_knob
- removed joint link_1_fixed_joint_3_hinge
- removed joint link_2_fixed_joint_1_handle_shaft
- removed joint link_2_fixed_joint_2_handle_knob
- removed joint link_3_fixed_joint_1_handle_shaft
- removed joint link_3_fixed_joint_2_handle_knob
- added joint link_10_fixed_handle_knob: type fixed, parent link_9_fixed_handle_shaft, child link_10_fixed_handle_knob, origin xyz=0 0 0.6 rpy=0 0 0
- added joint link_11_fixed_hinge: type fixed, parent link_1_joint_0, child link_11_fixed_hinge, origin xyz=0 0 0 rpy=0 0 0
- added joint link_13_fixed_handle_shaft: type fixed, parent link_2_joint_0, child link_13_fixed_handle_shaft, origin xyz=-0.95 0 0 rpy=0 -1.5708 0
- added joint link_14_fixed_handle_knob: type fixed, parent link_13_fixed_handle_shaft, child link_14_fixed_handle_knob, origin xyz=0 0 0.6 rpy=0 0 0
- added joint link_16_fixed_handle_shaft: type fixed, parent link_3_joint_0, child link_16_fixed_handle_shaft, origin xyz=0 0.95 0 rpy=-1.5708 0 0
- added joint link_17_fixed_handle_knob: type fixed, parent link_16_fixed_handle_shaft, child link_17_fixed_handle_knob, origin xyz=0 0 0.6 rpy=0 0 0
- added joint link_5_fixed_handle_shaft: type fixed, parent link_0_joint_0, child link_5_fixed_handle_shaft, origin xyz=1.0875 0 0.95 rpy=0 0 0
- added joint link_5_fixed_handle_shaft.001: type fixed, parent goal, child link_5_fixed_handle_shaft.001, origin xyz=1.0875 0 0.95 rpy=0 0 0
- added joint link_6_fixed_handle_knob: type fixed, parent link_5_fixed_handle_shaft, child link_6_fixed_handle_knob, origin xyz=0 0 0.6 rpy=0 0 0
- added joint link_6_fixed_handle_knob.001: type fixed, parent link_5_fixed_handle_shaft.001, child link_6_fixed_handle_knob.001, origin xyz=0 0 0.6 rpy=0 0 0
- added joint link_7_fixed_hinge: type fixed, parent link_0_joint_0, child link_7_fixed_hinge, origin xyz=0 0 0 rpy=0 0 0
- added joint link_7_fixed_hinge.001: type fixed, parent goal, child link_7_fixed_hinge.001, origin xyz=0 0 0 rpy=0 0 0
- added joint link_9_fixed_handle_shaft: type fixed, parent link_1_joint_0, child link_9_fixed_handle_shaft, origin xyz=1.0875 0 0.95 rpy=0 0 0

File: puzzles/lockbox2017/urdf/lockbox2017.urdf (robot description, URDF)
Before this commit: robot lockbox2017, 23 links, 22 joints
Links:
- removed link link_0_fixed_joint_1_hinge
- removed link link_0_fixed_joint_1_hinge.001
- removed link link_0_fixed_joint_2_door_panel
- removed link link_0_fixed_joint_2_door_panel.001
- removed link link_0_fixed_joint_3_door_handle
- removed link link_0_fixed_joint_3_door_handle.001
- removed link link_1_fixed_joint_1_handle_shaft
- removed link link_1_fixed_joint_2_handle_knob
- removed link link_2_fixed_joint_1_handle_shaft
- removed link link_2_fixed_joint_2_handle_knob
- removed link link_2_fixed_joint_3_hinge
- removed link link_3_fixed_joint_1_handle_shaft
- removed link link_3_fixed_joint_2_handle_knob
- removed link link_4_fixed_joint_1_hinge
- removed link link_4_fixed_joint_2_door_panel
- removed link link_4_fixed_joint_3_door_handle
- added link link_40_fixed_hinge, mass 0.001; visual cylinder length=2.099 radius=0.0495
- added link link_40_fixed_hinge.001, mass 0.001; visual cylinder length=2.099 radius=0.0495
- added link link_41_fixed_door_panel, mass 0.001; collision box size=1.999 0.199 1.999; visual box size=1.999 0.199 1.999
- added link link_41_fixed_door_panel.001, mass 0.001; visual box size=1.999 0.199 1.999
- added link link_42_fixed_door_handle, mass 0.001; collision box size=0.199 0.049 0.199; visual box size=0.199 0.049 0.199
- added link link_42_fixed_door_handle.001, mass 0.001; visual box size=0.199 0.049 0.199
- added link link_44_fixed_handle_shaft, mass 0.001; collision box size=0.199 0.199 0.999; visual box size=0.199 0.199 0.999
- added link link_45_fixed_handle_knob, mass 0.001; collision box size=0.049 0.049 0.199; visual box size=0.049 0.049 0.199
- added link link_47_fixed_handle_shaft, mass 0.001; collision cylinder length=0.999 radius=0.0995; visual cylinder length=0.999 radius=0.0995
- added link link_48_fixed_handle_knob, mass 0.001; collision box size=0.049 0.049 0.199; visual box size=0.049 0.049 0.199
- added link link_49_fixed_hinge, mass 0.001; visual cylinder length=1.099 radius=0.0495
- added link link_51_fixed_handle_shaft, mass 0.001; collision box size=0.199 0.199 0.999; visual box size=0.199 0.199 0.999
- added link link_52_fixed_handle_knob, mass 0.001; collision box size=0.049 0.049 0.199; visual box size=0.049 0.049 0.199
- added link link_54_fixed_hinge, mass 0.001; visual cylinder length=2.099 radius=0.0495
- added link link_55_fixed_door_panel, mass 0.001; collision box size=3.999 0.199 1.999; visual box size=3.999 0.199 1.999
- added link link_56_fixed_door_handle, mass 0.001; collision box size=0.199 0.049 0.199; visual box size=0.199 0.049 0.199
Joints:
- removed joint link_0_fixed_joint_1_hinge
- removed joint link_0_fixed_joint_1_hinge.001
- removed joint link_0_fixed_joint_2_door_panel
- removed joint link_0_fixed_joint_2_door_panel.001
- removed joint link_0_fixed_joint_3_door_handle
- removed joint link_0_fixed_joint_3_door_handle.001
- removed joint link_1_fixed_joint_1_handle_shaft
- removed joint link_1_fixed_joint_2_handle_knob
- removed joint link_2_fixed_joint_1_handle_shaft
- removed joint link_2_fixed_joint_2_handle_knob
- removed joint link_2_fixed_joint_3_hinge
- removed joint link_3_fixed_joint_1_handle_shaft
- removed joint link_3_fixed_joint_2_handle_knob
- removed joint link_4_fixed_joint_1_hinge
- removed joint link_4_fixed_joint_2_door_panel
- removed joint link_4_fixed_joint_3_door_handle
- added joint link_40_fixed_hinge: type fixed, parent link_0_joint_0, child link_40_fixed_hinge, origin xyz=0 0 0 rpy=0 0 0
- added joint link_40_fixed_hinge.001: type fixed, parent goal, child link_40_fixed_hinge.001, origin xyz=0 0 0 rpy=0 0 0
- added joint link_41_fixed_door_panel: type fixed, parent link_0_joint_0, child link_41_fixed_door_panel, origin xyz=1.0 0 0 rpy=0 0 0
- added joint link_41_fixed_door_panel.001: type fixed, parent goal, child link_41_fixed_door_panel.001, origin xyz=1.0 0 0 rpy=0 0 0
- added joint link_42_fixed_door_handle: type fixed, parent link_0_joint_0, child link_42_fixed_door_handle, origin xyz=1.5 0 1.1 rpy=0 0 0
- added joint link_42_fixed_door_handle.001: type fixed, parent goal, child link_42_fixed_door_handle.001, origin xyz=1.5 0 1.1 rpy=0 0 0
- added joint link_44_fixed_handle_shaft: type fixed, parent link_1_joint_0, child link_44_fixed_handle_shaft, origin xyz=0 -1.0 0 rpy=1.5708 0 0
- added joint link_45_fixed_handle_knob: type fixed, parent link_44_fixed_handle_shaft, child link_45_fixed_handle_knob, origin xyz=0 0 0.6 rpy=0 0 0
- added joint link_47_fixed_handle_shaft: type fixed, parent link_2_joint_0, child link_47_fixed_handle_shaft, origin xyz=0 1.5 1.0 rpy=0 0 0
- added joint link_48_fixed_handle_knob: type fixed, parent link_47_fixed_handle_shaft, child link_48_fixed_handle_knob, origin xyz=0 0 0.6 rpy=0 0 0
- added joint link_49_fixed_hinge: type fixed, parent link_2_joint_0, child link_49_fixed_hinge, origin xyz=0 0 0 rpy=0 0 0
- added joint link_51_fixed_handle_shaft: type fixed, parent link_3_joint_0, child link_51_fixed_handle_shaft, origin xyz=0 -1.0 0 rpy=1.5708 0 0
- added joint link_52_fixed_handle_knob: type fixed, parent link_51_fixed_handle_shaft, child link_52_fixed_handle_knob, origin xyz=0 0 0.6 rpy=0 0 0
- added joint link_54_fixed_hinge: type fixed, parent link_4_joint_0, child link_54_fixed_hinge, origin xyz=0 0 0 rpy=0 0 0
- added joint link_55_fixed_door_panel: type fixed, parent link_4_joint_0, child link_55_fixed_door_panel, origin xyz=2.0 0 0 rpy=0 0 0
- added joint link_56_fixed_door_handle: type fixed, parent link_4_joint_0, child link_56_fixed_door_handle, origin xyz=3.0 0 1.1 rpy=0 0 0
