Commit message: chore: name links from leaf to root

File: puzzles/lockbox_random/urdf/lockbox_random.urdf (robot description, URDF)
Before this commit: robot lockbox_random, 21 links, 20 joints
Links:
- removed link link_0_fixed_joint_1_handle_shaft
- removed link link_0_fixed_joint_1_handle_shaft.001
- removed link link_0_fixed_joint_2_handle_knob
- removed link link_0_fixed_joint_2_handle_knob.001
- removed link link_1_fixed_joint_1_handle_shaft
- removed link link_1_fixed_joint_2_handle_knob
- removed link link_1_fixed_joint_3_hinge
- removed link link_2_fixed_joint_1_handle_shaft
- removed link link_2_fixed_joint_2_handle_knob
- removed link link_3_fixed_joint_1_handle_shaft
- removed link link_3_fixed_joint_2_handle_knob
- removed link link_3_fixed_joint_3_hinge
- removed link link_4_fixed_joint_1_handle_shaft
- removed link link_4_fixed_joint_2_handle_knob
- added link link_58_fixed_handle_shaft, mass 0.001; collision box size=0.199 0.199 0.999; visual box size=0.199 0.199 0.999
- added link link_58_fixed_handle_shaft.001, mass 0.001; visual box size=0.199 0.199 0.999
- added link link_59_fixed_handle_knob, mass 0.001; collision box size=0.049 0.049 0.199; visual box size=0.049 0.049 0.199
- added link link_59_fixed_handle_knob.001, mass 0.001; visual box size=0.049 0.049 0.199
- added link link_61_fixed_handle_shaft, mass 0.001; collision cylinder length=0.999 radius=0.0995; visual cylinder length=0.999 radius=0.0995
- added link link_62_fixed_handle_knob, mass 0.001; collision box size=0.049 0.049 0.199; visual box size=0.049 0.049 0.199
- added link link_63_fixed_hinge, mass 0.001; visual cylinder length=1.099 radius=0.0495
- added link link_65_fixed_handle_shaft, mass 0.001; collision box size=0.199 0.199 0.999; visual box size=0.199 0.199 0.999
- added link link_66_fixed_handle_knob, mass 0.001; collision box size=0.049 0.049 0.199; visual box size=0.049 0.049 0.199
- added link link_68_fixed_handle_shaft, mass 0.001; collision cylinder length=0.999 radius=0.0995; visual cylinder length=0.999 radius=0.0995
- added link link_69_fixed_handle_knob, mass 0.001; collision box size=0.049 0.049 0.199; visual box size=0.049 0.049 0.199
- added link link_70_fixed_hinge, mass 0.001; visual cylinder length=1.099 radius=0.0495
- added link link_72_fixed_handle_shaft, mass 0.001; collision box size=0.199 0.199 0.999; visual box size=0.199 0.199 0.999
- added link link_73_fixed_handle_knob, mass 0.001; collision box size=0.049 0.049 0.199; visual box size=0.049 0.049 0.199
Joints:
- removed joint link_0_fixed_joint_1_handle_shaft
- removed joint link_0_fixed_joint_1_handle_shaft.001
- removed joint link_0_fixed_joint_2_handle_knob
- removed joint link_0_fixed_joint_2_handle_knob.001
- removed joint link_1_fixed_joint_1_handle_shaft
- removed joint link_1_fixed_joint_2_handle_knob
- removed joint link_1_fixed_joint_3_hinge
- removed joint link_2_fixed_joint_1_handle_shaft
- removed joint link_2_fixed_joint_2_handle_knob
- removed joint link_3_fixed_joint_1_handle_shaft
- removed joint link_3_fixed_joint_2_handle_knob
- removed joint link_3_fixed_joint_3_hinge
- removed joint link_4_fixed_joint_1_handle_shaft
- removed joint link_4_fixed_joint_2_handle_knob
- added joint link_58_fixed_handle_shaft: type fixed, parent link_0_joint_0, child link_58_fixed_handle_shaft, origin xyz=-1.0 0 0 rpy=0 -1.5708 0
- added joint link_58_fixed_handle_shaft.001: type fixed, parent goal, child link_58_fixed_handle_shaft.001, origin xyz=-1.0 0 0 rpy=0 -1.5708 0
- added joint link_59_fixed_handle_knob: type fixed, parent link_58_fixed_handle_shaft, child link_59_fixed_handle_knob, origin xyz=0 0 0.6 rpy=0 0 0
- added joint link_59_fixed_handle_knob.001: type fixed, parent link_58_fixed_handle_shaft.001, child link_59_fixed_handle_knob.001, origin xyz=0 0 0.6 rpy=0 0 0
- added joint link_61_fixed_handle_shaft: type fixed, parent link_1_joint_0, child link_61_fixed_handle_shaft, origin xyz=0 1.125 1.0 rpy=0 0 0
- added joint link_62_fixed_handle_knob: type fixed, parent link_61_fixed_handle_shaft, child link_62_fixed_handle_knob, origin xyz=0 0 0.6 rpy=0 0 0
- added joint link_63_fixed_hinge: type fixed, parent link_1_joint_0, child link_63_fixed_hinge, origin xyz=0 0 0 rpy=0 0 0
- added joint link_65_fixed_handle_shaft: type fixed, parent link_2_joint_0, child link_65_fixed_handle_shaft, origin xyz=-1.0 0 0 rpy=-0.06577 -1.5708 0.06577
- added joint link_66_fixed_handle_knob: type fixed, parent link_65_fixed_handle_shaft, child link_66_fixed_handle_knob, origin xyz=0 0 0.6 rpy=0 0 0
- added joint link_68_fixed_handle_shaft: type fixed, parent link_3_joint_0, child link_68_fixed_handle_shaft, origin xyz=0 1.125 1.0 rpy=0 0 0
- added joint link_69_fixed_handle_knob: type fixed, parent link_68_fixed_handle_shaft, child link_69_fixed_handle_knob, origin xyz=0 0 0.6 rpy=0 0 0
- added joint link_70_fixed_hinge: type fixed, parent link_3_joint_0, child link_70_fixed_hinge, origin xyz=0 0 0 rpy=0 0 0
- added joint link_72_fixed_handle_shaft: type fixed, parent link_4_joint_0, child link_72_fixed_handle_shaft, origin xyz=-1.0 0 0 rpy=-0.01294 -1.5708 0.01294
- added joint link_73_fixed_handle_knob: type fixed, parent link_72_fixed_handle_shaft, child link_73_fixed_handle_knob, origin xyz=0 0 0.6 rpy=0 0 0

File: puzzles/move_twice/urdf/move_twice.urdf (robot description, URDF)
Before this commit: robot move_twice, 14 links, 13 joints
Links:
- removed link link_0_fixed_joint_3_hinge
- removed link link_0_fixed_joint_3_hinge.001
- removed link link_0_joint_2.001
- removed link link_1_fixed_joint_0_wall_back
- removed link link_1_fixed_joint_0_wall_left
- removed link link_1_fixed_joint_0_wall_mid
- removed link link_1_fixed_joint_0_wall_right
- added link link_0_joint_0.001, mass 0.001; visual mesh filename=file:///home/userone/ba/puzzle-generator/puzzles/move_twice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 scale=1.0 1.0 1.0
- added link link_89_fixed_hinge, mass 0.001; visual cylinder length=1.099 radius=0.0495
- added link link_89_fixed_hinge.001, mass 0.001; visual cylinder length=1.099 radius=0.0495
- added link link_90_fixed_wall_left, mass 0.001; collision box size=3.999 0.199 0.999; visual box size=3.999 0.199 0.999
- added link link_91_fixed_wall_right, mass 0.001; collision box size=3.999 0.199 0.999; visual box size=3.999 0.199 0.999
- added link link_92_fixed_wall_mid, mass 0.001; collision box size=3.999 0.199 0.999; visual box size=3.999 0.199 0.999
- added link link_93_fixed_wall_back, mass 0.001; collision box size=0.199 5.999 0.999; visual box size=0.199 5.999 0.999
- link link_0_joint_0: geometry collision mesh filename=file:///home/userone/ba/puzzle-generator/puzzles/move_twice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 scale=1.0 1.0 1.0; visual mesh filename=file:///home/userone/ba/puzzle-generator/puzzles/move_twice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 scale=1.0 1.0 1.0
- link link_0_joint_2: geometry 
Joints:
- removed joint link_0_fixed_joint_3_hinge
- removed joint link_0_fixed_joint_3_hinge.001
- removed joint link_0_joint_2.001
- removed joint link_1_fixed_joint_0_wall_back
- removed joint link_1_fixed_joint_0_wall_left
- removed joint link_1_fixed_joint_0_wall_mid
- removed joint link_1_fixed_joint_0_wall_right
- added joint link_0_joint_0.001: type fixed, parent link_0_joint_1.001, child link_0_joint_0.001, origin xyz=0 0 0 rpy=0 0 0, limit effort=0 velocity=0
- added joint link_89_fixed_hinge: type fixed, parent link_0_joint_0, child link_89_fixed_hinge, origin xyz=0 0 0 rpy=0 0 0
- added joint link_89_fixed_hinge.001: type fixed, parent link_0_joint_0.001, child link_89_fixed_hinge.001, origin xyz=0 0 0 rpy=0 0 0
- added joint link_90_fixed_wall_left: type fixed, parent base_link, child link_90_fixed_wall_left, origin xyz=0 -1.4 0.6 rpy=0 0 0
- added joint link_91_fixed_wall_right: type fixed, parent base_link, child link_91_fixed_wall_right, origin xyz=0 4.4 0.6 rpy=0 0 0
- added joint link_92_fixed_wall_mid: type fixed, parent base_link, child link_92_fixed_wall_mid, origin xyz=0 1.5 0.6 rpy=0 0 0
- added joint link_93_fixed_wall_back: type fixed, parent base_link, child link_93_fixed_wall_back, origin xyz=-2.1 1.5 0.6 rpy=0 0 0
- joint goal: origin xyz=4.0 0 0.6 rpy=0 0 0 -> xyz=0 3.0 0.6 rpy=0 0 1.5708
- joint link_0_joint_0: axis 1.0 0 0 -> 0 0 1.0; limit lower=-16.0 upper=16.0 effort=0 velocity=0 -> lower=-3.14159 upper=3.14159 effort=0 velocity=0; origin xyz=0 0 0.6 rpy=0 0 0 -> xyz=0 0 0 rpy=0 0 0; parent base_link -> link_0_joint_1; type prismatic -> revolute
- joint link_0_joint_1: parent link_0_joint_0 -> link_0_joint_2
- joint link_0_joint_2: axis 0 0 1.0 -> 1.0 0 0; limit lower=-3.14159 upper=3.14159 effort=0 velocity=0 -> lower=-16.0 upper=16.0 effort=0 velocity=0; origin xyz=0 0 0 rpy=0 0 0 -> xyz=0 0 0.6 rpy=0 0 0; parent link_0_joint_1 -> base_link; type revolute -> prismatic
