Commit message: feat: add obstacle to escape_room

File: puzzles/continuous_space/urdf/continuous_space.urdf (robot description, URDF)
Before this commit: robot continuous_space, 19 links, 18 joints
Links:
- removed link link_37_fixed_handle_shaft
- removed link link_38_fixed_handle_knob
- added link link_40_fixed_handle_shaft, mass 0.001; collision box size=0.199 0.199 0.999; visual box size=0.199 0.199 0.999
- added link link_41_fixed_handle_knob, mass 0.001; collision box size=0.049 0.049 0.199; visual box size=0.049 0.049 0.199
Joints:
- removed joint link_37_fixed_handle_shaft
- removed joint link_38_fixed_handle_knob
- added joint link_40_fixed_handle_shaft: type fixed, parent link_3_joint_0, child link_40_fixed_handle_shaft, origin xyz=0 -1.0 0 rpy=1.5708 0 0
- added joint link_41_fixed_handle_knob: type fixed, parent link_40_fixed_handle_shaft, child link_41_fixed_handle_knob, origin xyz=0 0 0.6 rpy=0 0 0
- joint link_3_joint_0: limit lower=0 upper=2.2014 effort=0 velocity=0 -> lower=0 upper=3.93321 effort=0 velocity=0; origin xyz=5.40312 -1.16807 0.6 rpy=-1.5708 0 -1.98559 -> xyz=3.51572 -2.56206 0.6 rpy=-1.5708 0 -2.44487

File: puzzles/escape_room/urdf/escape_room.urdf (robot description, URDF)
Before this commit: robot escape_room, 17 links, 16 joints
Links:
- removed link link_77_fixed_hinge
- removed link link_77_fixed_hinge.001
- removed link link_79_fixed_hinge
- removed link link_80_fixed_door_panel
- removed link link_81_fixed_door_handle1
- removed link link_82_fixed_door_handle2
- removed link link_83_fixed_wall1
- removed link link_84_fixed_wall2
- removed link link_85_fixed_wall3
- added link link_1_joint_1, mass 0.001
- added link link_1_joint_2, mass 0.001
- added link link_2_joint_0, mass 0.001; collision cylinder length=0.999 radius=0.1995; visual cylinder length=0.999 radius=0.1995
- added link link_80_fixed_hinge, mass 0.001; visual cylinder length=1.099 radius=0.0495
- added link link_80_fixed_hinge.001, mass 0.001; visual cylinder length=1.099 radius=0.0495
- added link link_84_fixed_hinge, mass 0.001; visual cylinder length=0.349 radius=0.0495
- added link link_86_fixed_hinge, mass 0.001; visual cylinder length=1.099 radius=0.0495
- added link link_87_fixed_door_panel, mass 0.001; collision box size=2.999 0.199 0.999; visual box size=2.999 0.199 0.999
- added link link_88_fixed_door_handle1, mass 0.001; collision box size=0.049 0.199 0.199; visual box size=0.049 0.199 0.199
- added link link_89_fixed_door_handle2, mass 0.001; collision box size=0.049 0.199 0.199; visual box size=0.049 0.199 0.199
- added link link_90_fixed_wall_left, mass 0.001; collision box size=3.799 0.199 0.249; visual box size=3.799 0.199 0.249
- added link link_91_fixed_wall_front, mass 0.001; collision box size=0.199 7.999 0.249; visual box size=0.199 7.999 0.249
- added link link_92_fixed_wall_back, mass 0.001; collision box size=0.199 7.999 0.249; visual box size=0.199 7.999 0.249
- link link_1_joint_0: geometry collision box size=2.499 0.199 0.249; visual box size=2.499 0.199 0.249
Joints:
- removed joint link_77_fixed_hinge
- removed joint link_77_fixed_hinge.001
- removed joint link_79_fixed_hinge
- removed joint link_80_fixed_door_panel
- removed joint link_81_fixed_door_handle1
- removed joint link_82_fixed_door_handle2
- removed joint link_83_fixed_wall1
- removed joint link_84_fixed_wall2
- removed joint link_85_fixed_wall3
- added joint link_1_joint_1: type prismatic, parent link_1_joint_2, child link_1_joint_1, origin xyz=0 0 0 rpy=0 0 0, axis 0 1.0 0, limit lower=-16.0 upper=16.0 effort=0 velocity=0
- added joint link_1_joint_2: type prismatic, parent base_link, child link_1_joint_2, origin xyz=0 3.30215 0.225 rpy=0 0 0, axis 1.0 0 0, limit lower=-16.0 upper=16.0 effort=0 velocity=0
- added joint link_2_joint_0: type revolute, parent base_link, child link_2_joint_0, origin xyz=1.5 4.0 0.6 rpy=0 0 3.14159, axis 0 0 1.0, limit lower=0 upper=1.5708 effort=0 velocity=0
- added joint link_80_fixed_hinge: type fixed, parent link_0_joint_0, child link_80_fixed_hinge, origin xyz=0 0 0 rpy=0 0 0
- added joint link_80_fixed_hinge.001: type fixed, parent link_0_joint_0.001, child link_80_fixed_hinge.001, origin xyz=0 0 0 rpy=0 0 0
- added joint link_84_fixed_hinge: type fixed, parent link_1_joint_0, child link_84_fixed_hinge, origin xyz=0 0 0 rpy=0 0 0
- added joint link_86_fixed_hinge: type fixed, parent link_2_joint_0, child link_86_fixed_hinge, origin xyz=0 0 0 rpy=0 0 0
- added joint link_87_fixed_door_panel: type fixed, parent link_2_joint_0, child link_87_fixed_door_panel, origin xyz=1.5 0 0 rpy=0 0 0
- added joint link_88_fixed_door_handle1: type fixed, parent link_2_joint_0, child link_88_fixed_door_handle1, origin xyz=2.25 0.2 0 rpy=0 0 0
- added joint link_89_fixed_door_handle2: type fixed, parent link_2_joint_0, child link_89_fixed_door_handle2, origin xyz=2.25 -0.2 0 rpy=0 0 0
- added joint link_90_fixed_wall_left: type fixed, parent base_link, child link_90_fixed_wall_left, origin xyz=0 -4.0 0.225 rpy=0 0 0
- added joint link_91_fixed_wall_front: type fixed, parent base_link, child link_91_fixed_wall_front, origin xyz=2.0 0 0.225 rpy=0 0 0
- added joint link_92_fixed_wall_back: type fixed, parent base_link, child link_92_fixed_wall_back, origin xyz=-2.0 0 0.225 rpy=0 0 0
- joint goal: origin xyz=4.0 0 0.6 rpy=0 0 1.5708 -> xyz=0 5.0 0.6 rpy=0 0 1.5708
- joint link_1_joint_0: limit lower=0 upper=1.5708 effort=0 velocity=0 -> lower=-3.14159 upper=3.14159 effort=0 velocity=0; origin xyz=2.0 -1.0 0.6 rpy=0 0 1.5708 -> xyz=0 0 0 rpy=0 0 0; parent base_link -> link_1_joint_1

File: puzzles/lockbox2017/urdf/lockbox2017.urdf (robot description, URDF)
Before this commit: robot lockbox2017, 23 links, 22 joints
Links:
- removed link link_40_fixed_hinge
- removed link link_40_fixed_hinge.001
- removed link link_41_fixed_door_panel
- removed link link_41_fixed_door_panel.001
- removed link link_42_fixed_door_handle
- removed link link_42_fixed_door_handle.001
- removed link link_44_fixed_handle_shaft
- removed link link_45_fixed_handle_knob
- removed link link_49_fixed_hinge
- removed link link_51_fixed_handle_shaft
- removed link link_52_fixed_handle_knob
- removed link link_54_fixed_hinge
- removed link link_55_fixed_door_panel
- removed link link_56_fixed_door_handle
- added link link_43_fixed_hinge, mass 0.001; visual cylinder length=2.099 radius=0.0495
- added link link_43_fixed_hinge.001, mass 0.001; visual cylinder length=2.099 radius=0.0495
- added link link_44_fixed_door_panel, mass 0.001; collision box size=1.999 0.199 1.999; visual box size=1.999 0.199 1.999
- added link link_44_fixed_door_panel.001, mass 0.001; visual box size=1.999 0.199 1.999
- added link link_45_fixed_door_handle, mass 0.001; collision box size=0.199 0.049 0.199; visual box size=0.199 0.049 0.199
- added link link_45_fixed_door_handle.001, mass 0.001; visual box size=0.199 0.049 0.199
- added link link_50_fixed_handle_shaft, mass 0.001; collision cylinder length=0.999 radius=0.0995; visual cylinder length=0.999 radius=0.0995
- added link link_51_fixed_handle_knob, mass 0.001; collision box size=0.049 0.049 0.199; visual box size=0.049 0.049 0.199
- added link link_52_fixed_hinge, mass 0.001; visual cylinder length=1.099 radius=0.0495
- added link link_54_fixed_handle_shaft, mass 0.001; collision box size=0.199 0.199 0.999; visual box size=0.199 0.199 0.999
- added link link_55_fixed_handle_knob, mass 0.001; collision box size=0.049 0.049 0.199; visual box size=0.049 0.049 0.199
- added link link_57_fixed_hinge, mass 0.001; visual cylinder length=2.099 radius=0.0495
- added link link_58_fixed_door_panel, mass 0.001; collision box size=3.999 0.199 1.999; visual box size=3.999 0.199 1.999
- added link link_59_fixed_door_handle, mass 0.001; collision box size=0.199 0.049 0.199; visual box size=0.199 0.049 0.199
- link link_47_fixed_handle_shaft: geometry collision box size=0.199 0.199 0.999; visual box size=0.199 0.199 0.999
Joints:
- removed joint link_40_fixed_hinge
- removed joint link_40_fixed_hinge.001
- removed joint link_41_fixed_door_panel
- removed joint link_41_fixed_door_panel.001
- removed joint link_42_fixed_door_handle
- removed joint link_42_fixed_door_handle.001
- removed joint link_44_fixed_handle_shaft
- removed joint link_45_fixed_handle_knob
- removed joint link_49_fixed_hinge
- removed joint link_51_fixed_handle_shaft
- removed joint link_52_fixed_handle_knob
- removed joint link_54_fixed_hinge
- removed joint link_55_fixed_door_panel
- removed joint link_56_fixed_door_handle
- added joint link_43_fixed_hinge: type fixed, parent link_0_joint_0, child link_43_fixed_hinge, origin xyz=0 0 0 rpy=0 0 0
- added joint link_43_fixed_hinge.001: type fixed, parent goal, child link_43_fixed_hinge.001, origin xyz=0 0 0 rpy=0 0 0
- added joint link_44_fixed_door_panel: type fixed, parent link_0_joint_0, child link_44_fixed_door_panel, origin xyz=1.0 0 0 rpy=0 0 0
- added joint link_44_fixed_door_panel.001: type fixed, parent goal, child link_44_fixed_door_panel.001, origin xyz=1.0 0 0 rpy=0 0 0
- added joint link_45_fixed_door_handle: type fixed, parent link_0_joint_0, child link_45_fixed_door_handle, origin xyz=1.5 0 1.1 rpy=0 0 0
- added joint link_45_fixed_door_handle.001: type fixed, parent goal, child link_45_fixed_door_handle.001, origin xyz=1.5 0 1.1 rpy=0 0 0
- added joint link_50_fixed_handle_shaft: type fixed, parent link_2_joint_0, child link_50_fixed_handle_shaft, origin xyz=0 1.5 1.0 rpy=0 0 0
- added joint link_51_fixed_handle_knob: type fixed, parent link_50_fixed_handle_shaft, child link_51_fixed_handle_knob, origin xyz=0 0 0.6 rpy=0 0 0
- added joint link_52_fixed_hinge: type fixed, parent link_2_joint_0, child link_52_fixed_hinge, origin xyz=0 0 0 rpy=0 0 0
- added joint link_54_fixed_handle_shaft: type fixed, parent link_3_joint_0, child link_54_fixed_handle_shaft, origin xyz=0 -1.0 0 rpy=1.5708 0 0
- added joint link_55_fixed_handle_knob: type fixed, parent link_54_fixed_handle_shaft, child link_55_fixed_handle_knob, origin xyz=0 0 0.6 rpy=0 0 0
- added joint link_57_fixed_hinge: type fixed, parent link_4_joint_0, child link_57_fixed_hinge, origin xyz=0 0 0 rpy=0 0 0
- added joint link_58_fixed_door_panel: type fixed, parent link_4_joint_0, child link_58_fixed_door_panel, origin xyz=2.0 0 0 rpy=0 0 0
- added joint link_59_fixed_door_handle: type fixed, parent link_4_joint_0, child link_59_fixed_door_handle, origin xyz=3.0 0 1.1 rpy=0 0 0
- joint link_47_fixed_handle_shaft: origin xyz=0 1.5 1.0 rpy=0 0 0 -> xyz=0 -1.0 0 rpy=1.5708 0 0; parent link_2_joint_0 -> link_1_joint_0

File: puzzles/lockbox_random/urdf/lockbox_random.urdf (robot description, URDF)
Before this commit: robot lockbox_random, 21 links, 20 joints
Links:
- removed link link_58_fixed_handle_shaft
- removed link link_58_fixed_handle_shaft.001
- removed link link_59_fixed_handle_knob
- removed link link_59_fixed_handle_knob.001
- removed link link_63_fixed_hinge
- removed link link_65_fixed_handle_shaft
- removed link link_66_fixed_handle_knob
- removed link link_70_fixed_hinge
- removed link link_72_fixed_handle_shaft
- removed link link_73_fixed_handle_knob
- added link link_61_fixed_handle_shaft.001, mass 0.001; visual box size=0.199 0.199 0.999
- added link link_62_fixed_handle_knob.001, mass 0.001; visual box size=0.049 0.049 0.199
- added link link_64_fixed_handle_shaft, mass 0.001; collision cylinder length=0.999 radius=0.0995; visual cylinder length=0.999 radius=0.0995
- added link link_65_fixed_handle_knob, mass 0.001; collision box size=0.049 0.049 0.199; visual box size=0.049 0.049 0.199
- added link link_66_fixed_hinge, mass 0.001; visual cylinder length=1.099 radius=0.0495
- added link link_71_fixed_handle_shaft, mass 0.001; collision cylinder length=0.999 radius=0.0995; visual cylinder length=0.999 radius=0.0995
- added link link_72_fixed_handle_knob, mass 0.001; collision box size=0.049 0.049 0.199; visual box size=0.049 0.049 0.199
- added link link_73_fixed_hinge, mass 0.001; visual cylinder length=1.099 radius=0.0495
- added link link_75_fixed_handle_shaft, mass 0.001; collision box size=0.199 0.199 0.999; visual box size=0.199 0.199 0.999
- added link link_76_fixed_handle_knob, mass 0.001; collision box size=0.049 0.049 0.199; visual box size=0.049 0.049 0.199
- link link_61_fixed_handle_shaft: geometry collision box size=0.199 0.199 0.999; visual box size=0.199 0.199 0.999
- link link_68_fixed_handle_shaft: geometry collision box size=0.199 0.199 0.999; visual box size=0.199 0.199 0.999
Joints:
- removed joint link_58_fixed_handle_shaft
- removed joint link_58_fixed_handle_shaft.001
- removed joint link_59_fixed_handle_knob
- removed joint link_59_fixed_handle_knob.001
- removed joint link_63_fixed_hinge
- removed joint link_65_fixed_handle_shaft
- removed joint link_66_fixed_handle_knob
- removed joint link_70_fixed_hinge
- removed joint link_72_fixed_handle_shaft
- removed joint link_73_fixed_handle_knob
- added joint link_61_fixed_handle_shaft.001: type fixed, parent goal, child link_61_fixed_handle_shaft.001, origin xyz=-1.0 0 0 rpy=0 -1.5708 0
- added joint link_62_fixed_handle_knob.001: type fixed, parent link_61_fixed_handle_shaft.001, child link_62_fixed_handle_knob.001, origin xyz=0 0 0.6 rpy=0 0 0
- added joint link_64_fixed_handle_shaft: type fixed, parent link_1_joint_0, child link_64_fixed_handle_shaft, origin xyz=0 1.125 1.0 rpy=0 0 0
- added joint link_65_fixed_handle_knob: type fixed, parent link_64_fixed_handle_shaft, child link_65_fixed_handle_knob, origin xyz=0 0 0.6 rpy=0 0 0
- added joint link_66_fixed_hinge: type fixed, parent link_1_joint_0, child link_66_fixed_hinge, origin xyz=0 0 0 rpy=0 0 0
- added joint link_71_fixed_handle_shaft: type fixed, parent link_3_joint_0, child link_71_fixed_handle_shaft, origin xyz=0 1.125 1.0 rpy=0 0 0
- added joint link_72_fixed_handle_knob: type fixed, parent link_71_fixed_handle_shaft, child link_72_fixed_handle_knob, origin xyz=0 0 0.6 rpy=0 0 0
- added joint link_73_fixed_hinge: type fixed, parent link_3_joint_0, child link_73_fixed_hinge, origin xyz=0 0 0 rpy=0 0 0
- added joint link_75_fixed_handle_shaft: type fixed, parent link_4_joint_0, child link_75_fixed_handle_shaft, origin xyz=-1.0 0 0 rpy=-0.01294 -1.5708 0.01294
- added joint link_76_fixed_handle_knob: type fixed, parent link_75_fixed_handle_shaft, child link_76_fixed_handle_knob, origin xyz=0 0 0.6 rpy=0 0 0
- joint link_61_fixed_handle_shaft: origin xyz=0 1.125 1.0 rpy=0 0 0 -> xyz=-1.0 0 0 rpy=0 -1.5708 0; parent link_1_joint_0 -> link_0_joint_0
- joint link_68_fixed_handle_shaft: origin xyz=0 1.125 1.0 rpy=0 0 0 -> xyz=-1.0 0 0 rpy=-0.06577 -1.5708 0.06577; parent link_3_joint_0 -> link_2_joint_0

File: puzzles/move_twice/urdf/move_twice.urdf (robot description, URDF)
Before this commit: robot move_twice, 14 links, 13 joints
Links:
- removed link link_89_fixed_hinge
- removed link link_89_fixed_hinge.001
- removed link link_90_fixed_wall_left
- removed link link_91_fixed_wall_right
- removed link link_92_fixed_wall_mid
- removed link link_93_fixed_wall_back
- added link link_100_fixed_wall_back, mass 0.001; collision box size=0.199 5.999 0.999; visual box size=0.199 5.999 0.999
- added link link_96_fixed_hinge, mass 0.001; visual cylinder length=1.099 radius=0.0495
- added link link_96_fixed_hinge.001, mass 0.001; visual cylinder length=1.099 radius=0.0495
- added link link_97_fixed_wall_left, mass 0.001; collision box size=3.999 0.199 0.999; visual box size=3.999 0.199 0.999
- added link link_98_fixed_wall_right, mass 0.001; collision box size=3.999 0.199 0.999; visual box size=3.999 0.199 0.999
- added link link_99_fixed_wall_mid, mass 0.001; collision box size=3.999 0.199 0.999; visual box size=3.999 0.199 0.999
Joints:
- removed joint link_89_fixed_hinge
- removed joint link_89_fixed_hinge.001
- removed joint link_90_fixed_wall_left
- removed joint link_91_fixed_wall_right
- removed joint link_92_fixed_wall_mid
- removed joint link_93_fixed_wall_back
- added joint link_100_fixed_wall_back: type fixed, parent base_link, child link_100_fixed_wall_back, origin xyz=-2.1 1.5 0.6 rpy=0 0 0
- added joint link_96_fixed_hinge: type fixed, parent link_0_joint_0, child link_96_fixed_hinge, origin xyz=0 0 0 rpy=0 0 0
- added joint link_96_fixed_hinge.001: type fixed, parent link_0_joint_0.001, child link_96_fixed_hinge.001, origin xyz=0 0 0 rpy=0 0 0
- added joint link_97_fixed_wall_left: type fixed, parent base_link, child link_97_fixed_wall_left, origin xyz=0 -1.4 0.6 rpy=0 0 0
- added joint link_98_fixed_wall_right: type fixed, parent base_link, child link_98_fixed_wall_right, origin xyz=0 4.4 0.6 rpy=0 0 0
- added joint link_99_fixed_wall_mid: type fixed, parent base_link, child link_99_fixed_wall_mid, origin xyz=0 1.5 0.6 rpy=0 0 0
