Commit message: fix (minor): add joint_count, base_object to reset()

File: puzzles/continuous_space/urdf/continuous_space.urdf (robot description, URDF)
Before this commit: robot continuous_space, 19 links, 18 joints
Links:
- removed link link_19_fixed_handle_shaft
- removed link link_19_fixed_handle_shaft.001
- removed link link_20_fixed_handle_knob
- removed link link_20_fixed_handle_knob.001
- removed link link_21_fixed_hinge
- removed link link_21_fixed_hinge.001
- removed link link_27_fixed_handle_shaft
- removed link link_28_fixed_handle_knob
- removed link link_29_fixed_hinge
- removed link link_31_fixed_handle_shaft
- removed link link_32_fixed_handle_knob
- removed link link_40_fixed_handle_shaft
- removed link link_41_fixed_handle_knob
- added link link_10_fixed_handle_knob, mass 0.001; collision box size=0.049 0.049 0.199; visual box size=0.049 0.049 0.199
- added link link_11_fixed_hinge, mass 0.001; visual cylinder length=1.099 radius=0.0495
- added link link_13_fixed_handle_shaft, mass 0.001; collision box size=0.199 0.199 0.999; visual box size=0.199 0.199 0.999
- added link link_14_fixed_handle_knob, mass 0.001; collision box size=0.049 0.049 0.199; visual box size=0.049 0.049 0.199
- added link link_1_fixed_handle_shaft, mass 0.001; collision cylinder length=0.999 radius=0.0995; visual cylinder length=0.999 radius=0.0995
- added link link_1_fixed_handle_shaft.001, mass 0.001; visual cylinder length=0.999 radius=0.0995
- added link link_22_fixed_handle_shaft, mass 0.001; collision box size=0.199 0.199 0.999; visual box size=0.199 0.199 0.999
- added link link_23_fixed_handle_knob, mass 0.001; collision box size=0.049 0.049 0.199; visual box size=0.049 0.049 0.199
- added link link_2_fixed_handle_knob, mass 0.001; collision box size=0.049 0.049 0.199; visual box size=0.049 0.049 0.199
- added link link_2_fixed_handle_knob.001, mass 0.001; visual box size=0.049 0.049 0.199
- added link link_3_fixed_hinge, mass 0.001; visual cylinder length=1.099 radius=0.0495
- added link link_3_fixed_hinge.001, mass 0.001; visual cylinder length=1.099 radius=0.0495
- added link link_9_fixed_handle_shaft, mass 0.001; collision cylinder length=0.999 radius=0.0995; visual cylinder length=0.999 radius=0.0995
Joints:
- removed joint link_19_fixed_handle_shaft
- removed joint link_19_fixed_handle_shaft.001
- removed joint link_20_fixed_handle_knob
- removed joint link_20_fixed_handle_knob.001
- removed joint link_21_fixed_hinge
- removed joint link_21_fixed_hinge.001
- removed joint link_27_fixed_handle_shaft
- removed joint link_28_fixed_handle_knob
- removed joint link_29_fixed_hinge
- removed joint link_31_fixed_handle_shaft
- removed joint link_32_fixed_handle_knob
- removed joint link_40_fixed_handle_shaft
- removed joint link_41_fixed_handle_knob
- added joint link_10_fixed_handle_knob: type fixed, parent link_9_fixed_handle_shaft, child link_10_fixed_handle_knob, origin xyz=0 0 0.6 rpy=0 0 0
- added joint link_11_fixed_hinge: type fixed, parent link_1_joint_0, child link_11_fixed_hinge, origin xyz=0 0 0 rpy=0 0 0
- added joint link_13_fixed_handle_shaft: type fixed, parent link_2_joint_0, child link_13_fixed_handle_shaft, origin xyz=0 -1.0 0 rpy=1.5708 0 0
- added joint link_14_fixed_handle_knob: type fixed, parent link_13_fixed_handle_shaft, child link_14_fixed_handle_knob, origin xyz=0 0 0.6 rpy=0 0 0
- added joint link_1_fixed_handle_shaft: type fixed, parent link_0_joint_0, child link_1_fixed_handle_shaft, origin xyz=1.125 0 1.0 rpy=0 0 0
- added joint link_1_fixed_handle_shaft.001: type fixed, parent goal, child link_1_fixed_handle_shaft.001, origin xyz=1.125 0 1.0 rpy=0 0 0
- added joint link_22_fixed_handle_shaft: type fixed, parent link_3_joint_0, child link_22_fixed_handle_shaft, origin xyz=0 -1.0 0 rpy=1.5708 0 0
- added joint link_23_fixed_handle_knob: type fixed, parent link_22_fixed_handle_shaft, child link_23_fixed_handle_knob, origin xyz=0 0 0.6 rpy=0 0 0
- added joint link_2_fixed_handle_knob: type fixed, parent link_1_fixed_handle_shaft, child link_2_fixed_handle_knob, origin xyz=0 0 0.6 rpy=0 0 0
- added joint link_2_fixed_handle_knob.001: type fixed, parent link_1_fixed_handle_shaft.001, child link_2_fixed_handle_knob.001, origin xyz=0 0 0.6 rpy=0 0 0
- added joint link_3_fixed_hinge: type fixed, parent link_0_joint_0, child link_3_fixed_hinge, origin xyz=0 0 0 rpy=0 0 0
- added joint link_3_fixed_hinge.001: type fixed, parent goal, child link_3_fixed_hinge.001, origin xyz=0 0 0 rpy=0 0 0
- added joint link_9_fixed_handle_shaft: type fixed, parent link_1_joint_0, child link_9_fixed_handle_shaft, origin xyz=1.125 0 1.0 rpy=0 0 0

File: puzzles/escape_room/urdf/escape_room.urdf (robot description, URDF)
Before this commit: robot escape_room, 21 links, 20 joints
Links:
- removed link link_80_fixed_hinge
- removed link link_80_fixed_hinge.001
- removed link link_84_fixed_hinge
- removed link link_86_fixed_hinge
- removed link link_87_fixed_door_panel
- removed link link_88_fixed_door_handle1
- removed link link_89_fixed_door_handle2
- removed link link_90_fixed_wall_left
- removed link link_91_fixed_wall_front
- removed link link_92_fixed_wall_back
- added link link_10_fixed_door_panel, mass 0.001; collision box size=2.999 0.199 0.999; visual box size=2.999 0.199 0.999
- added link link_11_fixed_door_handle1, mass 0.001; collision box size=0.049 0.199 0.199; visual box size=0.049 0.199 0.199
- added link link_12_fixed_door_handle2, mass 0.001; collision box size=0.049 0.199 0.199; visual box size=0.049 0.199 0.199
- added link link_13_fixed_wall_left, mass 0.001; collision box size=3.799 0.199 0.249; visual box size=3.799 0.199 0.249
- added link link_14_fixed_wall_front, mass 0.001; collision box size=0.199 7.999 0.249; visual box size=0.199 7.999 0.249
- added link link_15_fixed_wall_back, mass 0.001; collision box size=0.199 7.999 0.249; visual box size=0.199 7.999 0.249
- added link link_3_fixed_hinge, mass 0.001; visual cylinder length=1.099 radius=0.0495
- added link link_3_fixed_hinge.001, mass 0.001; visual cylinder length=1.099 radius=0.0495
- added link link_7_fixed_hinge, mass 0.001; visual cylinder length=0.349 radius=0.0495
- added link link_9_fixed_hinge, mass 0.001; visual cylinder length=1.099 radius=0.0495
Joints:
- removed joint link_80_fixed_hinge
- removed joint link_80_fixed_hinge.001
- removed joint link_84_fixed_hinge
- removed joint link_86_fixed_hinge
- removed joint link_87_fixed_door_panel
- removed joint link_88_fixed_door_handle1
- removed joint link_89_fixed_door_handle2
- removed joint link_90_fixed_wall_left
- removed joint link_91_fixed_wall_front
- removed joint link_92_fixed_wall_back
- added joint link_10_fixed_door_panel: type fixed, parent link_2_joint_0, child link_10_fixed_door_panel, origin xyz=1.5 0 0 rpy=0 0 0
- added joint link_11_fixed_door_handle1: type fixed, parent link_2_joint_0, child link_11_fixed_door_handle1, origin xyz=2.25 0.2 0 rpy=0 0 0
- added joint link_12_fixed_door_handle2: type fixed, parent link_2_joint_0, child link_12_fixed_door_handle2, origin xyz=2.25 -0.2 0 rpy=0 0 0
- added joint link_13_fixed_wall_left: type fixed, parent base_link, child link_13_fixed_wall_left, origin xyz=0 -4.0 0.225 rpy=0 0 0
- added joint link_14_fixed_wall_front: type fixed, parent base_link, child link_14_fixed_wall_front, origin xyz=2.0 0 0.225 rpy=0 0 0
- added joint link_15_fixed_wall_back: type fixed, parent base_link, child link_15_fixed_wall_back, origin xyz=-2.0 0 0.225 rpy=0 0 0
- added joint link_3_fixed_hinge: type fixed, parent link_0_joint_0, child link_3_fixed_hinge, origin xyz=0 0 0 rpy=0 0 0
- added joint link_3_fixed_hinge.001: type fixed, parent link_0_joint_0.001, child link_3_fixed_hinge.001, origin xyz=0 0 0 rpy=0 0 0
- added joint link_7_fixed_hinge: type fixed, parent link_1_joint_0, child link_7_fixed_hinge, origin xyz=0 0 0 rpy=0 0 0
- added joint link_9_fixed_hinge: type fixed, parent link_2_joint_0, child link_9_fixed_hinge, origin xyz=0 0 0 rpy=0 0 0

File: puzzles/grid_world/urdf/grid_world.urdf (robot description, URDF)
Before this commit: robot grid_world, 19 links, 18 joints
Links:
- removed link link_11_fixed_hinge
- removed link link_13_fixed_handle_shaft
- removed link link_14_fixed_handle_knob
- removed link link_16_fixed_handle_shaft
- removed link link_17_fixed_handle_knob
- removed link link_5_fixed_handle_shaft.001
- removed link link_6_fixed_handle_knob.001
- removed link link_7_fixed_hinge.001
- added link link_12_fixed_handle_shaft, mass 0.001; collision box size=0.199 0.199 0.999; visual box size=0.199 0.199 0.999
- added link link_13_fixed_handle_knob, mass 0.001; collision box size=0.049 0.049 0.199; visual box size=0.049 0.049 0.199
- added link link_1_fixed_handle_shaft, mass 0.001; collision cylinder length=0.999 radius=0.0995; visual cylinder length=0.999 radius=0.0995
- added link link_1_fixed_handle_shaft.001, mass 0.001; visual cylinder length=0.999 radius=0.0995
- added link link_2_fixed_handle_knob, mass 0.001; collision box size=0.049 0.049 0.199; visual box size=0.049 0.049 0.199
- added link link_2_fixed_handle_knob.001, mass 0.001; visual box size=0.049 0.049 0.199
- added link link_3_fixed_hinge, mass 0.001; visual cylinder length=0.999 radius=0.0495
- added link link_3_fixed_hinge.001, mass 0.001; visual cylinder length=0.999 radius=0.0495
- link link_9_fixed_handle_shaft: geometry collision box size=0.199 0.199 0.999; visual box size=0.199 0.199 0.999
Joints:
- removed joint link_11_fixed_hinge
- removed joint link_13_fixed_handle_shaft
- removed joint link_14_fixed_handle_knob
- removed joint link_16_fixed_handle_shaft
- removed joint link_17_fixed_handle_knob
- removed joint link_5_fixed_handle_shaft.001
- removed joint link_6_fixed_handle_knob.001
- removed joint link_7_fixed_hinge.001
- added joint link_12_fixed_handle_shaft: type fixed, parent link_3_joint_0, child link_12_fixed_handle_shaft, origin xyz=0 0.95 0 rpy=-1.5708 0 0
- added joint link_13_fixed_handle_knob: type fixed, parent link_12_fixed_handle_shaft, child link_13_fixed_handle_knob, origin xyz=0 0 0.6 rpy=0 0 0
- added joint link_1_fixed_handle_shaft: type fixed, parent link_0_joint_0, child link_1_fixed_handle_shaft, origin xyz=1.0875 0 0.95 rpy=0 0 0
- added joint link_1_fixed_handle_shaft.001: type fixed, parent goal, child link_1_fixed_handle_shaft.001, origin xyz=1.0875 0 0.95 rpy=0 0 0
- added joint link_2_fixed_handle_knob: type fixed, parent link_1_fixed_handle_shaft, child link_2_fixed_handle_knob, origin xyz=0 0 0.6 rpy=0 0 0
- added joint link_2_fixed_handle_knob.001: type fixed, parent link_1_fixed_handle_shaft.001, child link_2_fixed_handle_knob.001, origin xyz=0 0 0.6 rpy=0 0 0
- added joint link_3_fixed_hinge: type fixed, parent link_0_joint_0, child link_3_fixed_hinge, origin xyz=0 0 0 rpy=0 0 0
- added joint link_3_fixed_hinge.001: type fixed, parent goal, child link_3_fixed_hinge.001, origin xyz=0 0 0 rpy=0 0 0
- joint link_5_fixed_handle_shaft: parent link_0_joint_0 -> link_1_joint_0
- joint link_7_fixed_hinge: parent link_0_joint_0 -> link_1_joint_0
- joint link_9_fixed_handle_shaft: origin xyz=1.0875 0 0.95 rpy=0 0 0 -> xyz=-0.95 0 0 rpy=0 -1.5708 0; parent link_1_joint_0 -> link_2_joint_0

File: puzzles/lockbox2017/urdf/lockbox2017.urdf (robot description, URDF)
Before this commit: robot lockbox2017, 23 links, 22 joints
Links:
- removed link link_43_fixed_hinge
- removed link link_43_fixed_hinge.001
- removed link link_44_fixed_door_panel
- removed link link_44_fixed_door_panel.001
- removed link link_45_fixed_door_handle
- removed link link_45_fixed_door_handle.001
- removed link link_47_fixed_handle_shaft
- removed link link_48_fixed_handle_knob
- removed link link_50_fixed_handle_shaft
- removed link link_51_fixed_handle_knob
- removed link link_52_fixed_hinge
- removed link link_54_fixed_handle_shaft
- removed link link_55_fixed_handle_knob
- removed link link_57_fixed_hinge
- removed link link_58_fixed_door_panel
- removed link link_59_fixed_door_handle
- added link link_10_fixed_hinge, mass 0.001; visual cylinder length=1.099 radius=0.0495
- added link link_12_fixed_handle_shaft, mass 0.001; collision box size=0.199 0.199 0.999; visual box size=0.199 0.199 0.999
- added link link_13_fixed_handle_knob, mass 0.001; collision box size=0.049 0.049 0.199; visual box size=0.049 0.049 0.199
- added link link_15_fixed_hinge, mass 0.001; visual cylinder length=2.099 radius=0.0495
- added link link_16_fixed_door_panel, mass 0.001; collision box size=3.999 0.199 1.999; visual box size=3.999 0.199 1.999
- added link link_17_fixed_door_handle, mass 0.001; collision box size=0.199 0.049 0.199; visual box size=0.199 0.049 0.199
- added link link_1_fixed_hinge, mass 0.001; visual cylinder length=2.099 radius=0.0495
- added link link_1_fixed_hinge.001, mass 0.001; visual cylinder length=2.099 radius=0.0495
- added link link_2_fixed_door_panel, mass 0.001; collision box size=1.999 0.199 1.999; visual box size=1.999 0.199 1.999
- added link link_2_fixed_door_panel.001, mass 0.001; visual box size=1.999 0.199 1.999
- added link link_3_fixed_door_handle, mass 0.001; collision box size=0.199 0.049 0.199; visual box size=0.199 0.049 0.199
- added link link_3_fixed_door_handle.001, mass 0.001; visual box size=0.199 0.049 0.199
- added link link_5_fixed_handle_shaft, mass 0.001; collision box size=0.199 0.199 0.999; visual box size=0.199 0.199 0.999
- added link link_6_fixed_handle_knob, mass 0.001; collision box size=0.049 0.049 0.199; visual box size=0.049 0.049 0.199
- added link link_8_fixed_handle_shaft, mass 0.001; collision cylinder length=0.999 radius=0.0995; visual cylinder length=0.999 radius=0.0995
- added link link_9_fixed_handle_knob, mass 0.001; collision box size=0.049 0.049 0.199; visual box size=0.049 0.049 0.199
Joints:
- removed joint link_43_fixed_hinge
- removed joint link_43_fixed_hinge.001
- removed joint link_44_fixed_door_panel
- removed joint link_44_fixed_door_panel.001
- removed joint link_45_fixed_door_handle
- removed joint link_45_fixed_door_handle.001
- removed joint link_47_fixed_handle_shaft
- removed joint link_48_fixed_handle_knob
- removed joint link_50_fixed_handle_shaft
- removed joint link_51_fixed_handle_knob
- removed joint link_52_fixed_hinge
- removed joint link_54_fixed_handle_shaft
- removed joint link_55_fixed_handle_knob
- removed joint link_57_fixed_hinge
- removed joint link_58_fixed_door_panel
- removed joint link_59_fixed_door_handle
- added joint link_10_fixed_hinge: type fixed, parent link_2_joint_0, child link_10_fixed_hinge, origin xyz=0 0 0 rpy=0 0 0
- added joint link_12_fixed_handle_shaft: type fixed, parent link_3_joint_0, child link_12_fixed_handle_shaft, origin xyz=0 -1.0 0 rpy=1.5708 0 0
- added joint link_13_fixed_handle_knob: type fixed, parent link_12_fixed_handle_shaft, child link_13_fixed_handle_knob, origin xyz=0 0 0.6 rpy=0 0 0
- added joint link_15_fixed_hinge: type fixed, parent link_4_joint_0, child link_15_fixed_hinge, origin xyz=0 0 0 rpy=0 0 0
- added joint link_16_fixed_door_panel: type fixed, parent link_4_joint_0, child link_16_fixed_door_panel, origin xyz=2.0 0 0 rpy=0 0 0
- added joint link_17_fixed_door_handle: type fixed, parent link_4_joint_0, child link_17_fixed_door_handle, origin xyz=3.0 0 1.1 rpy=0 0 0
- added joint link_1_fixed_hinge: type fixed, parent link_0_joint_0, child link_1_fixed_hinge, origin xyz=0 0 0 rpy=0 0 0
- added joint link_1_fixed_hinge.001: type fixed, parent goal, child link_1_fixed_hinge.001, origin xyz=0 0 0 rpy=0 0 0
- added joint link_2_fixed_door_panel: type fixed, parent link_0_joint_0, child link_2_fixed_door_panel, origin xyz=1.0 0 0 rpy=0 0 0
- added joint link_2_fixed_door_panel.001: type fixed, parent goal, child link_2_fixed_door_panel.001, origin xyz=1.0 0 0 rpy=0 0 0
- added joint link_3_fixed_door_handle: type fixed, parent link_0_joint_0, child link_3_fixed_door_handle, origin xyz=1.5 0 1.1 rpy=0 0 0
- added joint link_3_fixed_door_handle.001: type fixed, parent goal, child link_3_fixed_door_handle.001, origin xyz=1.5 0 1.1 rpy=0 0 0
- added joint link_5_fixed_handle_shaft: type fixed, parent link_1_joint_0, child link_5_fixed_handle_shaft, origin xyz=0 -1.0 0 rpy=1.5708 0 0
- added joint link_6_fixed_handle_knob: type fixed, parent link_5_fixed_handle_shaft, child link_6_fixed_handle_knob, origin xyz=0 0 0.6 rpy=0 0 0
- added joint link_8_fixed_handle_shaft: type fixed, parent link_2_joint_0, child link_8_fixed_handle_shaft, origin xyz=0 1.5 1.0 rpy=0 0 0
- added joint link_9_fixed_handle_knob: type fixed, parent link_8_fixed_handle_shaft, child link_9_fixed_handle_knob, origin xyz=0 0 0.6 rpy=0 0 0

File: puzzles/lockbox_random/urdf/lockbox_random.urdf (robot description, URDF)
Before this commit: robot lockbox_random, 21 links, 20 joints
Links:
- removed link link_61_fixed_handle_shaft
- removed link link_61_fixed_handle_shaft.001
- removed link link_62_fixed_handle_knob
- removed link link_62_fixed_handle_knob.001
- removed link link_64_fixed_handle_shaft
- removed link link_65_fixed_handle_knob
- removed link link_66_fixed_hinge
- removed link link_68_fixed_handle_shaft
- removed link link_69_fixed_handle_knob
- removed link link_71_fixed_handle_shaft
- removed link link_72_fixed_handle_knob
- removed link link_73_fixed_hinge
- removed link link_75_fixed_handle_shaft
- removed link link_76_fixed_handle_knob
- added link link_11_fixed_handle_shaft, mass 0.001; collision cylinder length=0.999 radius=0.0995; visual cylinder length=0.999 radius=0.0995
- added link link_12_fixed_handle_knob, mass 0.001; collision box size=0.049 0.049 0.199; visual box size=0.049 0.049 0.199
- added link link_13_fixed_hinge, mass 0.001; visual cylinder length=1.099 radius=0.0495
- added link link_15_fixed_handle_shaft, mass 0.001; collision box size=0.199 0.199 0.999; visual box size=0.199 0.199 0.999
- added link link_16_fixed_handle_knob, mass 0.001; collision box size=0.049 0.049 0.199; visual box size=0.049 0.049 0.199
- added link link_1_fixed_handle_shaft, mass 0.001; collision box size=0.199 0.199 0.999; visual box size=0.199 0.199 0.999
- added link link_1_fixed_handle_shaft.001, mass 0.001; visual box size=0.199 0.199 0.999
- added link link_2_fixed_handle_knob, mass 0.001; collision box size=0.049 0.049 0.199; visual box size=0.049 0.049 0.199
- added link link_2_fixed_handle_knob.001, mass 0.001; visual box size=0.049 0.049 0.199
- added link link_4_fixed_handle_shaft, mass 0.001; collision cylinder length=0.999 radius=0.0995; visual cylinder length=0.999 radius=0.0995
- added link link_5_fixed_handle_knob, mass 0.001; collision box size=0.049 0.049 0.199; visual box size=0.049 0.049 0.199
- added link link_6_fixed_hinge, mass 0.001; visual cylinder length=1.099 radius=0.0495
- added link link_8_fixed_handle_shaft, mass 0.001; collision box size=0.199 0.199 0.999; visual box size=0.199 0.199 0.999
- added link link_9_fixed_handle_knob, mass 0.001; collision box size=0.049 0.049 0.199; visual box size=0.049 0.049 0.199
Joints:
- removed joint link_61_fixed_handle_shaft
- removed joint link_61_fixed_handle_shaft.001
- removed joint link_62_fixed_handle_knob
- removed joint link_62_fixed_handle_knob.001
- removed joint link_64_fixed_handle_shaft
- removed joint link_65_fixed_handle_knob
- removed joint link_66_fixed_hinge
- removed joint link_68_fixed_handle_shaft
- removed joint link_69_fixed_handle_knob
- removed joint link_71_fixed_handle_shaft
- removed joint link_72_fixed_handle_knob
- removed joint link_73_fixed_hinge
- removed joint link_75_fixed_handle_shaft
- removed joint link_76_fixed_handle_knob
- added joint link_11_fixed_handle_shaft: type fixed, parent link_3_joint_0, child link_11_fixed_handle_shaft, origin xyz=0 1.125 1.0 rpy=0 0 0
- added joint link_12_fixed_handle_knob: type fixed, parent link_11_fixed_handle_shaft, child link_12_fixed_handle_knob, origin xyz=0 0 0.6 rpy=0 0 0
- added joint link_13_fixed_hinge: type fixed, parent link_3_joint_0, child link_13_fixed_hinge, origin xyz=0 0 0 rpy=0 0 0
- added joint link_15_fixed_handle_shaft: type fixed, parent link_4_joint_0, child link_15_fixed_handle_shaft, origin xyz=-1.0 0 0 rpy=-0.01294 -1.5708 0.01294
- added joint link_16_fixed_handle_knob: type fixed, parent link_15_fixed_handle_shaft, child link_16_fixed_handle_knob, origin xyz=0 0 0.6 rpy=0 0 0
- added joint link_1_fixed_handle_shaft: type fixed, parent link_0_joint_0, child link_1_fixed_handle_shaft, origin xyz=-1.0 0 0 rpy=0 -1.5708 0
- added joint link_1_fixed_handle_shaft.001: type fixed, parent goal, child link_1_fixed_handle_shaft.001, origin xyz=-1.0 0 0 rpy=0 -1.5708 0
- added joint link_2_fixed_handle_knob: type fixed, parent link_1_fixed_handle_shaft, child link_2_fixed_handle_knob, origin xyz=0 0 0.6 rpy=0 0 0
- added joint link_2_fixed_handle_knob.001: type fixed, parent link_1_fixed_handle_shaft.001, child link_2_fixed_handle_knob.001, origin xyz=0 0 0.6 rpy=0 0 0
- added joint link_4_fixed_handle_shaft: type fixed, parent link_1_joint_0, child link_4_fixed_handle_shaft, origin xyz=0 1.125 1.0 rpy=0 0 0
- added joint link_5_fixed_handle_knob: type fixed, parent link_4_fixed_handle_shaft, child link_5_fixed_handle_knob, origin xyz=0 0 0.6 rpy=0 0 0
- added joint link_6_fixed_hinge: type fixed, parent link_1_joint_0, child link_6_fixed_hinge, origin xyz=0 0 0 rpy=0 0 0
- added joint link_8_fixed_handle_shaft: type fixed, parent link_2_joint_0, child link_8_fixed_handle_shaft, origin xyz=-1.0 0 0 rpy=-0.06577 -1.5708 0.06577
- added joint link_9_fixed_handle_knob: type fixed, parent link_8_fixed_handle_shaft, child link_9_fixed_handle_knob, origin xyz=0 0 0.6 rpy=0 0 0
