Commit message: fix (minor): add joint_count, base_object to reset()

File: puzzles/move_twice/urdf/move_twice.urdf (robot description, URDF)
Before this commit: robot move_twice, 14 links, 13 joints
Links:
- removed link link_100_fixed_wall_back
- removed link link_96_fixed_hinge
- removed link link_96_fixed_hinge.001
- removed link link_97_fixed_wall_left
- removed link link_98_fixed_wall_right
- removed link link_99_fixed_wall_mid
- added link link_3_fixed_hinge, mass 0.001; visual cylinder length=1.099 radius=0.0495
- added link link_3_fixed_hinge.001, mass 0.001; visual cylinder length=1.099 radius=0.0495
- added link link_4_fixed_wall_left, mass 0.001; collision box size=3.999 0.199 0.999; visual box size=3.999 0.199 0.999
- added link link_5_fixed_wall_right, mass 0.001; collision box size=3.999 0.199 0.999; visual box size=3.999 0.199 0.999
- added link link_6_fixed_wall_mid, mass 0.001; collision box size=3.999 0.199 0.999; visual box size=3.999 0.199 0.999
- added link link_7_fixed_wall_back, mass 0.001; collision box size=0.199 5.999 0.999; visual box size=0.199 5.999 0.999
Joints:
- removed joint link_100_fixed_wall_back
- removed joint link_96_fixed_hinge
- removed joint link_96_fixed_hinge.001
- removed joint link_97_fixed_wall_left
- removed joint link_98_fixed_wall_right
- removed joint link_99_fixed_wall_mid
- added joint link_3_fixed_hinge: type fixed, parent link_0_joint_0, child link_3_fixed_hinge, origin xyz=0 0 0 rpy=0 0 0
- added joint link_3_fixed_hinge.001: type fixed, parent link_0_joint_0.001, child link_3_fixed_hinge.001, origin xyz=0 0 0 rpy=0 0 0
- added joint link_4_fixed_wall_left: type fixed, parent base_link, child link_4_fixed_wall_left, origin xyz=0 -1.4 0.6 rpy=0 0 0
- added joint link_5_fixed_wall_right: type fixed, parent base_link, child link_5_fixed_wall_right, origin xyz=0 4.4 0.6 rpy=0 0 0
- added joint link_6_fixed_wall_mid: type fixed, parent base_link, child link_6_fixed_wall_mid, origin xyz=0 1.5 0.6 rpy=0 0 0
- added joint link_7_fixed_wall_back: type fixed, parent base_link, child link_7_fixed_wall_back, origin xyz=-2.1 1.5 0.6 rpy=0 0 0

Commit message: feat: global scaling in config

File: puzzles/continuous_space/urdf/continuous_space.urdf (robot description, URDF)
Before this commit: robot continuous_space, 19 links, 18 joints
Links:
- link link_11_fixed_hinge: geometry visual cylinder length=1.099 radius=0.1245
- link link_3_fixed_hinge: geometry visual cylinder length=1.099 radius=0.1245
- link link_3_fixed_hinge.001: geometry visual cylinder length=1.099 radius=0.1245

File: puzzles/escape_room/urdf/escape_room.urdf (robot description, URDF)
Before this commit: robot escape_room, 21 links, 20 joints
Links:
- link link_3_fixed_hinge: geometry visual cylinder length=1.099 radius=0.09325
- link link_3_fixed_hinge.001: geometry visual cylinder length=1.099 radius=0.09325
- link link_7_fixed_hinge: geometry visual cylinder length=0.274 radius=0.0245

File: puzzles/grid_world/urdf/grid_world.urdf (robot description, URDF)
Before this commit: robot grid_world, 19 links, 18 joints
Links:
- link link_3_fixed_hinge: geometry visual cylinder length=0.989 radius=0.112
- link link_3_fixed_hinge.001: geometry visual cylinder length=0.989 radius=0.112
- link link_7_fixed_hinge: geometry visual cylinder length=0.989 radius=0.112

File: puzzles/lockbox2017/urdf/lockbox2017.urdf (robot description, URDF)
Before this commit: robot lockbox2017, 23 links, 22 joints
Links:
- link link_10_fixed_hinge: geometry visual cylinder length=1.099 radius=0.4995
- link link_15_fixed_hinge: geometry visual cylinder length=2.199 radius=0.0495
- link link_1_fixed_hinge: geometry visual cylinder length=2.199 radius=0.0495
- link link_1_fixed_hinge.001: geometry visual cylinder length=2.199 radius=0.0495

File: puzzles/lockbox_random/urdf/lockbox_random.urdf (robot description, URDF)
Before this commit: robot lockbox_random, 21 links, 20 joints
Links:
- link link_13_fixed_hinge: geometry visual cylinder length=1.099 radius=0.3745
- link link_6_fixed_hinge: geometry visual cylinder length=1.099 radius=0.3745

File: puzzles/move_twice/urdf/move_twice.urdf (robot description, URDF)
Before this commit: robot move_twice, 14 links, 13 joints
Links:
- link link_3_fixed_hinge: geometry visual cylinder length=1.099 radius=0.09325
- link link_3_fixed_hinge.001: geometry visual cylinder length=1.099 radius=0.09325

Commit message: refactor: z-axis always pointing up

File: puzzles/continuous_space/urdf/continuous_space.urdf (robot description, URDF)
Before this commit: robot continuous_space, 19 links, 18 joints
Links:
- removed link link_10_fixed_handle_knob
- removed link link_11_fixed_hinge
- removed link link_1_fixed_handle_shaft
- removed link link_1_fixed_handle_shaft.001
- removed link link_22_fixed_handle_shaft
- removed link link_23_fixed_handle_knob
- removed link link_2_fixed_handle_knob
- removed link link_2_fixed_handle_knob.001
- removed link link_3_fixed_hinge
- removed link link_3_fixed_hinge.001
- removed link link_9_fixed_handle_shaft
- added link link_10_fixed_handle_shaft, mass 0.001; collision cylinder length=0.999 radius=0.0995; visual cylinder length=0.999 radius=0.0995
- added link link_11_fixed_handle_knob, mass 0.001; collision box size=0.049 0.049 0.199; visual box size=0.049 0.049 0.199
- added link link_19_fixed_handle_shaft, mass 0.001; collision box size=0.199 0.199 0.999; visual box size=0.199 0.199 0.999
- added link link_1_fixed_hinge, mass 0.001; visual cylinder length=1.099 radius=0.1245
- added link link_1_fixed_hinge.001, mass 0.001; visual cylinder length=1.099 radius=0.1245
- added link link_20_fixed_handle_knob, mass 0.001; collision box size=0.049 0.049 0.199; visual box size=0.049 0.049 0.199
- added link link_2_fixed_handle_shaft, mass 0.001; collision cylinder length=0.999 radius=0.0995; visual cylinder length=0.999 radius=0.0995
- added link link_2_fixed_handle_shaft.001, mass 0.001; visual cylinder length=0.999 radius=0.0995
- added link link_3_fixed_handle_knob, mass 0.001; collision box size=0.049 0.049 0.199; visual box size=0.049 0.049 0.199
- added link link_3_fixed_handle_knob.001, mass 0.001; visual box size=0.049 0.049 0.199
- added link link_9_fixed_hinge, mass 0.001; visual cylinder length=1.099 radius=0.1245
- link link_2_joint_0: geometry collision box size=1.999 0.999 0.999; visual box size=1.999 0.999 0.999
- link link_3_joint_0: geometry collision box size=1.999 0.999 0.999; visual box size=1.999 0.999 0.999
Joints:
- removed joint link_10_fixed_handle_knob
- removed joint link_11_fixed_hinge
- removed joint link_1_fixed_handle_shaft
- removed joint link_1_fixed_handle_shaft.001
- removed joint link_22_fixed_handle_shaft
- removed joint link_23_fixed_handle_knob
- removed joint link_2_fixed_handle_knob
- removed joint link_2_fixed_handle_knob.001
- removed joint link_3_fixed_hinge
- removed joint link_3_fixed_hinge.001
- removed joint link_9_fixed_handle_shaft
- added joint link_10_fixed_handle_shaft: type fixed, parent link_1_joint_0, child link_10_fixed_handle_shaft, origin xyz=1.125 0 1.0 rpy=0 0 0
- added joint link_11_fixed_handle_knob: type fixed, parent link_10_fixed_handle_shaft, child link_11_fixed_handle_knob, origin xyz=0 0 0.6 rpy=0 0 0
- added joint link_19_fixed_handle_shaft: type fixed, parent link_3_joint_0, child link_19_fixed_handle_shaft, origin xyz=0 0 1.0 rpy=0 0 0
- added joint link_1_fixed_hinge: type fixed, parent link_0_joint_0, child link_1_fixed_hinge, origin xyz=0 0 0 rpy=0 0 0
- added joint link_1_fixed_hinge.001: type fixed, parent goal, child link_1_fixed_hinge.001, origin xyz=0 0 0 rpy=0 0 0
- added joint link_20_fixed_handle_knob: type fixed, parent link_19_fixed_handle_shaft, child link_20_fixed_handle_knob, origin xyz=0 0 0.6 rpy=0 0 0
- added joint link_2_fixed_handle_shaft: type fixed, parent link_0_joint_0, child link_2_fixed_handle_shaft, origin xyz=1.125 0 1.0 rpy=0 0 0
- added joint link_2_fixed_handle_shaft.001: type fixed, parent goal, child link_2_fixed_handle_shaft.001, origin xyz=1.125 0 1.0 rpy=0 0 0
- added joint link_3_fixed_handle_knob: type fixed, parent link_2_fixed_handle_shaft, child link_3_fixed_handle_knob, origin xyz=0 0 0.6 rpy=0 0 0
- added joint link_3_fixed_handle_knob.001: type fixed, parent link_2_fixed_handle_shaft.001, child link_3_fixed_handle_knob.001, origin xyz=0 0 0.6 rpy=0 0 0
- added joint link_9_fixed_hinge: type fixed, parent link_1_joint_0, child link_9_fixed_hinge, origin xyz=0 0 0 rpy=0 0 0
- joint link_13_fixed_handle_shaft: origin xyz=0 -1.0 0 rpy=1.5708 0 0 -> xyz=0 0 1.0 rpy=0 0 0
- joint link_2_joint_0: axis 0 0 1.0 -> 1.0 0 0; origin xyz=2.7436 -0.22317 0.6 rpy=-1.5708 0 -2.39786 -> xyz=2.7436 -0.22317 0.6 rpy=0 0 -0.82706
- joint link_3_joint_0: axis 0 0 1.0 -> 1.0 0 0; limit lower=0 upper=3.93321 effort=0 velocity=0 -> lower=0 upper=2.2014 effort=0 velocity=0; origin xyz=3.51572 -2.56206 0.6 rpy=-1.5708 0 -2.44487 -> xyz=5.40312 -1.16807 0.6 rpy=0 0 -0.41479

File: puzzles/escape_room/urdf/escape_room.urdf (robot description, URDF)
Before this commit: robot escape_room, 21 links, 20 joints
Joints:
- joint link_1_joint_2: origin xyz=0 3.30215 0.225 rpy=0 0 0 -> xyz=0 3.07216 0.225 rpy=0 0 0

File: puzzles/grid_world/urdf/grid_world.urdf (robot description, URDF)
Before this commit: robot grid_world, 19 links, 18 joints
Links:
- removed link link_1_fixed_handle_shaft
- removed link link_1_fixed_handle_shaft.001
- removed link link_2_fixed_handle_knob
- removed link link_2_fixed_handle_knob.001
- removed link link_3_fixed_hinge
- removed link link_3_fixed_hinge.001
- removed link link_5_fixed_handle_shaft
- removed link link_6_fixed_handle_knob
- removed link link_7_fixed_hinge
- added link link_1_fixed_hinge, mass 0.001; visual cylinder length=0.989 radius=0.112
- added link link_1_fixed_hinge.001, mass 0.001; visual cylinder length=0.989 radius=0.112
- added link link_2_fixed_handle_shaft, mass 0.001; collision cylinder length=0.999 radius=0.0995; visual cylinder length=0.999 radius=0.0995
- added link link_2_fixed_handle_shaft.001, mass 0.001; visual cylinder length=0.999 radius=0.0995
- added link link_3_fixed_handle_knob, mass 0.001; collision box size=0.049 0.049 0.199; visual box size=0.049 0.049 0.199
- added link link_3_fixed_handle_knob.001, mass 0.001; visual box size=0.049 0.049 0.199
- added link link_5_fixed_hinge, mass 0.001; visual cylinder length=0.989 radius=0.112
- added link link_6_fixed_handle_shaft, mass 0.001; collision cylinder length=0.999 radius=0.0995; visual cylinder length=0.999 radius=0.0995
- added link link_7_fixed_handle_knob, mass 0.001; collision box size=0.049 0.049 0.199; visual box size=0.049 0.049 0.199
- link link_2_joint_0: geometry collision box size=1.899 0.899 0.899; visual box size=1.899 0.899 0.899
- link link_3_joint_0: geometry collision box size=1.899 0.899 0.899; visual box size=1.899 0.899 0.899
Joints:
- removed joint link_1_fixed_handle_shaft
- removed joint link_1_fixed_handle_shaft.001
- removed joint link_2_fixed_handle_knob
- removed joint link_2_fixed_handle_knob.001
- removed joint link_3_fixed_hinge
- removed joint link_3_fixed_hinge.001
- removed joint link_5_fixed_handle_shaft
- removed joint link_6_fixed_handle_knob
- removed joint link_7_fixed_hinge
- added joint link_1_fixed_hinge: type fixed, parent link_0_joint_0, child link_1_fixed_hinge, origin xyz=0 0 0 rpy=0 0 0
- added joint link_1_fixed_hinge.001: type fixed, parent goal, child link_1_fixed_hinge.001, origin xyz=0 0 0 rpy=0 0 0
- added joint link_2_fixed_handle_shaft: type fixed, parent link_0_joint_0, child link_2_fixed_handle_shaft, origin xyz=1.0875 0 0.95 rpy=0 0 0
- added joint link_2_fixed_handle_shaft.001: type fixed, parent goal, child link_2_fixed_handle_shaft.001, origin xyz=1.0875 0 0.95 rpy=0 0 0
- added joint link_3_fixed_handle_knob: type fixed, parent link_2_fixed_handle_shaft, child link_3_fixed_handle_knob, origin xyz=0 0 0.6 rpy=0 0 0
- added joint link_3_fixed_handle_knob.001: type fixed, parent link_2_fixed_handle_shaft.001, child link_3_fixed_handle_knob.001, origin xyz=0 0 0.6 rpy=0 0 0
- added joint link_5_fixed_hinge: type fixed, parent link_1_joint_0, child link_5_fixed_hinge, origin xyz=0 0 0 rpy=0 0 0
- added joint link_6_fixed_handle_shaft: type fixed, parent link_1_joint_0, child link_6_fixed_handle_shaft, origin xyz=1.0875 0 0.95 rpy=0 0 0
- added joint link_7_fixed_handle_knob: type fixed, parent link_6_fixed_handle_shaft, child link_7_fixed_handle_knob, origin xyz=0 0 0.6 rpy=0 0 0
- joint link_12_fixed_handle_shaft: origin xyz=0 0.95 0 rpy=-1.5708 0 0 -> xyz=0 0 0.95 rpy=0 0 0
- joint link_2_joint_0: axis 0 0 1.0 -> 1.0 0 0; origin xyz=1.0 1.5 0.55 rpy=0 1.5708 0 -> xyz=1.0 1.5 0.55 rpy=0 0 0
- joint link_3_joint_0: axis 0 0 1.0 -> 1.0 0 0; origin xyz=-1.5 -2.0 0.55 rpy=1.5708 0 0 -> xyz=-1.5 -2.0 0.55 rpy=0 0 -1.5708
- joint link_9_fixed_handle_shaft: origin xyz=-0.95 0 0 rpy=0 -1.5708 0 -> xyz=0 0 0.95 rpy=0 0 0

File: puzzles/lockbox2017/urdf/lockbox2017.urdf (robot description, URDF)
Before this commit: robot lockbox2017, 23 links, 22 joints
Links:
- removed link link_10_fixed_hinge
- removed link link_8_fixed_handle_shaft
- removed link link_9_fixed_handle_knob
- added link link_10_fixed_handle_knob, mass 0.001; collision box size=0.049 0.049 0.199; visual box size=0.049 0.049 0.199
- added link link_8_fixed_hinge, mass 0.001; visual cylinder length=1.099 radius=0.4995
- added link link_9_fixed_handle_shaft, mass 0.001; collision cylinder length=0.999 radius=0.0995; visual cylinder length=0.999 radius=0.0995
- link link_1_joint_0: geometry collision box size=3.599 0.799 0.999; visual box size=3.599 0.799 0.999
- link link_3_joint_0: geometry collision box size=3.599 0.799 0.999; visual box size=3.599 0.799 0.999
Joints:
- removed joint link_10_fixed_hinge
- removed joint link_8_fixed_handle_shaft
- removed joint link_9_fixed_handle_knob
- added joint link_10_fixed_handle_knob: type fixed, parent link_9_fixed_handle_shaft, child link_10_fixed_handle_knob, origin xyz=0 0 0.6 rpy=0 0 0
- added joint link_8_fixed_hinge: type fixed, parent link_2_joint_0, child link_8_fixed_hinge, origin xyz=0 0 0 rpy=0 0 0
- added joint link_9_fixed_handle_shaft: type fixed, parent link_2_joint_0, child link_9_fixed_handle_shaft, origin xyz=0 1.5 1.0 rpy=0 0 0
- joint link_12_fixed_handle_shaft: origin xyz=0 -1.0 0 rpy=1.5708 0 0 -> xyz=0 0 1.0 rpy=0 0 0
- joint link_1_joint_0: axis 0 0 1.0 -> 1.0 0 0; origin xyz=-4.0 0 0.6 rpy=-1.5708 0 -1.5708 -> xyz=-4.0 0 0.6 rpy=0 0 0
- joint link_3_joint_0: axis 0 0 1.0 -> 1.0 0 0; origin xyz=0 2.0 0.6 rpy=-1.5708 0 0 -> xyz=0 2.0 0.6 rpy=0 0 1.5708
- joint link_5_fixed_handle_shaft: origin xyz=0 -1.0 0 rpy=1.5708 0 0 -> xyz=0 0 1.0 rpy=0 0 0

File: puzzles/lockbox_random/urdf/lockbox_random.urdf (robot description, URDF)
Before this commit: robot lockbox_random, 21 links, 20 joints
Links:
- removed link link_11_fixed_handle_shaft
- removed link link_12_fixed_handle_knob
- removed link link_13_fixed_hinge
- removed link link_4_fixed_handle_shaft
- removed link link_5_fixed_handle_knob
- removed link link_6_fixed_hinge
- added link link_11_fixed_hinge, mass 0.001; visual cylinder length=1.099 radius=0.3745
- added link link_12_fixed_handle_shaft, mass 0.001; collision cylinder length=0.999 radius=0.0995; visual cylinder length=0.999 radius=0.0995
- added link link_13_fixed_handle_knob, mass 0.001; collision box size=0.049 0.049 0.199; visual box size=0.049 0.049 0.199
- added link link_4_fixed_hinge, mass 0.001; visual cylinder length=1.099 radius=0.3745
- added link link_5_fixed_handle_shaft, mass 0.001; collision cylinder length=0.999 radius=0.0995; visual cylinder length=0.999 radius=0.0995
- added link link_6_fixed_handle_knob, mass 0.001; collision box size=0.049 0.049 0.199; visual box size=0.049 0.049 0.199
- link goal: geometry visual box size=1.399 0.199 0.999
- link link_0_joint_0: geometry collision box size=1.399 0.199 0.999; visual box size=1.399 0.199 0.999
- link link_2_joint_0: geometry collision box size=1.399 0.199 0.999; visual box size=1.399 0.199 0.999
- link link_4_joint_0: geometry collision box size=1.399 0.199 0.999; visual box size=1.399 0.199 0.999
Joints:
- removed joint link_11_fixed_handle_shaft
- removed joint link_12_fixed_handle_knob
- removed joint link_13_fixed_hinge
- removed joint link_4_fixed_handle_shaft
- removed joint link_5_fixed_handle_knob
- removed joint link_6_fixed_hinge
- added joint link_11_fixed_hinge: type fixed, parent link_3_joint_0, child link_11_fixed_hinge, origin xyz=0 0 0 rpy=0 0 0
- added joint link_12_fixed_handle_shaft: type fixed, parent link_3_joint_0, child link_12_fixed_handle_shaft, origin xyz=0 1.125 1.0 rpy=0 0 0
- added joint link_13_fixed_handle_knob: type fixed, parent link_12_fixed_handle_shaft, child link_13_fixed_handle_knob, origin xyz=0 0 0.6 rpy=0 0 0
- added joint link_4_fixed_hinge: type fixed, parent link_1_joint_0, child link_4_fixed_hinge, origin xyz=0 0 0 rpy=0 0 0
- added joint link_5_fixed_handle_shaft: type fixed, parent link_1_joint_0, child link_5_fixed_handle_shaft, origin xyz=0 1.125 1.0 rpy=0 0 0
- added joint link_6_fixed_handle_knob: type fixed, parent link_5_fixed_handle_shaft, child link_6_fixed_handle_knob, origin xyz=0 0 0.6 rpy=0 0 0
- joint goal: origin xyz=-1.0 0.5 0.6 rpy=0 1.5708 0 -> xyz=-1.0 0.5 0.6 rpy=0 0 0
- joint link_0_joint_0: axis 0 0 1.0 -> 1.0 0 0; origin xyz=-2.0 0.5 0.6 rpy=0 1.5708 0 -> xyz=-2.0 0.5 0.6 rpy=0 0 0
- joint link_15_fixed_handle_shaft: origin xyz=-1.0 0 0 rpy=-0.01294 -1.5708 0.01294 -> xyz=0 0 1.0 rpy=0 0 0
- joint link_1_fixed_handle_shaft: origin xyz=-1.0 0 0 rpy=0 -1.5708 0 -> xyz=0 0 1.0 rpy=0 0 0
- joint link_1_fixed_handle_shaft.001: origin xyz=-1.0 0 0 rpy=0 -1.5708 0 -> xyz=0 0 1.0 rpy=0 0 0
- joint link_2_joint_0: axis 0 0 1.0 -> 1.0 0 0; origin xyz=0.5 2.0 0.6 rpy=0 1.5708 1.5708 -> xyz=0.5 2.0 0.6 rpy=0 0 1.5708
- joint link_4_joint_0: axis 0 0 1.0 -> 1.0 0 0; origin xyz=-1.0 4.5 0.6 rpy=-3.14159 1.57079 0 -> xyz=-1.0 4.5 0.6 rpy=0 0 3.14159
- joint link_8_fixed_handle_shaft: origin xyz=-1.0 0 0 rpy=-0.06577 -1.5708 0.06577 -> xyz=0 0 1.0 rpy=0 0 0

File: puzzles/simple_sliders/urdf/simple_sliders.urdf (robot description, URDF)
Before this commit: robot simple_sliders, 6 links, 5 joints
Links:
- link goal: geometry visual box size=1.599 0.199 0.199
- link link_0_joint_0: geometry collision box size=1.599 0.199 0.199; visual box size=1.599 0.199 0.199
- link link_1_joint_0: geometry collision box size=1.599 0.199 0.199; visual box size=1.599 0.199 0.199
- link link_2_joint_0: geometry collision box size=1.599 0.199 0.199; visual box size=1.599 0.199 0.199
- link link_3_joint_0: geometry collision box size=1.599 0.199 0.199; visual box size=1.599 0.199 0.199
Joints:
- joint goal: origin xyz=0 -1.0 0.2 rpy=1.5708 0 0 -> xyz=0 -1.0 0.2 rpy=0 0 -1.5708
- joint link_0_joint_0: axis 0 0 1.0 -> 1.0 0 0; origin xyz=0 0 0.2 rpy=1.5708 0 0 -> xyz=0 0 0.2 rpy=0 0 -1.5708
- joint link_1_joint_0: axis 0 0 1.0 -> 1.0 0 0; origin xyz=0 -1.0 0.2 rpy=0 1.5708 0 -> xyz=0 -1.0 0.2 rpy=0 0 0
- joint link_2_joint_0: axis 0 0 1.0 -> 1.0 0 0; origin xyz=1.0 -1.0 0.2 rpy=1.5708 0 0 -> xyz=1.0 -1.0 0.2 rpy=0 0 -1.5708
- joint link_3_joint_0: axis 0 0 1.0 -> 1.0 0 0; origin xyz=1.0 -2.0 0.2 rpy=0 1.5708 0 -> xyz=1.0 -2.0 0.2 rpy=0 0 0
