Commit message: chore (minor): use appropriate hinge_diameter

File: puzzles/continuous_space/urdf/continuous_space.urdf (robot description, URDF)
Before this commit: robot continuous_space, 19 links, 18 joints
Links:
- removed link link_19_fixed_handle_shaft
- removed link link_20_fixed_handle_knob
- added link link_22_fixed_handle_shaft, mass 0.001; collision box size=0.199 0.199 0.999; visual box size=0.199 0.199 0.999
- added link link_23_fixed_handle_knob, mass 0.001; collision box size=0.049 0.049 0.199; visual box size=0.049 0.049 0.199
Joints:
- removed joint link_19_fixed_handle_shaft
- removed joint link_20_fixed_handle_knob
- added joint link_22_fixed_handle_shaft: type fixed, parent link_3_joint_0, child link_22_fixed_handle_shaft, origin xyz=0 0 1.0 rpy=0 0 0
- added joint link_23_fixed_handle_knob: type fixed, parent link_22_fixed_handle_shaft, child link_23_fixed_handle_knob, origin xyz=0 0 0.6 rpy=0 0 0
- joint link_3_joint_0: limit lower=0 upper=2.2014 effort=0 velocity=0 -> lower=0 upper=3.93321 effort=0 velocity=0; origin xyz=5.40312 -1.16807 0.6 rpy=0 0 -0.41479 -> xyz=3.51572 -2.56206 0.6 rpy=0 0 -0.87407

File: puzzles/escape_room/urdf/escape_room.urdf (robot description, URDF)
Before this commit: robot escape_room, 21 links, 20 joints
Links:
- removed link link_10_fixed_door_panel
- removed link link_11_fixed_door_handle1
- removed link link_12_fixed_door_handle2
- removed link link_13_fixed_wall_left
- removed link link_14_fixed_wall_front
- removed link link_15_fixed_wall_back
- removed link link_3_fixed_hinge
- removed link link_3_fixed_hinge.001
- removed link link_9_fixed_hinge
- added link link_10_fixed_door_handle2, mass 0.001; collision box size=0.049 0.199 0.199; visual box size=0.049 0.199 0.199
- added link link_11_fixed_wall_left, mass 0.001; collision box size=3.799 0.199 0.249; visual box size=3.799 0.199 0.249
- added link link_12_fixed_wall_front, mass 0.001; collision box size=0.199 7.999 0.249; visual box size=0.199 7.999 0.249
- added link link_13_fixed_wall_back, mass 0.001; collision box size=0.199 7.999 0.249; visual box size=0.199 7.999 0.249
- added link link_8_fixed_door_panel, mass 0.001; collision box size=3.199 0.199 0.999; visual box size=3.199 0.199 0.999
- added link link_9_fixed_door_handle1, mass 0.001; collision box size=0.049 0.199 0.199; visual box size=0.049 0.199 0.199
- link link_7_fixed_hinge: geometry visual cylinder length=1.099 radius=0.0495
Joints:
- removed joint link_10_fixed_door_panel
- removed joint link_11_fixed_door_handle1
- removed joint link_12_fixed_door_handle2
- removed joint link_13_fixed_wall_left
- removed joint link_14_fixed_wall_front
- removed joint link_15_fixed_wall_back
- removed joint link_3_fixed_hinge
- removed joint link_3_fixed_hinge.001
- removed joint link_9_fixed_hinge
- added joint link_10_fixed_door_handle2: type fixed, parent link_2_joint_0, child link_10_fixed_door_handle2, origin xyz=2.4 -0.2 0 rpy=0 0 0
- added joint link_11_fixed_wall_left: type fixed, parent base_link, child link_11_fixed_wall_left, origin xyz=0 -4.0 0.225 rpy=0 0 0
- added joint link_12_fixed_wall_front: type fixed, parent base_link, child link_12_fixed_wall_front, origin xyz=2.0 0 0.225 rpy=0 0 0
- added joint link_13_fixed_wall_back: type fixed, parent base_link, child link_13_fixed_wall_back, origin xyz=-2.0 0 0.225 rpy=0 0 0
- added joint link_8_fixed_door_panel: type fixed, parent link_2_joint_0, child link_8_fixed_door_panel, origin xyz=1.6 0 0 rpy=0 0 0
- added joint link_9_fixed_door_handle1: type fixed, parent link_2_joint_0, child link_9_fixed_door_handle1, origin xyz=2.4 0.2 0 rpy=0 0 0
- joint link_7_fixed_hinge: parent link_1_joint_0 -> link_2_joint_0

File: puzzles/lockbox2017/urdf/lockbox2017.urdf (robot description, URDF)
Before this commit: robot lockbox2017, 23 links, 22 joints
Links:
- link link_8_fixed_hinge: geometry visual cylinder length=1.099 radius=0.1245

File: puzzles/lockbox_random/urdf/lockbox_random.urdf (robot description, URDF)
Before this commit: robot lockbox_random, 21 links, 20 joints
Links:
- link link_11_fixed_hinge: geometry visual cylinder length=1.099 radius=0.1245
- link link_4_fixed_hinge: geometry visual cylinder length=1.099 radius=0.1245

File: puzzles/move_twice/urdf/move_twice.urdf (robot description, URDF)
Before this commit: robot move_twice, 14 links, 13 joints
Links:
- removed link link_3_fixed_hinge
- removed link link_3_fixed_hinge.001
- removed link link_4_fixed_wall_left
- removed link link_5_fixed_wall_right
- removed link link_6_fixed_wall_mid
- removed link link_7_fixed_wall_back
- added link link_3_fixed_wall_left, mass 0.001; collision box size=3.999 0.199 0.999; visual box size=3.999 0.199 0.999
- added link link_4_fixed_wall_right, mass 0.001; collision box size=3.999 0.199 0.999; visual box size=3.999 0.199 0.999
- added link link_5_fixed_wall_mid, mass 0.001; collision box size=3.999 0.199 0.999; visual box size=3.999 0.199 0.999
- added link link_6_fixed_wall_back, mass 0.001; collision box size=0.199 5.999 0.999; visual box size=0.199 5.999 0.999
Joints:
- removed joint link_3_fixed_hinge
- removed joint link_3_fixed_hinge.001
- removed joint link_4_fixed_wall_left
- removed joint link_5_fixed_wall_right
- removed joint link_6_fixed_wall_mid
- removed joint link_7_fixed_wall_back
- added joint link_3_fixed_wall_left: type fixed, parent base_link, child link_3_fixed_wall_left, origin xyz=0 -1.4 0.6 rpy=0 0 0
- added joint link_4_fixed_wall_right: type fixed, parent base_link, child link_4_fixed_wall_right, origin xyz=0 4.4 0.6 rpy=0 0 0
- added joint link_5_fixed_wall_mid: type fixed, parent base_link, child link_5_fixed_wall_mid, origin xyz=0 1.5 0.6 rpy=0 0 0
- added joint link_6_fixed_wall_back: type fixed, parent base_link, child link_6_fixed_wall_back, origin xyz=-2.1 1.5 0.6 rpy=0 0 0

Commit message: refactor: use stick mesh for obstacle add param concave_collision_mesh to export() minor renaming

File: puzzles/continuous_space/urdf/continuous_space.urdf (robot description, URDF)
Before this commit: robot continuous_space, 19 links, 18 joints
Links:
- removed link link_22_fixed_handle_shaft
- removed link link_23_fixed_handle_knob
- added link link_19_fixed_handle_shaft, mass 0.001; collision box size=0.199 0.199 0.999; visual box size=0.199 0.199 0.999
- added link link_20_fixed_handle_knob, mass 0.001; collision box size=0.049 0.049 0.199; visual box size=0.049 0.049 0.199
Joints:
- removed joint link_22_fixed_handle_shaft
- removed joint link_23_fixed_handle_knob
- added joint link_19_fixed_handle_shaft: type fixed, parent link_3_joint_0, child link_19_fixed_handle_shaft, origin xyz=0 0 1.0 rpy=0 0 0
- added joint link_20_fixed_handle_knob: type fixed, parent link_19_fixed_handle_shaft, child link_20_fixed_handle_knob, origin xyz=0 0 0.6 rpy=0 0 0
- joint link_3_joint_0: limit lower=0 upper=3.93321 effort=0 velocity=0 -> lower=0 upper=2.2014 effort=0 velocity=0; origin xyz=3.51572 -2.56206 0.6 rpy=0 0 -0.87407 -> xyz=5.40312 -1.16807 0.6 rpy=0 0 -0.41479

File: puzzles/escape_room/urdf/escape_room.urdf (robot description, URDF)
Before this commit: robot escape_room, 18 links, 17 joints
Links:
- link link_11_fixed_wall_left: geometry collision box size=3.799 0.199 0.499; visual box size=3.799 0.199 0.499
- link link_12_fixed_wall_front: geometry collision box size=0.199 7.999 0.499; visual box size=0.199 7.999 0.499
- link link_13_fixed_wall_back: geometry collision box size=0.199 7.999 0.499; visual box size=0.199 7.999 0.499
- link link_1_joint_0: geometry collision mesh filename=file:///home/userone/ba/puzzle-generator/puzzles/escape_roo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 scale=1.0 1.0 1.0; visual mesh filename=file:///home/userone/ba/puzzle-generator/puzzles/escape_roo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 scale=1.0 1.0 1.0
Joints:
- joint link_11_fixed_wall_left: origin xyz=0 -4.0 0.225 rpy=0 0 0 -> xyz=0 -4.0 0.35 rpy=0 0 0
- joint link_12_fixed_wall_front: origin xyz=2.0 0 0.225 rpy=0 0 0 -> xyz=2.0 0 0.35 rpy=0 0 0
- joint link_13_fixed_wall_back: origin xyz=-2.0 0 0.225 rpy=0 0 0 -> xyz=-2.0 0 0.35 rpy=0 0 0
- joint link_1_joint_2: origin xyz=0 3.07216 0.225 rpy=0 0 0 -> xyz=-0.75 2.68884 0.35 rpy=0 0 0

Commit message: refactor: ContinuousSpaceSampler * outer loop: attempts, inner loop: attempts_per_link * new start points on both sides of revolute link * pybullet solve() call not verbose (ompl still is)

File: puzzles/continuous_space/urdf/continuous_space.urdf (robot description, URDF)
Before this commit: robot continuous_space, 19 links, 18 joints
Links:
- removed link link_10_fixed_handle_shaft
- removed link link_11_fixed_handle_knob
- removed link link_19_fixed_handle_shaft
- removed link link_1_fixed_hinge
- removed link link_1_fixed_hinge.001
- removed link link_20_fixed_handle_knob
- removed link link_2_fixed_handle_shaft
- removed link link_2_fixed_handle_shaft.001
- removed link link_3_fixed_handle_knob
- removed link link_3_fixed_handle_knob.001
- removed link link_9_fixed_hinge
- added link link_123_fixed_hinge, mass 0.001; visual cylinder length=1.099 radius=0.1245
- added link link_124_fixed_handle_shaft, mass 0.001; collision cylinder length=0.999 radius=0.0995; visual cylinder length=0.999 radius=0.0995
- added link link_125_fixed_handle_knob, mass 0.001; collision box size=0.049 0.049 0.199; visual box size=0.049 0.049 0.199
- added link link_151_fixed_handle_shaft, mass 0.001; collision box size=0.199 0.199 0.999; visual box size=0.199 0.199 0.999
- added link link_152_fixed_handle_knob, mass 0.001; collision box size=0.049 0.049 0.199; visual box size=0.049 0.049 0.199
- added link link_1_fixed_handle_shaft, mass 0.001; collision box size=0.199 0.199 0.999; visual box size=0.199 0.199 0.999
- added link link_1_fixed_handle_shaft.001, mass 0.001; visual box size=0.199 0.199 0.999
- added link link_2_fixed_handle_knob, mass 0.001; collision box size=0.049 0.049 0.199; visual box size=0.049 0.049 0.199
- added link link_2_fixed_handle_knob.001, mass 0.001; visual box size=0.049 0.049 0.199
- added link link_4_joint_0, mass 0.001; collision box size=1.999 0.999 0.999; visual box size=1.999 0.999 0.999
- added link link_61_fixed_hinge, mass 0.001; visual cylinder length=1.099 radius=0.1245
- added link link_62_fixed_handle_shaft, mass 0.001; collision cylinder length=0.999 radius=0.0995; visual cylinder length=0.999 radius=0.0995
- added link link_63_fixed_handle_knob, mass 0.001; collision box size=0.049 0.049 0.199; visual box size=0.049 0.049 0.199
- link goal: geometry visual box size=1.999 0.999 0.999
- link link_0_joint_0: geometry collision box size=1.999 0.999 0.999; visual box size=1.999 0.999 0.999
- link link_1_joint_0: geometry collision box size=1.999 0.999 0.999; visual box size=1.999 0.999 0.999
- link link_2_joint_0: geometry collision box size=2.999 0.999 0.999; visual box size=2.999 0.999 0.999
- link link_3_joint_0: geometry collision box size=2.999 0.999 0.999; visual box size=2.999 0.999 0.999
Joints:
- removed joint link_10_fixed_handle_shaft
- removed joint link_11_fixed_handle_knob
- removed joint link_19_fixed_handle_shaft
- removed joint link_1_fixed_hinge
- removed joint link_1_fixed_hinge.001
- removed joint link_20_fixed_handle_knob
- removed joint link_2_fixed_handle_shaft
- removed joint link_2_fixed_handle_shaft.001
- removed joint link_3_fixed_handle_knob
- removed joint link_3_fixed_handle_knob.001
- removed joint link_9_fixed_hinge
- added joint link_123_fixed_hinge: type fixed, parent link_3_joint_0, child link_123_fixed_hinge, origin xyz=0 0 0 rpy=0 0 0
- added joint link_124_fixed_handle_shaft: type fixed, parent link_3_joint_0, child link_124_fixed_handle_shaft, origin xyz=1.125 0 1.0 rpy=0 0 0
- added joint link_125_fixed_handle_knob: type fixed, parent link_124_fixed_handle_shaft, child link_125_fixed_handle_knob, origin xyz=0 0 0.6 rpy=0 0 0
- added joint link_151_fixed_handle_shaft: type fixed, parent link_4_joint_0, child link_151_fixed_handle_shaft, origin xyz=0 0 1.0 rpy=0 0 0
- added joint link_152_fixed_handle_knob: type fixed, parent link_151_fixed_handle_shaft, child link_152_fixed_handle_knob, origin xyz=0 0 0.6 rpy=0 0 0
- added joint link_1_fixed_handle_shaft: type fixed, parent link_0_joint_0, child link_1_fixed_handle_shaft, origin xyz=0 0 1.0 rpy=0 0 0
- added joint link_1_fixed_handle_shaft.001: type fixed, parent goal, child link_1_fixed_handle_shaft.001, origin xyz=0 0 1.0 rpy=0 0 0
- added joint link_2_fixed_handle_knob: type fixed, parent link_1_fixed_handle_shaft, child link_2_fixed_handle_knob, origin xyz=0 0 0.6 rpy=0 0 0
- added joint link_2_fixed_handle_knob.001: type fixed, parent link_1_fixed_handle_shaft.001, child link_2_fixed_handle_knob.001, origin xyz=0 0 0.6 rpy=0 0 0
- added joint link_4_joint_0: type prismatic, parent base_link, child link_4_joint_0, origin xyz=3.4627 -1.85032 0.6 rpy=0 0 1.59111, axis 1.0 0 0, limit lower=0 upper=3.4642 effort=0 velocity=0
- added joint link_61_fixed_hinge: type fixed, parent link_2_joint_0, child link_61_fixed_hinge, origin xyz=0 0 0 rpy=0 0 0
- added joint link_62_fixed_handle_shaft: type fixed, parent link_2_joint_0, child link_62_fixed_handle_shaft, origin xyz=1.125 0 1.0 rpy=0 0 0
- added joint link_63_fixed_handle_knob: type fixed, parent link_62_fixed_handle_shaft, child link_63_fixed_handle_knob, origin xyz=0 0 0.6 rpy=0 0 0
- joint goal: origin xyz=0 0 0.6 rpy=0 0 -2.79786 -> xyz=0.99739 -2.4812 0.6 rpy=0 0 -1.18859
- joint link_0_joint_0: axis 0 0 1.0 -> 1.0 0 0; limit lower=-1.82033 upper=0 effort=0 velocity=0 -> lower=0 upper=2.67416 effort=0 velocity=0; origin xyz=0 0 0.6 rpy=0 0 -0.97753 -> xyz=0 0 0.6 rpy=0 0 -1.18859; type revolute -> prismatic
- joint link_13_fixed_handle_shaft: parent link_2_joint_0 -> link_1_joint_0
- joint link_1_joint_0: axis 0 0 1.0 -> 1.0 0 0; limit lower=0 upper=1.58552 effort=0 velocity=0 -> lower=0 upper=3.11295 effort=0 velocity=0; origin xyz=1.89728 1.60703 0.6 rpy=0 0 -2.61769 -> xyz=-0.03422 -3.00526 0.6 rpy=0 0 -2.29454; type revolute -> prismatic
- joint link_2_joint_0: axis 1.0 0 0 -> 0 0 1.0; limit lower=0 upper=3.81949 effort=0 velocity=0 -> lower=0 upper=2.87617 effort=0 velocity=0; origin xyz=2.7436 -0.22317 0.6 rpy=0 0 -0.82706 -> xyz=-1.10798 -5.00962 0.6 rpy=0 0 -1.25698; type prismatic -> revolute
- joint link_3_joint_0: axis 1.0 0 0 -> 0 0 1.0; limit lower=0 upper=2.2014 effort=0 velocity=0 -> lower=-2.54743 upper=0 effort=0 velocity=0; origin xyz=5.40312 -1.16807 0.6 rpy=0 0 -0.41479 -> xyz=2.8631 -3.5405 0.6 rpy=0 0 -3.02217; type prismatic -> revolute

Commit message: feat (minor): shrink goal duplicate

File: puzzles/continuous_space/urdf/continuous_space.urdf (robot description, URDF)
Before this commit: robot continuous_space, 21 links, 20 joints
Links:
- link goal: geometry visual box size=1.997 0.998 0.998
- link link_1_fixed_handle_shaft.001: geometry visual box size=0.1988 0.1988 0.998
- link link_2_fixed_handle_knob.001: geometry visual box size=0.04895 0.04895 0.1988
Joints:
- joint link_1_fixed_handle_shaft.001: origin xyz=0 0 1.0 rpy=0 0 0 -> xyz=0 0 0.999 rpy=0 0 0
- joint link_2_fixed_handle_knob.001: origin xyz=0 0 0.6 rpy=0 0 0 -> xyz=0 0 0.5994 rpy=0 0 0

File: puzzles/escape_room/urdf/escape_room.urdf (robot description, URDF)
Before this commit: robot escape_room, 18 links, 17 joints
Links:
- link link_0_joint_0.001: geometry visual mesh filename=file:///home/userone/ba/puzzle-generator/puzzles/escape_roo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 scale=0.999 0.999 0.999

File: puzzles/grid_world/urdf/grid_world.urdf (robot description, URDF)
Before this commit: robot grid_world, 25 links, 24 joints
Links:
- link goal: geometry visual box size=2.8961 0.8981 0.8981
- link link_1_fixed_hinge.001: geometry visual cylinder length=0.98801 radius=0.11189
- link link_2_fixed_handle_shaft.001: geometry visual cylinder length=0.998 radius=0.0994
- link link_3_fixed_handle_knob.001: geometry visual box size=0.04895 0.04895 0.1988
Joints:
- joint link_2_fixed_handle_shaft.001: origin xyz=1.0875 0 0.95 rpy=0 0 0 -> xyz=1.08641 0 0.94905 rpy=0 0 0
- joint link_3_fixed_handle_knob.001: origin xyz=0 0 0.6 rpy=0 0 0 -> xyz=0 0 0.5994 rpy=0 0 0

File: puzzles/lockbox2017/urdf/lockbox2017.urdf (robot description, URDF)
Before this commit: robot lockbox2017, 23 links, 22 joints
Links:
- link goal: geometry visual cylinder length=1.997 radius=0.1993
- link link_1_fixed_hinge.001: geometry visual cylinder length=2.1968 radius=0.04945
- link link_2_fixed_door_panel.001: geometry visual box size=1.997 0.1988 1.997
- link link_3_fixed_door_handle.001: geometry visual box size=0.1988 0.04895 0.1988
Joints:
- joint link_2_fixed_door_panel.001: origin xyz=1.0 0 0 rpy=0 0 0 -> xyz=0.999 0 0 rpy=0 0 0
- joint link_3_fixed_door_handle.001: origin xyz=1.5 0 1.1 rpy=0 0 0 -> xyz=1.4985 0 1.0989 rpy=0 0 0

File: puzzles/lockbox_random/urdf/lockbox_random.urdf (robot description, URDF)
Before this commit: robot lockbox_random, 21 links, 20 joints
Links:
- link goal: geometry visual box size=1.3976 0.1988 0.998
- link link_1_fixed_handle_shaft.001: geometry visual box size=0.1988 0.1988 0.998
- link link_2_fixed_handle_knob.001: geometry visual box size=0.04895 0.04895 0.1988
Joints:
- joint link_1_fixed_handle_shaft.001: origin xyz=0 0 1.0 rpy=0 0 0 -> xyz=0 0 0.999 rpy=0 0 0
- joint link_2_fixed_handle_knob.001: origin xyz=0 0 0.6 rpy=0 0 0 -> xyz=0 0 0.5994 rpy=0 0 0

File: puzzles/move_twice/urdf/move_twice.urdf (robot description, URDF)
Before this commit: robot move_twice, 12 links, 11 joints
Links:
- link link_0_joint_0.001: geometry visual mesh filename=file:///home/userone/ba/puzzle-generator/puzzles/move_twice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 scale=0.999 0.999 0.999

File: puzzles/simple_sliders/urdf/simple_sliders.urdf (robot description, URDF)
Before this commit: robot simple_sliders, 16 links, 15 joints
Links:
- link goal: geometry visual box size=1.5974 0.1988 0.1988
- link link_1_fixed_handle_shaft.001: geometry visual box size=0.1988 0.1988 0.998
- link link_2_fixed_handle_knob.001: geometry visual box size=0.04895 0.04895 0.1988
Joints:
- joint link_1_fixed_handle_shaft.001: origin xyz=0 0 0.6 rpy=0 0 0 -> xyz=0 0 0.5994 rpy=0 0 0
- joint link_2_fixed_handle_knob.001: origin xyz=0 0 0.6 rpy=0 0 0 -> xyz=0 0 0.5994 rpy=0 0 0
