Commit message: refactor: separate floor from base_link

File: puzzles/continuous_space/urdf/continuous_space.urdf (robot description, URDF)
Before this commit: robot continuous_space, 21 links, 20 joints
Links:
- removed link link_123_fixed_hinge
- removed link link_124_fixed_handle_shaft
- removed link link_125_fixed_handle_knob
- removed link link_13_fixed_handle_shaft
- removed link link_14_fixed_handle_knob
- removed link link_151_fixed_handle_shaft
- removed link link_152_fixed_handle_knob
- removed link link_1_fixed_handle_shaft
- removed link link_1_fixed_handle_shaft.001
- removed link link_2_fixed_handle_knob
- removed link link_2_fixed_handle_knob.001
- removed link link_61_fixed_hinge
- removed link link_62_fixed_handle_shaft
- removed link link_63_fixed_handle_knob
- added link link_fixed_0_floor, mass 0.001; collision box size=31.999 31.999 0.199; visual box size=31.999 31.999 0.199
- added link link_fixed_124_hinge, mass 0.001; visual cylinder length=1.099 radius=0.1245
- added link link_fixed_125_handle_shaft, mass 0.001; collision cylinder length=0.999 radius=0.0995; visual cylinder length=0.999 radius=0.0995
- added link link_fixed_126_handle_knob, mass 0.001; collision box size=0.049 0.049 0.199; visual box size=0.049 0.049 0.199
- added link link_fixed_14_handle_shaft, mass 0.001; collision box size=0.199 0.199 0.999; visual box size=0.199 0.199 0.999
- added link link_fixed_152_handle_shaft, mass 0.001; collision box size=0.199 0.199 0.999; visual box size=0.199 0.199 0.999
- added link link_fixed_153_handle_knob, mass 0.001; collision box size=0.049 0.049 0.199; visual box size=0.049 0.049 0.199
- added link link_fixed_15_handle_knob, mass 0.001; collision box size=0.049 0.049 0.199; visual box size=0.049 0.049 0.199
- added link link_fixed_2_handle_shaft, mass 0.001; collision box size=0.199 0.199 0.999; visual box size=0.199 0.199 0.999
- added link link_fixed_2_handle_shaft.001, mass 0.001; visual box size=0.1988 0.1988 0.998
- added link link_fixed_3_handle_knob, mass 0.001; collision box size=0.049 0.049 0.199; visual box size=0.049 0.049 0.199
- added link link_fixed_3_handle_knob.001, mass 0.001; visual box size=0.04895 0.04895 0.1988
- added link link_fixed_62_hinge, mass 0.001; visual cylinder length=1.099 radius=0.1245
- added link link_fixed_63_handle_shaft, mass 0.001; collision cylinder length=0.999 radius=0.0995; visual cylinder length=0.999 radius=0.0995
- added link link_fixed_64_handle_knob, mass 0.001; collision box size=0.049 0.049 0.199; visual box size=0.049 0.049 0.199
- link base_link: geometry 
Joints:
- removed joint link_123_fixed_hinge
- removed joint link_124_fixed_handle_shaft
- removed joint link_125_fixed_handle_knob
- removed joint link_13_fixed_handle_shaft
- removed joint link_14_fixed_handle_knob
- removed joint link_151_fixed_handle_shaft
- removed joint link_152_fixed_handle_knob
- removed joint link_1_fixed_handle_shaft
- removed joint link_1_fixed_handle_shaft.001
- removed joint link_2_fixed_handle_knob
- removed joint link_2_fixed_handle_knob.001
- removed joint link_61_fixed_hinge
- removed joint link_62_fixed_handle_shaft
- removed joint link_63_fixed_handle_knob
- added joint link_fixed_0_floor: type fixed, parent base_link, child link_fixed_0_floor, origin xyz=0 0 -0.1 rpy=0 0 0
- added joint link_fixed_124_hinge: type fixed, parent link_3_joint_0, child link_fixed_124_hinge, origin xyz=0 0 0 rpy=0 0 0
- added joint link_fixed_125_handle_shaft: type fixed, parent link_3_joint_0, child link_fixed_125_handle_shaft, origin xyz=1.125 0 1.0 rpy=0 0 0
- added joint link_fixed_126_handle_knob: type fixed, parent link_fixed_125_handle_shaft, child link_fixed_126_handle_knob, origin xyz=0 0 0.6 rpy=0 0 0
- added joint link_fixed_14_handle_shaft: type fixed, parent link_1_joint_0, child link_fixed_14_handle_shaft, origin xyz=0 0 1.0 rpy=0 0 0
- added joint link_fixed_152_handle_shaft: type fixed, parent link_4_joint_0, child link_fixed_152_handle_shaft, origin xyz=0 0 1.0 rpy=0 0 0
- added joint link_fixed_153_handle_knob: type fixed, parent link_fixed_152_handle_shaft, child link_fixed_153_handle_knob, origin xyz=0 0 0.6 rpy=0 0 0
- added joint link_fixed_15_handle_knob: type fixed, parent link_fixed_14_handle_shaft, child link_fixed_15_handle_knob, origin xyz=0 0 0.6 rpy=0 0 0
- added joint link_fixed_2_handle_shaft: type fixed, parent link_0_joint_0, child link_fixed_2_handle_shaft, origin xyz=0 0 1.0 rpy=0 0 0
- added joint link_fixed_2_handle_shaft.001: type fixed, parent goal, child link_fixed_2_handle_shaft.001, origin xyz=0 0 0.999 rpy=0 0 0
- added joint link_fixed_3_handle_knob: type fixed, parent link_fixed_2_handle_shaft, child link_fixed_3_handle_knob, origin xyz=0 0 0.6 rpy=0 0 0
- added joint link_fixed_3_handle_knob.001: type fixed, parent link_fixed_2_handle_shaft.001, child link_fixed_3_handle_knob.001, origin xyz=0 0 0.5994 rpy=0 0 0
- added joint link_fixed_62_hinge: type fixed, parent link_2_joint_0, child link_fixed_62_hinge, origin xyz=0 0 0 rpy=0 0 0
- added joint link_fixed_63_handle_shaft: type fixed, parent link_2_joint_0, child link_fixed_63_handle_shaft, origin xyz=1.125 0 1.0 rpy=0 0 0
- added joint link_fixed_64_handle_knob: type fixed, parent link_fixed_63_handle_shaft, child link_fixed_64_handle_knob, origin xyz=0 0 0.6 rpy=0 0 0
- joint goal: origin xyz=0.99739 -2.4812 0.6 rpy=0 0 -1.18859 -> xyz=0.99739 -2.4812 0.5 rpy=0 0 -1.18859
- joint link_0_joint_0: origin xyz=0 0 0.6 rpy=0 0 -1.18859 -> xyz=0 0 0.5 rpy=0 0 -1.18859
- joint link_1_joint_0: origin xyz=-0.03422 -3.00526 0.6 rpy=0 0 -2.29454 -> xyz=-0.03422 -3.00526 0.5 rpy=0 0 -2.29454
- joint link_2_joint_0: origin xyz=-1.10798 -5.00962 0.6 rpy=0 0 -1.25698 -> xyz=-1.10798 -5.00962 0.5 rpy=0 0 -1.25698
- joint link_3_joint_0: origin xyz=2.8631 -3.5405 0.6 rpy=0 0 -3.02217 -> xyz=2.8631 -3.5405 0.5 rpy=0 0 -3.02217
- joint link_4_joint_0: origin xyz=3.4627 -1.85032 0.6 rpy=0 0 1.59111 -> xyz=3.4627 -1.85032 0.5 rpy=0 0 1.59111

File: puzzles/escape_room/urdf/escape_room.urdf (robot description, URDF)
Before this commit: robot escape_room, 18 links, 17 joints
Links:
- removed link link_10_fixed_door_handle2
- removed link link_11_fixed_wall_left
- removed link link_12_fixed_wall_front
- removed link link_13_fixed_wall_back
- removed link link_7_fixed_hinge
- removed link link_8_fixed_door_panel
- removed link link_9_fixed_door_handle1
- added link link_fixed_0_floor, mass 0.001; collision box size=31.999 31.999 0.199; visual box size=31.999 31.999 0.199
- added link link_fixed_10_door_handle1, mass 0.001; collision box size=0.049 0.199 0.199; visual box size=0.049 0.199 0.199
- added link link_fixed_11_door_handle2, mass 0.001; collision box size=0.049 0.199 0.199; visual box size=0.049 0.199 0.199
- added link link_fixed_12_wall_left, mass 0.001; collision box size=3.799 0.199 0.499; visual box size=3.799 0.199 0.499
- added link link_fixed_13_wall_front, mass 0.001; collision box size=0.199 7.999 0.499; visual box size=0.199 7.999 0.499
- added link link_fixed_14_wall_back, mass 0.001; collision box size=0.199 7.999 0.499; visual box size=0.199 7.999 0.499
- added link link_fixed_8_hinge, mass 0.001; visual cylinder length=1.099 radius=0.0495
- added link link_fixed_9_door_panel, mass 0.001; collision box size=3.199 0.199 0.999; visual box size=3.199 0.199 0.999
- link base_link: geometry 
Joints:
- removed joint link_10_fixed_door_handle2
- removed joint link_11_fixed_wall_left
- removed joint link_12_fixed_wall_front
- removed joint link_13_fixed_wall_back
- removed joint link_7_fixed_hinge
- removed joint link_8_fixed_door_panel
- removed joint link_9_fixed_door_handle1
- added joint link_fixed_0_floor: type fixed, parent base_link, child link_fixed_0_floor, origin xyz=0 0 -0.1 rpy=0 0 0
- added joint link_fixed_10_door_handle1: type fixed, parent link_2_joint_0, child link_fixed_10_door_handle1, origin xyz=2.4 0.2 0 rpy=0 0 0
- added joint link_fixed_11_door_handle2: type fixed, parent link_2_joint_0, child link_fixed_11_door_handle2, origin xyz=2.4 -0.2 0 rpy=0 0 0
- added joint link_fixed_12_wall_left: type fixed, parent base_link, child link_fixed_12_wall_left, origin xyz=0 -4.0 0.25 rpy=0 0 0
- added joint link_fixed_13_wall_front: type fixed, parent base_link, child link_fixed_13_wall_front, origin xyz=2.0 0 0.25 rpy=0 0 0
- added joint link_fixed_14_wall_back: type fixed, parent base_link, child link_fixed_14_wall_back, origin xyz=-2.0 0 0.25 rpy=0 0 0
- added joint link_fixed_8_hinge: type fixed, parent link_2_joint_0, child link_fixed_8_hinge, origin xyz=0 0 0 rpy=0 0 0
- added joint link_fixed_9_door_panel: type fixed, parent link_2_joint_0, child link_fixed_9_door_panel, origin xyz=1.6 0 0 rpy=0 0 0
- joint goal: origin xyz=0 5.0 0.6 rpy=0 0 1.5708 -> xyz=0 5.0 0.5 rpy=0 0 1.5708
- joint link_0_joint_2: origin xyz=0 0 0.6 rpy=0 0 0 -> xyz=0 0 0.5 rpy=0 0 0
- joint link_1_joint_2: origin xyz=-0.75 2.68884 0.35 rpy=0 0 0 -> xyz=-0.75 2.68884 0.25 rpy=0 0 0
- joint link_2_joint_0: origin xyz=1.5 4.0 0.6 rpy=0 0 3.14159 -> xyz=1.5 4.0 0.5 rpy=0 0 3.14159

File: puzzles/grid_world/urdf/grid_world.urdf (robot description, URDF)
Before this commit: robot grid_world, 25 links, 24 joints
Links:
- removed link link_10_fixed_handle_knob
- removed link link_12_fixed_handle_shaft
- removed link link_13_fixed_handle_knob
- removed link link_15_fixed_handle_shaft
- removed link link_16_fixed_handle_knob
- removed link link_18_fixed_handle_shaft
- removed link link_19_fixed_handle_knob
- removed link link_1_fixed_hinge
- removed link link_1_fixed_hinge.001
- removed link link_2_fixed_handle_shaft
- removed link link_2_fixed_handle_shaft.001
- removed link link_3_fixed_handle_knob
- removed link link_3_fixed_handle_knob.001
- removed link link_5_fixed_handle_shaft
- removed link link_6_fixed_handle_knob
- removed link link_8_fixed_hinge
- removed link link_9_fixed_handle_shaft
- added link link_fixed_0_floor, mass 0.001; collision box size=31.999 31.999 0.199; visual box size=31.999 31.999 0.199
- added link link_fixed_10_handle_shaft, mass 0.001; collision cylinder length=0.999 radius=0.0995; visual cylinder length=0.999 radius=0.0995
- added link link_fixed_11_handle_knob, mass 0.001; collision box size=0.049 0.049 0.199; visual box size=0.049 0.049 0.199
- added link link_fixed_13_handle_shaft, mass 0.001; collision box size=0.199 0.199 0.999; visual box size=0.199 0.199 0.999
- added link link_fixed_14_handle_knob, mass 0.001; collision box size=0.049 0.049 0.199; visual box size=0.049 0.049 0.199
- added link link_fixed_16_handle_shaft, mass 0.001; collision box size=0.199 0.199 0.999; visual box size=0.199 0.199 0.999
- added link link_fixed_17_handle_knob, mass 0.001; collision box size=0.049 0.049 0.199; visual box size=0.049 0.049 0.199
- added link link_fixed_19_handle_shaft, mass 0.001; collision box size=0.199 0.199 0.999; visual box size=0.199 0.199 0.999
- added link link_fixed_20_handle_knob, mass 0.001; collision box size=0.049 0.049 0.199; visual box size=0.049 0.049 0.199
- added link link_fixed_2_hinge, mass 0.001; visual cylinder length=0.989 radius=0.112
- added link link_fixed_2_hinge.001, mass 0.001; visual cylinder length=0.98801 radius=0.11189
- added link link_fixed_3_handle_shaft, mass 0.001; collision cylinder length=0.999 radius=0.0995; visual cylinder length=0.999 radius=0.0995
- added link link_fixed_3_handle_shaft.001, mass 0.001; visual cylinder length=0.998 radius=0.0994
- added link link_fixed_4_handle_knob, mass 0.001; collision box size=0.049 0.049 0.199; visual box size=0.049 0.049 0.199
- added link link_fixed_4_handle_knob.001, mass 0.001; visual box size=0.04895 0.04895 0.1988
- added link link_fixed_6_handle_shaft, mass 0.001; collision box size=0.199 0.199 0.999; visual box size=0.199 0.199 0.999
- added link link_fixed_7_handle_knob, mass 0.001; collision box size=0.049 0.049 0.199; visual box size=0.049 0.049 0.199
- added link link_fixed_9_hinge, mass 0.001; visual cylinder length=0.989 radius=0.112
- link base_link: geometry 
Joints:
- removed joint link_10_fixed_handle_knob
- removed joint link_12_fixed_handle_shaft
- removed joint link_13_fixed_handle_knob
- removed joint link_15_fixed_handle_shaft
- removed joint link_16_fixed_handle_knob
- removed joint link_18_fixed_handle_shaft
- removed joint link_19_fixed_handle_knob
- removed joint link_1_fixed_hinge
- removed joint link_1_fixed_hinge.001
- removed joint link_2_fixed_handle_shaft
- removed joint link_2_fixed_handle_shaft.001
- removed joint link_3_fixed_handle_knob
- removed joint link_3_fixed_handle_knob.001
- removed joint link_5_fixed_handle_shaft
- removed joint link_6_fixed_handle_knob
- removed joint link_8_fixed_hinge
- removed joint link_9_fixed_handle_shaft
- added joint link_fixed_0_floor: type fixed, parent base_link, child link_fixed_0_floor, origin xyz=0 0 -0.1 rpy=0 0 0
- added joint link_fixed_10_handle_shaft: type fixed, parent link_2_joint_0, child link_fixed_10_handle_shaft, origin xyz=1.0875 0 0.95 rpy=0 0 0
- added joint link_fixed_11_handle_knob: type fixed, parent link_fixed_10_handle_shaft, child link_fixed_11_handle_knob, origin xyz=0 0 0.6 rpy=0 0 0
- added joint link_fixed_13_handle_shaft: type fixed, parent link_3_joint_0, child link_fixed_13_handle_shaft, origin xyz=0 0 0.95 rpy=0 0 0
- added joint link_fixed_14_handle_knob: type fixed, parent link_fixed_13_handle_shaft, child link_fixed_14_handle_knob, origin xyz=0 0 0.6 rpy=0 0 0
- added joint link_fixed_16_handle_shaft: type fixed, parent link_4_joint_0, child link_fixed_16_handle_shaft, origin xyz=0 0 0.95 rpy=0 0 0
- added joint link_fixed_17_handle_knob: type fixed, parent link_fixed_16_handle_shaft, child link_fixed_17_handle_knob, origin xyz=0 0 0.6 rpy=0 0 0
- added joint link_fixed_19_handle_shaft: type fixed, parent link_5_joint_0, child link_fixed_19_handle_shaft, origin xyz=0 0 0.95 rpy=0 0 0
- added joint link_fixed_20_handle_knob: type fixed, parent link_fixed_19_handle_shaft, child link_fixed_20_handle_knob, origin xyz=0 0 0.6 rpy=0 0 0
- added joint link_fixed_2_hinge: type fixed, parent link_0_joint_0, child link_fixed_2_hinge, origin xyz=0 0 0 rpy=0 0 0
- added joint link_fixed_2_hinge.001: type fixed, parent goal, child link_fixed_2_hinge.001, origin xyz=0 0 0 rpy=0 0 0
- added joint link_fixed_3_handle_shaft: type fixed, parent link_0_joint_0, child link_fixed_3_handle_shaft, origin xyz=1.0875 0 0.95 rpy=0 0 0
- added joint link_fixed_3_handle_shaft.001: type fixed, parent goal, child link_fixed_3_handle_shaft.001, origin xyz=1.08641 0 0.94905 rpy=0 0 0
- added joint link_fixed_4_handle_knob: type fixed, parent link_fixed_3_handle_shaft, child link_fixed_4_handle_knob, origin xyz=0 0 0.6 rpy=0 0 0
- added joint link_fixed_4_handle_knob.001: type fixed, parent link_fixed_3_handle_shaft.001, child link_fixed_4_handle_knob.001, origin xyz=0 0 0.5994 rpy=0 0 0
- added joint link_fixed_6_handle_shaft: type fixed, parent link_1_joint_0, child link_fixed_6_handle_shaft, origin xyz=0 0 0.95 rpy=0 0 0
- added joint link_fixed_7_handle_knob: type fixed, parent link_fixed_6_handle_shaft, child link_fixed_7_handle_knob, origin xyz=0 0 0.6 rpy=0 0 0
- added joint link_fixed_9_hinge: type fixed, parent link_2_joint_0, child link_fixed_9_hinge, origin xyz=0 0 0 rpy=0 0 0
- joint goal: origin xyz=-0.5 0.5 0.55 rpy=0 0 1.5708 -> xyz=-0.5 0.5 0.45 rpy=0 0 1.5708
- joint link_0_joint_0: origin xyz=-0.5 0.5 0.55 rpy=0 0 0 -> xyz=-0.5 0.5 0.45 rpy=0 0 0
- joint link_1_joint_0: origin xyz=-1.0 1.5 0.55 rpy=0 0 3.14159 -> xyz=-1.0 1.5 0.45 rpy=0 0 3.14159
- joint link_2_joint_0: origin xyz=-2.5 -0.5 0.55 rpy=0 0 0 -> xyz=-2.5 -0.5 0.45 rpy=0 0 0
- joint link_3_joint_0: origin xyz=1.0 1.5 0.55 rpy=0 0 0 -> xyz=1.0 1.5 0.45 rpy=0 0 0
- joint link_4_joint_0: origin xyz=0 -0.5 0.55 rpy=0 0 0 -> xyz=0 -0.5 0.45 rpy=0 0 0
- joint link_5_joint_0: origin xyz=-2.5 2.0 0.55 rpy=0 0 1.5708 -> xyz=-2.5 2.0 0.45 rpy=0 0 1.5708

File: puzzles/lockbox2017/urdf/lockbox2017.urdf (robot description, URDF)
Before this commit: robot lockbox2017, 23 links, 22 joints
Links:
- removed link link_10_fixed_handle_knob
- removed link link_12_fixed_handle_shaft
- removed link link_13_fixed_handle_knob
- removed link link_15_fixed_hinge
- removed link link_16_fixed_door_panel
- removed link link_17_fixed_door_handle
- removed link link_1_fixed_hinge
- removed link link_1_fixed_hinge.001
- removed link link_2_fixed_door_panel
- removed link link_2_fixed_door_panel.001
- removed link link_3_fixed_door_handle
- removed link link_3_fixed_door_handle.001
- removed link link_5_fixed_handle_shaft
- removed link link_6_fixed_handle_knob
- removed link link_8_fixed_hinge
- removed link link_9_fixed_handle_shaft
- added link link_fixed_0_floor, mass 0.001; collision box size=31.999 31.999 0.199; visual box size=31.999 31.999 0.199
- added link link_fixed_10_handle_shaft, mass 0.001; collision cylinder length=0.999 radius=0.0995; visual cylinder length=0.999 radius=0.0995
- added link link_fixed_11_handle_knob, mass 0.001; collision box size=0.049 0.049 0.199; visual box size=0.049 0.049 0.199
- added link link_fixed_13_handle_shaft, mass 0.001; collision box size=0.199 0.199 0.999; visual box size=0.199 0.199 0.999
- added link link_fixed_14_handle_knob, mass 0.001; collision box size=0.049 0.049 0.199; visual box size=0.049 0.049 0.199
- added link link_fixed_16_hinge, mass 0.001; visual cylinder length=2.199 radius=0.0495
- added link link_fixed_17_door_panel, mass 0.001; collision box size=3.999 0.199 1.999; visual box size=3.999 0.199 1.999
- added link link_fixed_18_door_handle, mass 0.001; collision box size=0.199 0.049 0.199; visual box size=0.199 0.049 0.199
- added link link_fixed_2_hinge, mass 0.001; visual cylinder length=2.199 radius=0.0495
- added link link_fixed_2_hinge.001, mass 0.001; visual cylinder length=2.1968 radius=0.04945
- added link link_fixed_3_door_panel, mass 0.001; collision box size=1.999 0.199 1.999; visual box size=1.999 0.199 1.999
- added link link_fixed_3_door_panel.001, mass 0.001; visual box size=1.997 0.1988 1.997
- added link link_fixed_4_door_handle, mass 0.001; collision box size=0.199 0.049 0.199; visual box size=0.199 0.049 0.199
- added link link_fixed_4_door_handle.001, mass 0.001; visual box size=0.1988 0.04895 0.1988
- added link link_fixed_6_handle_shaft, mass 0.001; collision box size=0.199 0.199 0.999; visual box size=0.199 0.199 0.999
- added link link_fixed_7_handle_knob, mass 0.001; collision box size=0.049 0.049 0.199; visual box size=0.049 0.049 0.199
- added link link_fixed_9_hinge, mass 0.001; visual cylinder length=1.099 radius=0.1245
- link base_link: geometry 
Joints:
- removed joint link_10_fixed_handle_knob
- removed joint link_12_fixed_handle_shaft
- removed joint link_13_fixed_handle_knob
- removed joint link_15_fixed_hinge
- removed joint link_16_fixed_door_panel
- removed joint link_17_fixed_door_handle
- removed joint link_1_fixed_hinge
- removed joint link_1_fixed_hinge.001
- removed joint link_2_fixed_door_panel
- removed joint link_2_fixed_door_panel.001
- removed joint link_3_fixed_door_handle
- removed joint link_3_fixed_door_handle.001
- removed joint link_5_fixed_handle_shaft
- removed joint link_6_fixed_handle_knob
- removed joint link_8_fixed_hinge
- removed joint link_9_fixed_handle_shaft
- added joint link_fixed_0_floor: type fixed, parent base_link, child link_fixed_0_floor, origin xyz=0 0 -0.1 rpy=0 0 0
- added joint link_fixed_10_handle_shaft: type fixed, parent link_2_joint_0, child link_fixed_10_handle_shaft, origin xyz=0 1.5 1.0 rpy=0 0 0
- added joint link_fixed_11_handle_knob: type fixed, parent link_fixed_10_handle_shaft, child link_fixed_11_handle_knob, origin xyz=0 0 0.6 rpy=0 0 0
- added joint link_fixed_13_handle_shaft: type fixed, parent link_3_joint_0, child link_fixed_13_handle_shaft, origin xyz=0 0 1.0 rpy=0 0 0
- added joint link_fixed_14_handle_knob: type fixed, parent link_fixed_13_handle_shaft, child link_fixed_14_handle_knob, origin xyz=0 0 0.6 rpy=0 0 0
- added joint link_fixed_16_hinge: type fixed, parent link_4_joint_0, child link_fixed_16_hinge, origin xyz=0 0 0 rpy=0 0 0
- added joint link_fixed_17_door_panel: type fixed, parent link_4_joint_0, child link_fixed_17_door_panel, origin xyz=2.0 0 0 rpy=0 0 0
- added joint link_fixed_18_door_handle: type fixed, parent link_4_joint_0, child link_fixed_18_door_handle, origin xyz=3.0 0 1.1 rpy=0 0 0
- added joint link_fixed_2_hinge: type fixed, parent link_0_joint_0, child link_fixed_2_hinge, origin xyz=0 0 0 rpy=0 0 0
- added joint link_fixed_2_hinge.001: type fixed, parent goal, child link_fixed_2_hinge.001, origin xyz=0 0 0 rpy=0 0 0
- added joint link_fixed_3_door_panel: type fixed, parent link_0_joint_0, child link_fixed_3_door_panel, origin xyz=1.0 0 0 rpy=0 0 0
- added joint link_fixed_3_door_panel.001: type fixed, parent goal, child link_fixed_3_door_panel.001, origin xyz=0.999 0 0 rpy=0 0 0
- added joint link_fixed_4_door_handle: type fixed, parent link_0_joint_0, child link_fixed_4_door_handle, origin xyz=1.5 0 1.1 rpy=0 0 0
- added joint link_fixed_4_door_handle.001: type fixed, parent goal, child link_fixed_4_door_handle.001, origin xyz=1.4985 0 1.0989 rpy=0 0 0
- added joint link_fixed_6_handle_shaft: type fixed, parent link_1_joint_0, child link_fixed_6_handle_shaft, origin xyz=0 0 1.0 rpy=0 0 0
- added joint link_fixed_7_handle_knob: type fixed, parent link_fixed_6_handle_shaft, child link_fixed_7_handle_knob, origin xyz=0 0 0.6 rpy=0 0 0
- added joint link_fixed_9_hinge: type fixed, parent link_2_joint_0, child link_fixed_9_hinge, origin xyz=0 0 0 rpy=0 0 0
- joint goal: origin xyz=-6.0 -1.0 1.1 rpy=0 0 1.5708 -> xyz=-6.0 -1.0 1.0 rpy=0 0 1.5708
- joint link_0_joint_0: origin xyz=-6.0 -1.0 1.1 rpy=0 0 0 -> xyz=-6.0 -1.0 1.0 rpy=0 0 0
- joint link_1_joint_0: origin xyz=-4.0 0 0.6 rpy=0 0 0 -> xyz=-4.0 0 0.5 rpy=0 0 0
- joint link_2_joint_0: origin xyz=0 0 0.6 rpy=0 0 1.5708 -> xyz=0 0 0.5 rpy=0 0 1.5708
- joint link_3_joint_0: origin xyz=0 2.0 0.6 rpy=0 0 1.5708 -> xyz=0 2.0 0.5 rpy=0 0 1.5708
- joint link_4_joint_0: origin xyz=-2.0 4.0 1.1 rpy=0 0 0 -> xyz=-2.0 4.0 1.0 rpy=0 0 0
