Commit message: refactor: separate floor from base_link

File: puzzles/lockbox_random/urdf/lockbox_random.urdf (robot description, URDF)
Before this commit: robot lockbox_random, 21 links, 20 joints
Links:
- removed link link_11_fixed_hinge
- removed link link_12_fixed_handle_shaft
- removed link link_13_fixed_handle_knob
- removed link link_15_fixed_handle_shaft
- removed link link_16_fixed_handle_knob
- removed link link_1_fixed_handle_shaft
- removed link link_1_fixed_handle_shaft.001
- removed link link_2_fixed_handle_knob
- removed link link_2_fixed_handle_knob.001
- removed link link_4_fixed_hinge
- removed link link_5_fixed_handle_shaft
- removed link link_6_fixed_handle_knob
- removed link link_8_fixed_handle_shaft
- removed link link_9_fixed_handle_knob
- added link link_fixed_0_floor, mass 0.001; collision box size=31.999 31.999 0.199; visual box size=31.999 31.999 0.199
- added link link_fixed_10_handle_knob, mass 0.001; collision box size=0.049 0.049 0.199; visual box size=0.049 0.049 0.199
- added link link_fixed_12_hinge, mass 0.001; visual cylinder length=1.099 radius=0.1245
- added link link_fixed_13_handle_shaft, mass 0.001; collision cylinder length=0.999 radius=0.0995; visual cylinder length=0.999 radius=0.0995
- added link link_fixed_14_handle_knob, mass 0.001; collision box size=0.049 0.049 0.199; visual box size=0.049 0.049 0.199
- added link link_fixed_16_handle_shaft, mass 0.001; collision box size=0.199 0.199 0.999; visual box size=0.199 0.199 0.999
- added link link_fixed_17_handle_knob, mass 0.001; collision box size=0.049 0.049 0.199; visual box size=0.049 0.049 0.199
- added link link_fixed_2_handle_shaft, mass 0.001; collision box size=0.199 0.199 0.999; visual box size=0.199 0.199 0.999
- added link link_fixed_2_handle_shaft.001, mass 0.001; visual box size=0.1988 0.1988 0.998
- added link link_fixed_3_handle_knob, mass 0.001; collision box size=0.049 0.049 0.199; visual box size=0.049 0.049 0.199
- added link link_fixed_3_handle_knob.001, mass 0.001; visual box size=0.04895 0.04895 0.1988
- added link link_fixed_5_hinge, mass 0.001; visual cylinder length=1.099 radius=0.1245
- added link link_fixed_6_handle_shaft, mass 0.001; collision cylinder length=0.999 radius=0.0995; visual cylinder length=0.999 radius=0.0995
- added link link_fixed_7_handle_knob, mass 0.001; collision box size=0.049 0.049 0.199; visual box size=0.049 0.049 0.199
- added link link_fixed_9_handle_shaft, mass 0.001; collision box size=0.199 0.199 0.999; visual box size=0.199 0.199 0.999
- link base_link: geometry 
Joints:
- removed joint link_11_fixed_hinge
- removed joint link_12_fixed_handle_shaft
- removed joint link_13_fixed_handle_knob
- removed joint link_15_fixed_handle_shaft
- removed joint link_16_fixed_handle_knob
- removed joint link_1_fixed_handle_shaft
- removed joint link_1_fixed_handle_shaft.001
- removed joint link_2_fixed_handle_knob
- removed joint link_2_fixed_handle_knob.001
- removed joint link_4_fixed_hinge
- removed joint link_5_fixed_handle_shaft
- removed joint link_6_fixed_handle_knob
- removed joint link_8_fixed_handle_shaft
- removed joint link_9_fixed_handle_knob
- added joint link_fixed_0_floor: type fixed, parent base_link, child link_fixed_0_floor, origin xyz=0 0 -0.1 rpy=0 0 0
- added joint link_fixed_10_handle_knob: type fixed, parent link_fixed_9_handle_shaft, child link_fixed_10_handle_knob, origin xyz=0 0 0.6 rpy=0 0 0
- added joint link_fixed_12_hinge: type fixed, parent link_3_joint_0, child link_fixed_12_hinge, origin xyz=0 0 0 rpy=0 0 0
- added joint link_fixed_13_handle_shaft: type fixed, parent link_3_joint_0, child link_fixed_13_handle_shaft, origin xyz=0 1.125 1.0 rpy=0 0 0
- added joint link_fixed_14_handle_knob: type fixed, parent link_fixed_13_handle_shaft, child link_fixed_14_handle_knob, origin xyz=0 0 0.6 rpy=0 0 0
- added joint link_fixed_16_handle_shaft: type fixed, parent link_4_joint_0, child link_fixed_16_handle_shaft, origin xyz=0 0 1.0 rpy=0 0 0
- added joint link_fixed_17_handle_knob: type fixed, parent link_fixed_16_handle_shaft, child link_fixed_17_handle_knob, origin xyz=0 0 0.6 rpy=0 0 0
- added joint link_fixed_2_handle_shaft: type fixed, parent link_0_joint_0, child link_fixed_2_handle_shaft, origin xyz=0 0 1.0 rpy=0 0 0
- added joint link_fixed_2_handle_shaft.001: type fixed, parent goal, child link_fixed_2_handle_shaft.001, origin xyz=0 0 0.999 rpy=0 0 0
- added joint link_fixed_3_handle_knob: type fixed, parent link_fixed_2_handle_shaft, child link_fixed_3_handle_knob, origin xyz=0 0 0.6 rpy=0 0 0
- added joint link_fixed_3_handle_knob.001: type fixed, parent link_fixed_2_handle_shaft.001, child link_fixed_3_handle_knob.001, origin xyz=0 0 0.5994 rpy=0 0 0
- added joint link_fixed_5_hinge: type fixed, parent link_1_joint_0, child link_fixed_5_hinge, origin xyz=0 0 0 rpy=0 0 0
- added joint link_fixed_6_handle_shaft: type fixed, parent link_1_joint_0, child link_fixed_6_handle_shaft, origin xyz=0 1.125 1.0 rpy=0 0 0
- added joint link_fixed_7_handle_knob: type fixed, parent link_fixed_6_handle_shaft, child link_fixed_7_handle_knob, origin xyz=0 0 0.6 rpy=0 0 0
- added joint link_fixed_9_handle_shaft: type fixed, parent link_2_joint_0, child link_fixed_9_handle_shaft, origin xyz=0 0 1.0 rpy=0 0 0
- joint goal: origin xyz=-1.0 0.5 0.6 rpy=0 0 0 -> xyz=-1.0 0.5 0.5 rpy=0 0 0
- joint link_0_joint_0: origin xyz=-2.0 0.5 0.6 rpy=0 0 0 -> xyz=-2.0 0.5 0.5 rpy=0 0 0
- joint link_1_joint_0: origin xyz=0.5 0.5 0.6 rpy=0 0 1.5708 -> xyz=0.5 0.5 0.5 rpy=0 0 1.5708
- joint link_2_joint_0: origin xyz=0.5 2.0 0.6 rpy=0 0 1.5708 -> xyz=0.5 2.0 0.5 rpy=0 0 1.5708
- joint link_3_joint_0: origin xyz=0.5 4.5 0.6 rpy=0 0 3.14159 -> xyz=0.5 4.5 0.5 rpy=0 0 3.14159
- joint link_4_joint_0: origin xyz=-1.0 4.5 0.6 rpy=0 0 3.14159 -> xyz=-1.0 4.5 0.5 rpy=0 0 3.14159

File: puzzles/move_twice/urdf/move_twice.urdf (robot description, URDF)
Before this commit: robot move_twice, 12 links, 11 joints
Links:
- removed link link_3_fixed_wall_left
- removed link link_4_fixed_wall_right
- removed link link_5_fixed_wall_mid
- removed link link_6_fixed_wall_back
- added link link_fixed_0_floor, mass 0.001; collision box size=31.999 31.999 0.199; visual box size=31.999 31.999 0.199
- added link link_fixed_4_wall_left, mass 0.001; collision box size=3.999 0.199 0.999; visual box size=3.999 0.199 0.999
- added link link_fixed_5_wall_right, mass 0.001; collision box size=3.999 0.199 0.999; visual box size=3.999 0.199 0.999
- added link link_fixed_6_wall_mid, mass 0.001; collision box size=3.999 0.199 0.999; visual box size=3.999 0.199 0.999
- added link link_fixed_7_wall_back, mass 0.001; collision box size=0.199 5.999 0.999; visual box size=0.199 5.999 0.999
- link base_link: geometry 
Joints:
- removed joint link_3_fixed_wall_left
- removed joint link_4_fixed_wall_right
- removed joint link_5_fixed_wall_mid
- removed joint link_6_fixed_wall_back
- added joint link_fixed_0_floor: type fixed, parent base_link, child link_fixed_0_floor, origin xyz=0 0 -0.1 rpy=0 0 0
- added joint link_fixed_4_wall_left: type fixed, parent base_link, child link_fixed_4_wall_left, origin xyz=0 -1.4 0.5 rpy=0 0 0
- added joint link_fixed_5_wall_right: type fixed, parent base_link, child link_fixed_5_wall_right, origin xyz=0 4.4 0.5 rpy=0 0 0
- added joint link_fixed_6_wall_mid: type fixed, parent base_link, child link_fixed_6_wall_mid, origin xyz=0 1.5 0.5 rpy=0 0 0
- added joint link_fixed_7_wall_back: type fixed, parent base_link, child link_fixed_7_wall_back, origin xyz=-2.1 1.5 0.5 rpy=0 0 0
- joint goal: origin xyz=1.03327 3.36114 0.6 rpy=0 0 -0.49906 -> xyz=1.03327 3.36114 0.5 rpy=0 0 -0.49906
- joint link_0_joint_2: origin xyz=0 0 0.6 rpy=0 0 0 -> xyz=0 0 0.5 rpy=0 0 0
- joint link_1_joint_0: origin xyz=2.1 1.5 0.6 rpy=0 0 0 -> xyz=2.1 1.5 0.5 rpy=0 0 0

File: puzzles/simple_sliders/urdf/simple_sliders.urdf (robot description, URDF)
Before this commit: robot simple_sliders, 16 links, 15 joints
Links:
- removed link link_10_fixed_handle_shaft
- removed link link_11_fixed_handle_knob
- removed link link_1_fixed_handle_shaft
- removed link link_1_fixed_handle_shaft.001
- removed link link_2_fixed_handle_knob
- removed link link_2_fixed_handle_knob.001
- removed link link_4_fixed_handle_shaft
- removed link link_5_fixed_handle_knob
- removed link link_7_fixed_handle_shaft
- removed link link_8_fixed_handle_knob
- added link link_fixed_0_floor, mass 0.001; collision box size=31.999 31.999 0.199; visual box size=31.999 31.999 0.199
- added link link_fixed_11_handle_shaft, mass 0.001; collision box size=0.199 0.199 0.999; visual box size=0.199 0.199 0.999
- added link link_fixed_12_handle_knob, mass 0.001; collision box size=0.049 0.049 0.199; visual box size=0.049 0.049 0.199
- added link link_fixed_2_handle_shaft, mass 0.001; collision box size=0.199 0.199 0.999; visual box size=0.199 0.199 0.999
- added link link_fixed_2_handle_shaft.001, mass 0.001; visual box size=0.1988 0.1988 0.998
- added link link_fixed_3_handle_knob, mass 0.001; collision box size=0.049 0.049 0.199; visual box size=0.049 0.049 0.199
- added link link_fixed_3_handle_knob.001, mass 0.001; visual box size=0.04895 0.04895 0.1988
- added link link_fixed_5_handle_shaft, mass 0.001; collision box size=0.199 0.199 0.999; visual box size=0.199 0.199 0.999
- added link link_fixed_6_handle_knob, mass 0.001; collision box size=0.049 0.049 0.199; visual box size=0.049 0.049 0.199
- added link link_fixed_8_handle_shaft, mass 0.001; collision box size=0.199 0.199 0.999; visual box size=0.199 0.199 0.999
- added link link_fixed_9_handle_knob, mass 0.001; collision box size=0.049 0.049 0.199; visual box size=0.049 0.049 0.199
- link base_link: geometry 
Joints:
- removed joint link_10_fixed_handle_shaft
- removed joint link_11_fixed_handle_knob
- removed joint link_1_fixed_handle_shaft
- removed joint link_1_fixed_handle_shaft.001
- removed joint link_2_fixed_handle_knob
- removed joint link_2_fixed_handle_knob.001
- removed joint link_4_fixed_handle_shaft
- removed joint link_5_fixed_handle_knob
- removed joint link_7_fixed_handle_shaft
- removed joint link_8_fixed_handle_knob
- added joint link_fixed_0_floor: type fixed, parent base_link, child link_fixed_0_floor, origin xyz=0 0 -0.1 rpy=0 0 0
- added joint link_fixed_11_handle_shaft: type fixed, parent link_3_joint_0, child link_fixed_11_handle_shaft, origin xyz=0 0 0.6 rpy=0 0 0
- added joint link_fixed_12_handle_knob: type fixed, parent link_fixed_11_handle_shaft, child link_fixed_12_handle_knob, origin xyz=0 0 0.6 rpy=0 0 0
- added joint link_fixed_2_handle_shaft: type fixed, parent link_0_joint_0, child link_fixed_2_handle_shaft, origin xyz=0 0 0.6 rpy=0 0 0
- added joint link_fixed_2_handle_shaft.001: type fixed, parent goal, child link_fixed_2_handle_shaft.001, origin xyz=0 0 0.5994 rpy=0 0 0
- added joint link_fixed_3_handle_knob: type fixed, parent link_fixed_2_handle_shaft, child link_fixed_3_handle_knob, origin xyz=0 0 0.6 rpy=0 0 0
- added joint link_fixed_3_handle_knob.001: type fixed, parent link_fixed_2_handle_shaft.001, child link_fixed_3_handle_knob.001, origin xyz=0 0 0.5994 rpy=0 0 0
- added joint link_fixed_5_handle_shaft: type fixed, parent link_1_joint_0, child link_fixed_5_handle_shaft, origin xyz=0 0 0.6 rpy=0 0 0
- added joint link_fixed_6_handle_knob: type fixed, parent link_fixed_5_handle_shaft, child link_fixed_6_handle_knob, origin xyz=0 0 0.6 rpy=0 0 0
- added joint link_fixed_8_handle_shaft: type fixed, parent link_2_joint_0, child link_fixed_8_handle_shaft, origin xyz=0 0 0.6 rpy=0 0 0
- added joint link_fixed_9_handle_knob: type fixed, parent link_fixed_8_handle_shaft, child link_fixed_9_handle_knob, origin xyz=0 0 0.6 rpy=0 0 0
- joint goal: origin xyz=0 -1.0 0.2 rpy=0 0 -1.5708 -> xyz=0 -1.0 0.1 rpy=0 0 -1.5708
- joint link_0_joint_0: origin xyz=0 0 0.2 rpy=0 0 -1.5708 -> xyz=0 0 0.1 rpy=0 0 -1.5708
- joint link_1_joint_0: origin xyz=0 -1.0 0.2 rpy=0 0 0 -> xyz=0 -1.0 0.1 rpy=0 0 0
- joint link_2_joint_0: origin xyz=1.0 -1.0 0.2 rpy=0 0 -1.5708 -> xyz=1.0 -1.0 0.1 rpy=0 0 -1.5708
- joint link_3_joint_0: origin xyz=1.0 -2.0 0.2 rpy=0 0 0 -> xyz=1.0 -2.0 0.1 rpy=0 0 0

Commit message: feat: render_images() images from 9 different angles

File: puzzles/continuous_space/urdf/continuous_space.urdf (robot description, URDF)
Before this commit: robot continuous_space, 22 links, 21 joints
Links:
- removed link link_fixed_124_hinge
- removed link link_fixed_125_handle_shaft
- removed link link_fixed_126_handle_knob
- removed link link_fixed_14_handle_shaft
- removed link link_fixed_152_handle_shaft
- removed link link_fixed_153_handle_knob
- removed link link_fixed_15_handle_knob
- removed link link_fixed_2_handle_shaft
- removed link link_fixed_2_handle_shaft.001
- removed link link_fixed_3_handle_knob
- removed link link_fixed_3_handle_knob.001
- removed link link_fixed_62_hinge
- removed link link_fixed_63_handle_shaft
- removed link link_fixed_64_handle_knob
- added link link_fixed_10_handle_knob, mass 0.001; collision box size=0.049 0.049 0.199; visual box size=0.049 0.049 0.199
- added link link_fixed_2_hinge, mass 0.001; visual cylinder length=1.099 radius=0.1245
- added link link_fixed_2_hinge.001, mass 0.001; visual cylinder length=1.0979 radius=0.12438
- added link link_fixed_3_handle_shaft, mass 0.001; collision cylinder length=0.999 radius=0.0995; visual cylinder length=0.999 radius=0.0995
- added link link_fixed_3_handle_shaft.001, mass 0.001; visual cylinder length=0.998 radius=0.0994
- added link link_fixed_4_handle_knob, mass 0.001; collision box size=0.049 0.049 0.199; visual box size=0.049 0.049 0.199
- added link link_fixed_4_handle_knob.001, mass 0.001; visual box size=0.04895 0.04895 0.1988
- added link link_fixed_60_handle_shaft, mass 0.001; collision box size=0.199 0.199 0.999; visual box size=0.199 0.199 0.999
- added link link_fixed_61_handle_knob, mass 0.001; collision box size=0.049 0.049 0.199; visual box size=0.049 0.049 0.199
- added link link_fixed_77_handle_shaft, mass 0.001; collision box size=0.199 0.199 0.999; visual box size=0.199 0.199 0.999
- added link link_fixed_78_handle_knob, mass 0.001; collision box size=0.049 0.049 0.199; visual box size=0.049 0.049 0.199
- added link link_fixed_88_hinge, mass 0.001; visual cylinder length=1.099 radius=0.1245
- added link link_fixed_89_handle_shaft, mass 0.001; collision cylinder length=0.999 radius=0.0995; visual cylinder length=0.999 radius=0.0995
- added link link_fixed_90_handle_knob, mass 0.001; collision box size=0.049 0.049 0.199; visual box size=0.049 0.049 0.199
- added link link_fixed_9_handle_shaft, mass 0.001; collision box size=0.199 0.199 0.999; visual box size=0.199 0.199 0.999
- link goal: geometry visual box size=2.996 0.998 0.998
- link link_0_joint_0: geometry collision box size=2.999 0.999 0.999; visual box size=2.999 0.999 0.999
- link link_2_joint_0: geometry collision box size=1.999 0.999 0.999; visual box size=1.999 0.999 0.999
- link link_3_joint_0: geometry collision box size=1.999 0.999 0.999; visual box size=1.999 0.999 0.999
- link link_4_joint_0: geometry collision box size=2.999 0.999 0.999; visual box size=2.999 0.999 0.999
Joints:
- removed joint link_fixed_124_hinge
- removed joint link_fixed_125_handle_shaft
- removed joint link_fixed_126_handle_knob
- removed joint link_fixed_14_handle_shaft
- removed joint link_fixed_152_handle_shaft
- removed joint link_fixed_153_handle_knob
- removed joint link_fixed_15_handle_knob
- removed joint link_fixed_2_handle_shaft
- removed joint link_fixed_2_handle_shaft.001
- removed joint link_fixed_3_handle_knob
- removed joint link_fixed_3_handle_knob.001
- removed joint link_fixed_62_hinge
- removed joint link_fixed_63_handle_shaft
- removed joint link_fixed_64_handle_knob
- added joint link_fixed_10_handle_knob: type fixed, parent link_fixed_9_handle_shaft, child link_fixed_10_handle_knob, origin xyz=0 0 0.6 rpy=0 0 0
- added joint link_fixed_2_hinge: type fixed, parent link_0_joint_0, child link_fixed_2_hinge, origin xyz=0 0 0 rpy=0 0 0
- added joint link_fixed_2_hinge.001: type fixed, parent goal, child link_fixed_2_hinge.001, origin xyz=0 0 0 rpy=0 0 0
- added joint link_fixed_3_handle_shaft: type fixed, parent link_0_joint_0, child link_fixed_3_handle_shaft, origin xyz=1.125 0 1.0 rpy=0 0 0
- added joint link_fixed_3_handle_shaft.001: type fixed, parent goal, child link_fixed_3_handle_shaft.001, origin xyz=1.12388 0 0.999 rpy=0 0 0
- added joint link_fixed_4_handle_knob: type fixed, parent link_fixed_3_handle_shaft, child link_fixed_4_handle_knob, origin xyz=0 0 0.6 rpy=0 0 0
- added joint link_fixed_4_handle_knob.001: type fixed, parent link_fixed_3_handle_shaft.001, child link_fixed_4_handle_knob.001, origin xyz=0 0 0.5994 rpy=0 0 0
- added joint link_fixed_60_handle_shaft: type fixed, parent link_2_joint_0, child link_fixed_60_handle_shaft, origin xyz=0 0 1.0 rpy=0 0 0
- added joint link_fixed_61_handle_knob: type fixed, parent link_fixed_60_handle_shaft, child link_fixed_61_handle_knob, origin xyz=0 0 0.6 rpy=0 0 0
- added joint link_fixed_77_handle_shaft: type fixed, parent link_3_joint_0, child link_fixed_77_handle_shaft, origin xyz=0 0 1.0 rpy=0 0 0
- added joint link_fixed_78_handle_knob: type fixed, parent link_fixed_77_handle_shaft, child link_fixed_78_handle_knob, origin xyz=0 0 0.6 rpy=0 0 0
- added joint link_fixed_88_hinge: type fixed, parent link_4_joint_0, child link_fixed_88_hinge, origin xyz=0 0 0 rpy=0 0 0
- added joint link_fixed_89_handle_shaft: type fixed, parent link_4_joint_0, child link_fixed_89_handle_shaft, origin xyz=1.125 0 1.0 rpy=0 0 0
- added joint link_fixed_90_handle_knob: type fixed, parent link_fixed_89_handle_shaft, child link_fixed_90_handle_knob, origin xyz=0 0 0.6 rpy=0 0 0
- added joint link_fixed_9_handle_shaft: type fixed, parent link_1_joint_0, child link_fixed_9_handle_shaft, origin xyz=0 0 1.0 rpy=0 0 0
- joint goal: origin xyz=0.99739 -2.4812 0.5 rpy=0 0 -1.18859 -> xyz=0 0 0.5 rpy=0 0 -0.23802
- joint link_0_joint_0: axis 1.0 0 0 -> 0 0 1.0; limit lower=0 upper=2.67416 effort=0 velocity=0 -> lower=0 upper=3.06691 effort=0 velocity=0; origin xyz=0 0 0.5 rpy=0 0 -1.18859 -> xyz=0 0 0.5 rpy=0 0 2.97826; type prismatic -> revolute
- joint link_1_joint_0: limit lower=0 upper=3.11295 effort=0 velocity=0 -> lower=0 upper=3.94912 effort=0 velocity=0; origin xyz=-0.03422 -3.00526 0.5 rpy=0 0 -2.29454 -> xyz=0.21644 -1.77687 0.5 rpy=0 0 -0.77445
- joint link_2_joint_0: axis 0 0 1.0 -> 1.0 0 0; limit lower=0 upper=2.87617 effort=0 velocity=0 -> lower=0 upper=2.74264 effort=0 velocity=0; origin xyz=-1.10798 -5.00962 0.5 rpy=0 0 -1.25698 -> xyz=-0.02039 1.94214 0.5 rpy=0 0 0.74579; type revolute -> prismatic
- joint link_3_joint_0: axis 0 0 1.0 -> 1.0 0 0; limit lower=-2.54743 upper=0 effort=0 velocity=0 -> lower=0 upper=2.52402 effort=0 velocity=0; origin xyz=2.8631 -3.5405 0.5 rpy=0 0 -3.02217 -> xyz=1.38858 -3.83648 0.5 rpy=0 0 -2.62206; type revolute -> prismatic
- joint link_4_joint_0: axis 1.0 0 0 -> 0 0 1.0; limit lower=0 upper=3.4642 effort=0 velocity=0 -> lower=0 upper=3.09983 effort=0 velocity=0; origin xyz=3.4627 -1.85032 0.5 rpy=0 0 1.59111 -> xyz=-0.63097 -6.0368 0.5 rpy=0 0 -2.05119; type prismatic -> revolute
