Commit message: fix (minor): increase link_shrink

File: puzzles/continuous_space/urdf/continuous_space.urdf (robot description, URDF)
Before this commit: robot continuous_space, 23 links, 22 joints
Links:
- link goal: geometry visual box size=2.98003 0.99003 0.99002
- link link_0_joint_0: geometry collision box size=2.995 0.995 0.995; visual box size=2.995 0.995 0.995
- link link_1_joint_0: geometry collision box size=1.995 0.995 0.995; visual box size=1.995 0.995 0.995
- link link_2_joint_0: geometry collision box size=1.995 0.995 0.995; visual box size=1.995 0.995 0.995
- link link_3_joint_0: geometry collision box size=1.995 0.995 0.995; visual box size=1.995 0.995 0.995
- link link_4_joint_0: geometry collision box size=2.995 0.995 0.995; visual box size=2.995 0.995 0.995
- link link_fixed_0_floor: geometry collision box size=31.995 31.995 0.195; visual box size=31.995 31.995 0.195
- link link_fixed_10_handle_knob: geometry collision box size=0.045 0.045 0.195; visual box size=0.045 0.045 0.195
- link link_fixed_2_hinge: geometry visual cylinder length=1.095 radius=0.1225
- link link_fixed_2_hinge.001: geometry visual cylinder length=1.08952 radius=0.12189
- link link_fixed_3_handle_shaft: geometry collision cylinder length=0.995 radius=0.0975; visual cylinder length=0.995 radius=0.0975
- link link_fixed_3_handle_shaft.001: geometry visual cylinder length=0.99002 radius=0.09701
- link link_fixed_4_handle_knob: geometry collision box size=0.045 0.045 0.195; visual box size=0.045 0.045 0.195
- link link_fixed_4_handle_knob.001: geometry visual box size=0.04478 0.04478 0.19402
- link link_fixed_60_handle_shaft: geometry collision box size=0.195 0.195 0.995; visual box size=0.195 0.195 0.995
- link link_fixed_61_handle_knob: geometry collision box size=0.045 0.045 0.195; visual box size=0.045 0.045 0.195
- link link_fixed_77_handle_shaft: geometry collision box size=0.195 0.195 0.995; visual box size=0.195 0.195 0.995
- link link_fixed_78_handle_knob: geometry collision box size=0.045 0.045 0.195; visual box size=0.045 0.045 0.195
- link link_fixed_88_hinge: geometry visual cylinder length=1.095 radius=0.1225
- link link_fixed_89_handle_shaft: geometry collision cylinder length=0.995 radius=0.0975; visual cylinder length=0.995 radius=0.0975
- link link_fixed_90_handle_knob: geometry collision box size=0.045 0.045 0.195; visual box size=0.045 0.045 0.195
- link link_fixed_9_handle_shaft: geometry collision box size=0.195 0.195 0.995; visual box size=0.195 0.195 0.995
Joints:
- joint link_fixed_3_handle_shaft.001: origin xyz=1.12388 0 0.999 rpy=0 0 0 -> xyz=1.11937 0 0.995 rpy=0 0 0
- joint link_fixed_4_handle_knob.001: origin xyz=0 0 0.5994 rpy=0 0 0 -> xyz=0 0 0.597 rpy=0 0 0

File: puzzles/escape_room/urdf/escape_room.urdf (robot description, URDF)
Before this commit: robot escape_room, 19 links, 18 joints
Links:
- link link_0_joint_0.001: geometry visual mesh filename=file:///home/userone/ba/puzzle-generator/puzzles/escape_roo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 scale=0.995 0.995 0.995
- link link_2_joint_0: geometry collision cylinder length=0.995 radius=0.1975; visual cylinder length=0.995 radius=0.1975
- link link_fixed_0_floor: geometry collision box size=31.995 31.995 0.195; visual box size=31.995 31.995 0.195
- link link_fixed_10_door_handle1: geometry collision box size=0.045 0.195 0.195; visual box size=0.045 0.195 0.195
- link link_fixed_11_door_handle2: geometry collision box size=0.045 0.195 0.195; visual box size=0.045 0.195 0.195
- link link_fixed_12_wall_left: geometry collision box size=3.795 0.195 0.495; visual box size=3.795 0.195 0.495
- link link_fixed_13_wall_front: geometry collision box size=0.195 7.995 0.495; visual box size=0.195 7.995 0.495
- link link_fixed_14_wall_back: geometry collision box size=0.195 7.995 0.495; visual box size=0.195 7.995 0.495
- link link_fixed_8_hinge: geometry visual cylinder length=1.095 radius=0.0475
- link link_fixed_9_door_panel: geometry collision box size=3.195 0.195 0.995; visual box size=3.195 0.195 0.995

File: puzzles/grid_world/urdf/grid_world.urdf (robot description, URDF)
Before this commit: robot grid_world, 26 links, 25 joints
Links:
- link goal: geometry visual box size=2.88053 0.89052 0.89052
- link link_0_joint_0: geometry collision box size=2.895 0.895 0.895; visual box size=2.895 0.895 0.895
- link link_1_joint_0: geometry collision box size=1.895 0.895 0.895; visual box size=1.895 0.895 0.895
- link link_2_joint_0: geometry collision box size=2.895 0.895 0.895; visual box size=2.895 0.895 0.895
- link link_3_joint_0: geometry collision box size=1.895 0.895 0.895; visual box size=1.895 0.895 0.895
- link link_4_joint_0: geometry collision box size=1.895 0.895 0.895; visual box size=1.895 0.895 0.895
- link link_5_joint_0: geometry collision box size=1.895 0.895 0.895; visual box size=1.895 0.895 0.895
- link link_fixed_0_floor: geometry collision box size=31.995 31.995 0.195; visual box size=31.995 31.995 0.195
- link link_fixed_10_handle_shaft: geometry collision cylinder length=0.995 radius=0.0975; visual cylinder length=0.995 radius=0.0975
- link link_fixed_11_handle_knob: geometry collision box size=0.045 0.045 0.195; visual box size=0.045 0.045 0.195
- link link_fixed_13_handle_shaft: geometry collision box size=0.195 0.195 0.995; visual box size=0.195 0.195 0.995
- link link_fixed_14_handle_knob: geometry collision box size=0.045 0.045 0.195; visual box size=0.045 0.045 0.195
- link link_fixed_16_handle_shaft: geometry collision box size=0.195 0.195 0.995; visual box size=0.195 0.195 0.995
- link link_fixed_17_handle_knob: geometry collision box size=0.045 0.045 0.195; visual box size=0.045 0.045 0.195
- link link_fixed_19_handle_shaft: geometry collision box size=0.195 0.195 0.995; visual box size=0.195 0.195 0.995
- link link_fixed_20_handle_knob: geometry collision box size=0.045 0.045 0.195; visual box size=0.045 0.045 0.195
- link link_fixed_2_hinge: geometry visual cylinder length=0.985 radius=0.11
- link link_fixed_2_hinge.001: geometry visual cylinder length=0.98008 radius=0.10945
- link link_fixed_3_handle_shaft: geometry collision cylinder length=0.995 radius=0.0975; visual cylinder length=0.995 radius=0.0975
- link link_fixed_3_handle_shaft.001: geometry visual cylinder length=0.99002 radius=0.09701
- link link_fixed_4_handle_knob: geometry collision box size=0.045 0.045 0.195; visual box size=0.045 0.045 0.195
- link link_fixed_4_handle_knob.001: geometry visual box size=0.04478 0.04478 0.19402
- link link_fixed_6_handle_shaft: geometry collision box size=0.195 0.195 0.995; visual box size=0.195 0.195 0.995
- link link_fixed_7_handle_knob: geometry collision box size=0.045 0.045 0.195; visual box size=0.045 0.045 0.195
- link link_fixed_9_hinge: geometry visual cylinder length=0.985 radius=0.11
Joints:
- joint link_fixed_3_handle_shaft.001: origin xyz=1.08641 0 0.94905 rpy=0 0 0 -> xyz=1.08206 0 0.94525 rpy=0 0 0
- joint link_fixed_4_handle_knob.001: origin xyz=0 0 0.5994 rpy=0 0 0 -> xyz=0 0 0.597 rpy=0 0 0

File: puzzles/lockbox2017/urdf/lockbox2017.urdf (robot description, URDF)
Before this commit: robot lockbox2017, 24 links, 23 joints
Links:
- link goal: geometry visual cylinder length=1.98503 radius=0.19651
- link link_0_joint_0: geometry collision cylinder length=1.995 radius=0.1975; visual cylinder length=1.995 radius=0.1975
- link link_1_joint_0: geometry collision box size=2.995 0.495 0.995; visual box size=2.995 0.495 0.995
- link link_3_joint_0: geometry collision box size=2.995 0.495 0.995; visual box size=2.995 0.495 0.995
- link link_4_joint_0: geometry collision cylinder length=1.995 radius=0.1975; visual cylinder length=1.995 radius=0.1975
- link link_fixed_0_floor: geometry collision box size=31.995 31.995 0.195; visual box size=31.995 31.995 0.195
- link link_fixed_10_handle_shaft: geometry collision cylinder length=0.995 radius=0.0975; visual cylinder length=0.995 radius=0.0975
- link link_fixed_11_handle_knob: geometry collision box size=0.045 0.045 0.195; visual box size=0.045 0.045 0.195
- link link_fixed_13_handle_shaft: geometry collision box size=0.195 0.195 0.995; visual box size=0.195 0.195 0.995
- link link_fixed_14_handle_knob: geometry collision box size=0.045 0.045 0.195; visual box size=0.045 0.045 0.195
- link link_fixed_16_hinge: geometry visual cylinder length=2.195 radius=0.0475
- link link_fixed_17_door_panel: geometry collision box size=3.995 0.195 1.995; visual box size=3.995 0.195 1.995
- link link_fixed_18_door_handle: geometry collision box size=0.195 0.045 0.195; visual box size=0.195 0.045 0.195
- link link_fixed_2_hinge: geometry visual cylinder length=2.195 radius=0.0475
- link link_fixed_2_hinge.001: geometry visual cylinder length=2.18403 radius=0.04726
- link link_fixed_3_door_panel: geometry collision box size=1.995 0.195 1.995; visual box size=1.995 0.195 1.995
- link link_fixed_3_door_panel.001: geometry visual box size=1.98503 0.19402 1.98503
- link link_fixed_4_door_handle: geometry collision box size=0.195 0.045 0.195; visual box size=0.195 0.045 0.195
- link link_fixed_4_door_handle.001: geometry visual box size=0.19402 0.04478 0.19402
- link link_fixed_6_handle_shaft: geometry collision box size=0.195 0.195 0.995; visual box size=0.195 0.195 0.995
- link link_fixed_7_handle_knob: geometry collision box size=0.045 0.045 0.195; visual box size=0.045 0.045 0.195
- link link_fixed_9_hinge: geometry visual cylinder length=1.095 radius=0.1225
Joints:
- joint link_fixed_3_door_panel.001: origin xyz=0.999 0 0 rpy=0 0 0 -> xyz=0.995 0 0 rpy=0 0 0
- joint link_fixed_4_door_handle.001: origin xyz=1.4985 0 1.0989 rpy=0 0 0 -> xyz=1.4925 0 1.0945 rpy=0 0 0

File: puzzles/lockbox_random/urdf/lockbox_random.urdf (robot description, URDF)
Before this commit: robot lockbox_random, 22 links, 21 joints
Links:
- link goal: geometry visual box size=1.38803 0.19402 0.99002
- link link_0_joint_0: geometry collision box size=1.395 0.195 0.995; visual box size=1.395 0.195 0.995
- link link_2_joint_0: geometry collision box size=1.395 0.195 0.995; visual box size=1.395 0.195 0.995
- link link_4_joint_0: geometry collision box size=1.395 0.195 0.995; visual box size=1.395 0.195 0.995
- link link_fixed_0_floor: geometry collision box size=31.995 31.995 0.195; visual box size=31.995 31.995 0.195
- link link_fixed_10_handle_knob: geometry collision box size=0.045 0.045 0.195; visual box size=0.045 0.045 0.195
- link link_fixed_12_hinge: geometry visual cylinder length=1.095 radius=0.11062
- link link_fixed_13_handle_shaft: geometry collision cylinder length=0.995 radius=0.0975; visual cylinder length=0.995 radius=0.0975
- link link_fixed_14_handle_knob: geometry collision box size=0.045 0.045 0.195; visual box size=0.045 0.045 0.195
- link link_fixed_16_handle_shaft: geometry collision box size=0.195 0.195 0.995; visual box size=0.195 0.195 0.995
- link link_fixed_17_handle_knob: geometry collision box size=0.045 0.045 0.195; visual box size=0.045 0.045 0.195
- link link_fixed_2_handle_shaft: geometry collision box size=0.195 0.195 0.995; visual box size=0.195 0.195 0.995
- link link_fixed_2_handle_shaft.001: geometry visual box size=0.19402 0.19402 0.99002
- link link_fixed_3_handle_knob: geometry collision box size=0.045 0.045 0.195; visual box size=0.045 0.045 0.195
- link link_fixed_3_handle_knob.001: geometry visual box size=0.04478 0.04478 0.19402
- link link_fixed_5_hinge: geometry visual cylinder length=1.095 radius=0.09236
- link link_fixed_6_handle_shaft: geometry collision cylinder length=0.995 radius=0.0975; visual cylinder length=0.995 radius=0.0975
- link link_fixed_7_handle_knob: geometry collision box size=0.045 0.045 0.195; visual box size=0.045 0.045 0.195
- link link_fixed_9_handle_shaft: geometry collision box size=0.195 0.195 0.995; visual box size=0.195 0.195 0.995
Joints:
- joint link_fixed_2_handle_shaft.001: origin xyz=0 0 0.999 rpy=0 0 0 -> xyz=0 0 0.995 rpy=0 0 0
- joint link_fixed_3_handle_knob.001: origin xyz=0 0 0.5994 rpy=0 0 0 -> xyz=0 0 0.597 rpy=0 0 0

File: puzzles/simple_sliders/urdf/simple_sliders.urdf (robot description, URDF)
Before this commit: robot simple_sliders, 17 links, 16 joints
Links:
- link goal: geometry visual box size=1.58703 0.19402 0.19402
- link link_0_joint_0: geometry collision box size=1.595 0.195 0.195; visual box size=1.595 0.195 0.195
- link link_1_joint_0: geometry collision box size=1.595 0.195 0.195; visual box size=1.595 0.195 0.195
- link link_2_joint_0: geometry collision box size=1.595 0.195 0.195; visual box size=1.595 0.195 0.195
- link link_3_joint_0: geometry collision box size=1.595 0.195 0.195; visual box size=1.595 0.195 0.195
- link link_fixed_0_floor: geometry collision box size=31.995 31.995 0.195; visual box size=31.995 31.995 0.195
- link link_fixed_11_handle_shaft: geometry collision box size=0.195 0.195 0.995; visual box size=0.195 0.195 0.995
- link link_fixed_12_handle_knob: geometry collision box size=0.045 0.045 0.195; visual box size=0.045 0.045 0.195
- link link_fixed_2_handle_shaft: geometry collision box size=0.195 0.195 0.995; visual box size=0.195 0.195 0.995
- link link_fixed_2_handle_shaft.001: geometry visual box size=0.19402 0.19402 0.99002
- link link_fixed_3_handle_knob: geometry collision box size=0.045 0.045 0.195; visual box size=0.045 0.045 0.195
- link link_fixed_3_handle_knob.001: geometry visual box size=0.04478 0.04478 0.19402
- link link_fixed_5_handle_shaft: geometry collision box size=0.195 0.195 0.995; visual box size=0.195 0.195 0.995
- link link_fixed_6_handle_knob: geometry collision box size=0.045 0.045 0.195; visual box size=0.045 0.045 0.195
- link link_fixed_8_handle_shaft: geometry collision box size=0.195 0.195 0.995; visual box size=0.195 0.195 0.995
- link link_fixed_9_handle_knob: geometry collision box size=0.045 0.045 0.195; visual box size=0.045 0.045 0.195
Joints:
- joint link_fixed_2_handle_shaft.001: origin xyz=0 0 0.5994 rpy=0 0 0 -> xyz=0 0 0.597 rpy=0 0 0
- joint link_fixed_3_handle_knob.001: origin xyz=0 0 0.5994 rpy=0 0 0 -> xyz=0 0 0.597 rpy=0 0 0

Commit message: chore: update puzzles according to code changes

File: puzzles/continuous_space/urdf/continuous_space.urdf (robot description, URDF)
Before this commit: robot continuous_space, 23 links, 22 joints
Links:
- removed link link_fixed_10_handle_knob
- removed link link_fixed_2_hinge
- removed link link_fixed_2_hinge.001
- removed link link_fixed_3_handle_shaft
- removed link link_fixed_3_handle_shaft.001
- removed link link_fixed_4_handle_knob
- removed link link_fixed_4_handle_knob.001
- removed link link_fixed_60_handle_shaft
- removed link link_fixed_61_handle_knob
- removed link link_fixed_77_handle_shaft
- removed link link_fixed_78_handle_knob
- removed link link_fixed_88_hinge
- removed link link_fixed_89_handle_shaft
- removed link link_fixed_90_handle_knob
- removed link link_fixed_9_handle_shaft
- added link link_fixed_124_hinge, mass 0.001; visual cylinder length=1.095 radius=0.1225
- added link link_fixed_125_handle_shaft, mass 0.001; collision cylinder length=0.995 radius=0.0975; visual cylinder length=0.995 radius=0.0975
- added link link_fixed_126_handle_knob, mass 0.001; collision box size=0.045 0.045 0.195; visual box size=0.045 0.045 0.195
- added link link_fixed_14_handle_shaft, mass 0.001; collision box size=0.195 0.195 0.995; visual box size=0.195 0.195 0.995
- added link link_fixed_152_handle_shaft, mass 0.001; collision box size=0.195 0.195 0.995; visual box size=0.195 0.195 0.995
- added link link_fixed_153_handle_knob, mass 0.001; collision box size=0.045 0.045 0.195; visual box size=0.045 0.045 0.195
- added link link_fixed_15_handle_knob, mass 0.001; collision box size=0.045 0.045 0.195; visual box size=0.045 0.045 0.195
- added link link_fixed_2_handle_shaft, mass 0.001; collision box size=0.195 0.195 0.995; visual box size=0.195 0.195 0.995
- added link link_fixed_2_handle_shaft.001, mass 0.001; visual box size=0.19402 0.19402 0.99002
- added link link_fixed_3_handle_knob, mass 0.001; collision box size=0.045 0.045 0.195; visual box size=0.045 0.045 0.195
- added link link_fixed_3_handle_knob.001, mass 0.001; visual box size=0.04477 0.04477 0.19402
- added link link_fixed_62_hinge, mass 0.001; visual cylinder length=1.095 radius=0.1225
- added link link_fixed_63_handle_shaft, mass 0.001; collision cylinder length=0.995 radius=0.0975; visual cylinder length=0.995 radius=0.0975
- added link link_fixed_64_handle_knob, mass 0.001; collision box size=0.045 0.045 0.195; visual box size=0.045 0.045 0.195
- link goal: geometry visual box size=1.98503 0.99002 0.99002
- link link_0_joint_0: geometry collision box size=1.995 0.995 0.995; visual box size=1.995 0.995 0.995
- link link_2_joint_0: geometry collision box size=2.995 0.995 0.995; visual box size=2.995 0.995 0.995
- link link_3_joint_0: geometry collision box size=2.995 0.995 0.995; visual box size=2.995 0.995 0.995
- link link_4_joint_0: geometry collision box size=1.995 0.995 0.995; visual box size=1.995 0.995 0.995
Joints:
- removed joint link_fixed_10_handle_knob
- removed joint link_fixed_2_hinge
- removed joint link_fixed_2_hinge.001
- removed joint link_fixed_3_handle_shaft
- removed joint link_fixed_3_handle_shaft.001
- removed joint link_fixed_4_handle_knob
- removed joint link_fixed_4_handle_knob.001
- removed joint link_fixed_60_handle_shaft
- removed joint link_fixed_61_handle_knob
- removed joint link_fixed_77_handle_shaft
- removed joint link_fixed_78_handle_knob
- removed joint link_fixed_88_hinge
- removed joint link_fixed_89_handle_shaft
- removed joint link_fixed_90_handle_knob
- removed joint link_fixed_9_handle_shaft
- added joint link_fixed_124_hinge: type fixed, parent link_3_joint_0, child link_fixed_124_hinge, origin xyz=0 0 0 rpy=0 0 0
- added joint link_fixed_125_handle_shaft: type fixed, parent link_3_joint_0, child link_fixed_125_handle_shaft, origin xyz=1.125 0 1.0 rpy=0 0 0
- added joint link_fixed_126_handle_knob: type fixed, parent link_fixed_125_handle_shaft, child link_fixed_126_handle_knob, origin xyz=0 0 0.6 rpy=0 0 0
- added joint link_fixed_14_handle_shaft: type fixed, parent link_1_joint_0, child link_fixed_14_handle_shaft, origin xyz=0 0 1.0 rpy=0 0 0
- added joint link_fixed_152_handle_shaft: type fixed, parent link_4_joint_0, child link_fixed_152_handle_shaft, origin xyz=0 0 1.0 rpy=0 0 0
- added joint link_fixed_153_handle_knob: type fixed, parent link_fixed_152_handle_shaft, child link_fixed_153_handle_knob, origin xyz=0 0 0.6 rpy=0 0 0
- added joint link_fixed_15_handle_knob: type fixed, parent link_fixed_14_handle_shaft, child link_fixed_15_handle_knob, origin xyz=0 0 0.6 rpy=0 0 0
- added joint link_fixed_2_handle_shaft: type fixed, parent link_0_joint_0, child link_fixed_2_handle_shaft, origin xyz=0 0 1.0 rpy=0 0 0
- added joint link_fixed_2_handle_shaft.001: type fixed, parent goal, child link_fixed_2_handle_shaft.001, origin xyz=0 0 0.995 rpy=0 0 0
- added joint link_fixed_3_handle_knob: type fixed, parent link_fixed_2_handle_shaft, child link_fixed_3_handle_knob, origin xyz=0 0 0.6 rpy=0 0 0
- added joint link_fixed_3_handle_knob.001: type fixed, parent link_fixed_2_handle_shaft.001, child link_fixed_3_handle_knob.001, origin xyz=0 0 0.597 rpy=0 0 0
- added joint link_fixed_62_hinge: type fixed, parent link_2_joint_0, child link_fixed_62_hinge, origin xyz=0 0 0 rpy=0 0 0
- added joint link_fixed_63_handle_shaft: type fixed, parent link_2_joint_0, child link_fixed_63_handle_shaft, origin xyz=1.125 0 1.0 rpy=0 0 0
- added joint link_fixed_64_handle_knob: type fixed, parent link_fixed_63_handle_shaft, child link_fixed_64_handle_knob, origin xyz=0 0 0.6 rpy=0 0 0
- joint goal: origin xyz=0 0 0.5 rpy=0 0 -0.23802 -> xyz=0.99739 -2.4812 0.5 rpy=0 0 -1.18859
- joint link_0_joint_0: axis 0 0 1.0 -> 1.0 0 0; limit lower=0 upper=3.06691 effort=0 velocity=0 -> lower=0 upper=2.67416 effort=0 velocity=0; origin xyz=0 0 0.5 rpy=0 0 2.97826 -> xyz=0 0 0.5 rpy=0 0 -1.18859; type revolute -> prismatic
- joint link_1_joint_0: limit lower=0 upper=3.94912 effort=0 velocity=0 -> lower=0 upper=3.11295 effort=0 velocity=0; origin xyz=0.21644 -1.77687 0.5 rpy=0 0 -0.77445 -> xyz=-0.03422 -3.00526 0.5 rpy=0 0 -2.29454
- joint link_2_joint_0: axis 1.0 0 0 -> 0 0 1.0; limit lower=0 upper=2.74264 effort=0 velocity=0 -> lower=0 upper=2.87617 effort=0 velocity=0; origin xyz=-0.02039 1.94214 0.5 rpy=0 0 0.74579 -> xyz=-1.10798 -5.00962 0.5 rpy=0 0 -1.25698; type prismatic -> revolute
- joint link_3_joint_0: axis 1.0 0 0 -> 0 0 1.0; limit lower=0 upper=2.52402 effort=0 velocity=0 -> lower=-2.54743 upper=0 effort=0 velocity=0; origin xyz=1.38858 -3.83648 0.5 rpy=0 0 -2.62206 -> xyz=2.8631 -3.5405 0.5 rpy=0 0 -3.02217; type prismatic -> revolute
- joint link_4_joint_0: axis 0 0 1.0 -> 1.0 0 0; limit lower=0 upper=3.09983 effort=0 velocity=0 -> lower=0 upper=3.4642 effort=0 velocity=0; origin xyz=-0.63097 -6.0368 0.5 rpy=0 0 -2.05119 -> xyz=3.4627 -1.85032 0.5 rpy=0 0 1.59111; type revolute -> prismatic

File: puzzles/escape_room/urdf/escape_room.urdf (robot description, URDF)
Before this commit: robot escape_room, 19 links, 18 joints
Links:
- link link_fixed_9_door_panel: geometry collision box size=3.195 0.195 0.99; visual box size=3.195 0.195 0.99

File: puzzles/lockbox2017/urdf/lockbox2017.urdf (robot description, URDF)
Before this commit: robot lockbox2017, 24 links, 23 joints
Links:
- link link_fixed_17_door_panel: geometry collision box size=3.995 0.195 1.99; visual box size=3.995 0.195 1.99
- link link_fixed_3_door_panel: geometry collision box size=1.995 0.195 1.99; visual box size=1.995 0.195 1.99
- link link_fixed_3_door_panel.001: geometry visual box size=1.98503 0.19402 1.98005

File: puzzles/lockbox_random/urdf/lockbox_random.urdf (robot description, URDF)
Before this commit: robot lockbox_random, 22 links, 21 joints
Links:
- link link_fixed_12_hinge: geometry visual cylinder length=1.095 radius=0.15375
- link link_fixed_5_hinge: geometry visual cylinder length=1.095 radius=0.1225
Joints:
- joint link_1_joint_0: origin xyz=-2.51783 0 0.5 rpy=0 0 3.14159 -> xyz=-3.0 0 0.5 rpy=0 0 3.14159
- joint link_2_joint_0: origin xyz=-4.03566 0 0.5 rpy=0 0 3.14159 -> xyz=-5.0 0 0.5 rpy=0 0 3.14159
- joint link_3_joint_0: origin xyz=-6.84553 0 0.5 rpy=0 0 3.14159 -> xyz=-8.5 0 0.5 rpy=0 0 3.14159
- joint link_4_joint_0: origin xyz=-8.6554 0 0.5 rpy=0 0 3.14159 -> xyz=-11.0 0 0.5 rpy=0 0 3.14159
- joint link_fixed_13_handle_shaft: origin xyz=0 1.3574 1.0 rpy=0 0 0 -> xyz=0 1.875 1.0 rpy=0 0 0
- joint link_fixed_6_handle_shaft: origin xyz=0 1.13838 1.0 rpy=0 0 0 -> xyz=0 1.5 1.0 rpy=0 0 0
