Commit message: fix: enable mesh output in phobos

File: puzzles/my_custom/urdf/my_custom.urdf (robot description, URDF)
Before this commit: robot my_custom, 6 links, 5 joints
Links:
- removed link link3
- removed link link4
- link link2: geometry collision mesh filename=file:///home/userone/ba/puzzle-generator/puzzles/my_custom/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 scale=1.0 1.0 1.0; visual mesh filename=file:///home/userone/ba/puzzle-generator/puzzles/my_custom/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 scale=2.0 2.0 0.5
Joints:
- removed joint link3
- removed joint link4
- joint link2: limit lower=0 upper=0 effort=0 velocity=0 -> lower=-0.7854 upper=0.7854 effort=0 velocity=0; origin xyz=0 4.0 0.1 rpy=0 0 0 -> xyz=0 -5.0 0.5 rpy=0 0 0; type prismatic -> revolute

Commit message: refactor: automatically create collision when adding new objects to the scene

File: puzzles/my_custom/urdf/my_custom.urdf (robot description, URDF)
Before this commit: robot my_custom, 4 links, 3 joints
Joints:
- joint link0: origin xyz=0 5.0 2.0 rpy=0 0 0 -> xyz=0 5.0 2.1 rpy=0 0 0
- joint link1: origin xyz=0 0 0.5 rpy=-1.5708 0 0.7854 -> xyz=0 0 0.6 rpy=-1.5708 0 0.7854
- joint link2: origin xyz=0 -5.0 0.5 rpy=0 0 0 -> xyz=0 -5.0 0.6 rpy=0 0 0

Commit message: feat: new_object() can take child_visuals to become parent of them remove unnecessary shape argument from create_collision()

File: puzzles/my_custom/urdf/my_custom.urdf (robot description, URDF)
Before this commit: robot my_custom, 4 links, 3 joints
Links:
- link link0: geometry collision box size=2.0 1.0 2.0; collision cylinder length=2.0 radius=0.5
Joints:
- joint link0: origin xyz=0 5.0 2.1 rpy=0 0 0 -> xyz=0 5.0 1.1 rpy=0 0 0

Commit message: feat: name can be specified in new_object() improve default naming/numbering of objects

File: puzzles/my_custom/urdf/my_custom.urdf (robot description, URDF)
Before this commit: robot my_custom, 4 links, 3 joints
Links:
- removed link link0
- removed link link1
- removed link link2
- added link link_0, mass 0.001; collision box size=2.0 1.0 2.0; collision cylinder length=2.0 radius=0.5
- added link link_1, mass 0.001; collision box size=1.0 1.0 4.0; visual box size=1.0 1.0 4.0
- added link link_2, mass 0.001; collision mesh filename=file:///home/userone/ba/puzzle-generator/puzzles/my_custom/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 scale=1.0 1.0 1.0; visual mesh filename=file:///home/userone/ba/puzzle-generator/puzzles/my_custom/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 scale=1.0 1.0 1.0
Joints:
- removed joint link0
- removed joint link1
- removed joint link2
- added joint link_0: type revolute, parent base_link, child link_0, origin xyz=0 5.0 1.1 rpy=0 0 0, axis 0 0 1.0, limit lower=-0.7854 upper=0.7854 effort=0 velocity=0
- added joint link_1: type prismatic, parent base_link, child link_1, origin xyz=0 0 0.6 rpy=-1.5708 0 0.7854, axis 0 0 1.0, limit lower=0 upper=2.0 effort=0 velocity=0
- added joint link_2: type revolute, parent base_link, child link_2, origin xyz=0 -5.0 0.6 rpy=0 0 0, axis 0 0 1.0, limit lower=-0.7854 upper=0.7854 effort=0 velocity=0

Commit message: feat: add new_door() simplify the creation of this specific type of revolute joint, add determine_link_color()

File: puzzles/my_custom/urdf/my_custom.urdf (robot description, URDF)
Before this commit: robot my_custom, 4 links, 3 joints
Links:
- added link link_door_3, mass 0.001; collision box size=2.0 0.2 4.0; collision cylinder length=4.0 radius=0.2
Joints:
- added joint link_door_3: type revolute, parent base_link, child link_door_3, origin xyz=4.0 4.0 2.1 rpy=0 0 0, axis 0 0 1.0, limit lower=0 upper=1.5708 effort=0 velocity=0

Commit message: feat: add door handle, add default name for door simplify naming of blender objects in new_link()

File: puzzles/my_custom/urdf/my_custom.urdf (robot description, URDF)
Before this commit: robot my_custom, 5 links, 4 joints
Links:
- link link_door_3: geometry collision box size=0.2 0.2 0.2; collision box size=2.0 0.2 4.0

Commit message: fix: add second handle for door

File: puzzles/my_custom/urdf/my_custom.urdf (robot description, URDF)
Before this commit: robot my_custom, 5 links, 4 joints
Links:
- link link_door_3: geometry collision box size=0.2 0.2 0.2; collision box size=0.2 0.2 0.2

Commit message: feat: door handle can be placed on top

File: puzzles/my_custom/urdf/my_custom.urdf (robot description, URDF)
Before this commit: robot my_custom, 5 links, 4 joints
Links:
- added link link_door_4, mass 0.001; collision box size=0.2 0.05 0.2; collision box size=2.0 0.2 4.0
- link link_door_3: geometry collision box size=0.05 0.2 0.2; collision box size=0.05 0.2 0.2
Joints:
- added joint link_door_4: type revolute, parent base_link, child link_door_4, origin xyz=4.0 -4.0 2.1 rpy=0 0 0, axis 0 0 1.0, limit lower=0 upper=1.5708 effort=0 velocity=0

Commit message: fix: add link_is_child parameter in determine_link_color()

File: puzzles/my_custom/urdf/my_custom.urdf (robot description, URDF)
Before this commit: robot my_custom, 11 links, 10 joints
Links:
- removed link link_0
- removed link link_1
- removed link link_door_3
- removed link link_door_4
- removed link link_door_handle1_5
- removed link link_door_handle2_5
- removed link link_door_handle_4
- removed link link_door_panel_4
- removed link link_door_panel_5
- added link link_3, mass 0.001; collision box size=1.0 1.0 4.0; visual box size=1.0 1.0 4.0
- added link link_4, mass 0.001; collision mesh filename=file:///home/userone/ba/puzzle-generator/puzzles/my_custom/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 scale=1.0 1.0 1.0; visual mesh filename=file:///home/userone/ba/puzzle-generator/puzzles/my_custom/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 scale=1.0 1.0 1.0
- added link link_door_0, mass 0.001; collision cylinder length=4.0 radius=0.2; visual cylinder length=4.0 radius=0.2
- added link link_door_1, mass 0.001; collision cylinder length=4.0 radius=0.2; visual cylinder length=4.0 radius=0.2
- added link link_door_handle1_2, mass 0.001; collision box size=0.05 0.2 0.2; visual box size=0.05 0.2 0.2
- added link link_door_handle2_2, mass 0.001; collision box size=0.05 0.2 0.2; visual box size=0.05 0.2 0.2
- added link link_door_handle_1, mass 0.001; collision box size=0.2 0.05 0.2; visual box size=0.2 0.05 0.2
- added link link_door_panel_1, mass 0.001; collision box size=2.0 0.2 4.0; visual box size=2.0 0.2 4.0
- added link link_door_panel_2, mass 0.001; collision box size=2.0 0.2 4.0; visual box size=2.0 0.2 4.0
- link link_2: geometry collision cylinder length=2.0 radius=0.5; visual cylinder length=2.0 radius=0.5
Joints:
- removed joint link_0
- removed joint link_1
- removed joint link_door_3
- removed joint link_door_4
- removed joint link_door_handle1_5
- removed joint link_door_handle2_5
- removed joint link_door_handle_4
- removed joint link_door_panel_4
- removed joint link_door_panel_5
- added joint link_3: type prismatic, parent base_link, child link_3, origin xyz=0 0 0.6 rpy=-1.5708 0 0.7854, axis 0 0 1.0, limit lower=0 upper=2.0 effort=0 velocity=0
- added joint link_4: type revolute, parent base_link, child link_4, origin xyz=0 -5.0 0.6 rpy=0 0 0, axis 0 0 1.0, limit lower=-0.7854 upper=0.7854 effort=0 velocity=0
- added joint link_door_0: type revolute, parent base_link, child link_door_0, origin xyz=4.0 4.0 2.1 rpy=0 0 0, axis 0 0 1.0, limit lower=0 upper=1.5708 effort=0 velocity=0
- added joint link_door_1: type revolute, parent base_link, child link_door_1, origin xyz=4.0 -4.0 2.1 rpy=0 0 0, axis 0 0 1.0, limit lower=-1.5708 upper=0.7854 effort=0 velocity=0
- added joint link_door_handle1_2: type fixed, parent link_door_1, child link_door_handle1_2, origin xyz=1.5 0.2 0 rpy=0 0 0
- added joint link_door_handle2_2: type fixed, parent link_door_1, child link_door_handle2_2, origin xyz=1.5 -0.2 0 rpy=0 0 0
- added joint link_door_handle_1: type fixed, parent link_door_0, child link_door_handle_1, origin xyz=1.5 0 2.1 rpy=0 0 0
- added joint link_door_panel_1: type fixed, parent link_door_0, child link_door_panel_1, origin xyz=1.0 0 0 rpy=0 0 0
- added joint link_door_panel_2: type fixed, parent link_door_1, child link_door_panel_2, origin xyz=1.0 0 0 rpy=0 0 0
- joint link_2: origin xyz=0 -5.0 0.6 rpy=0 0 0 -> xyz=0 5.0 1.1 rpy=0 0 0

Commit message: chore (minor): update config according to new structure

File: puzzles/my_custom/urdf/my_custom.urdf (robot description, URDF)
Before this commit: robot my_custom, 21 links, 20 joints
Links:
- removed link link_door_0
- removed link link_door_1
- added link link_0, mass 0.001; collision cylinder length=4.0 radius=0.2; visual cylinder length=4.0 radius=0.2
- added link link_1, mass 0.001; collision cylinder length=4.0 radius=0.2; visual cylinder length=4.0 radius=0.2
- link link_hinge_0: geometry visual cylinder length=4.1 radius=0.05
- link link_hinge_1: geometry visual cylinder length=4.1 radius=0.05
- link link_hinge_2: geometry visual cylinder length=2.1 radius=0.05
- link link_hinge_4: geometry visual cylinder length=1.1 radius=0.05
Joints:
- removed joint link_door_0
- removed joint link_door_1
- added joint link_0: type revolute, parent base_link, child link_0, origin xyz=4.0 4.0 2.1 rpy=0 0 0, axis 0 0 1.0, limit lower=0 upper=1.5708 effort=0 velocity=0
- added joint link_1: type revolute, parent base_link, child link_1, origin xyz=4.0 -4.0 2.1 rpy=0 0 0, axis 0 0 1.0, limit lower=-1.5708 upper=0.7854 effort=0 velocity=0
- joint link_door_handle1_1: parent link_door_1 -> link_1
- joint link_door_handle2_1: parent link_door_1 -> link_1
- joint link_door_handle_0: parent link_door_0 -> link_0
- joint link_door_panel_0: parent link_door_0 -> link_0
- joint link_door_panel_1: parent link_door_1 -> link_1
- joint link_hinge_0: parent link_door_0 -> link_0
- joint link_hinge_1: parent link_door_1 -> link_1

Commit message: feat: add droids to my_custom.urdf

File: puzzles/my_custom/urdf/my_custom.urdf (robot description, URDF)
Before this commit: robot my_custom, 5 links, 4 joints
Links:
- added link link_1_fixed_joint_1_handle_shaft, mass 0.001; collision cylinder length=1.0 radius=0.1; visual cylinder length=1.0 radius=0.1
- added link link_1_fixed_joint_2_handle_knob, mass 0.001; collision box size=0.05 0.05 0.2; visual box size=0.05 0.05 0.2
- added link link_1_fixed_joint_3_hinge, mass 0.001; visual cylinder length=1.1 radius=0.05
- added link link_1_joint_0, mass 0.001; collision mesh filename=file:///home/userone/ba/puzzle-generator/puzzles/my_custom/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 scale=1.0 1.0 1.0; visual mesh filename=file:///home/userone/ba/puzzle-generator/puzzles/my_custom/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 scale=4.0 4.0 1.0
- added link link_2_fixed_joint_1_handle_shaft, mass 0.001; collision cylinder length=1.0 radius=0.1; visual cylinder length=1.0 radius=0.1
- added link link_2_fixed_joint_2_handle_knob, mass 0.001; collision box size=0.05 0.05 0.2; visual box size=0.05 0.05 0.2
- added link link_2_fixed_joint_3_hinge, mass 0.001; visual cylinder length=1.1 radius=0.05
- added link link_2_joint_0, mass 0.001; collision mesh filename=file:///home/userone/ba/puzzle-generator/puzzles/my_custom/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 scale=1.0 1.0 1.0; visual mesh filename=file:///home/userone/ba/puzzle-generator/puzzles/my_custom/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 scale=2.0 2.0 1.0
- link link_0_joint_2: geometry collision mesh filename=file:///home/userone/ba/puzzle-generator/puzzles/my_custom/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 scale=1.0 1.0 1.0; visual mesh filename=file:///home/userone/ba/puzzle-generator/puzzles/my_custom/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 scale=0.75 1.0 1.0
Joints:
- added joint link_1_fixed_joint_1_handle_shaft: type fixed, parent link_1_joint_0, child link_1_fixed_joint_1_handle_shaft, origin xyz=0 1.5 1.0 rpy=0 0 0
- added joint link_1_fixed_joint_2_handle_knob: type fixed, parent link_1_fixed_joint_1_handle_shaft, child link_1_fixed_joint_2_handle_knob, origin xyz=0 0 0.6 rpy=0 0 0
- added joint link_1_fixed_joint_3_hinge: type fixed, parent link_1_joint_0, child link_1_fixed_joint_3_hinge, origin xyz=0 0 0 rpy=0 0 0
- added joint link_1_joint_0: type revolute, parent base_link, child link_1_joint_0, origin xyz=0 -5.0 0.6 rpy=0 0 0, axis 0 0 1.0, limit lower=-0.7854 upper=0.7854 effort=0 velocity=0
- added joint link_2_fixed_joint_1_handle_shaft: type fixed, parent link_2_joint_0, child link_2_fixed_joint_1_handle_shaft, origin xyz=0 0.75 1.0 rpy=0 0 0
- added joint link_2_fixed_joint_2_handle_knob: type fixed, parent link_2_fixed_joint_1_handle_shaft, child link_2_fixed_joint_2_handle_knob, origin xyz=0 0 0.6 rpy=0 0 0
- added joint link_2_fixed_joint_3_hinge: type fixed, parent link_2_joint_0, child link_2_fixed_joint_3_hinge, origin xyz=0 0 0 rpy=0 0 0
- added joint link_2_joint_0: type revolute, parent base_link, child link_2_joint_0, origin xyz=0 5.0 0.6 rpy=0 0 0, axis 0 0 1.0, limit lower=-0.7854 upper=0.7854 effort=0 velocity=0
- joint link_0_joint_2: limit lower=0 upper=2.0 effort=0 velocity=0 -> lower=-3.14159 upper=3.14159 effort=0 velocity=0
