Commit message: feat: add EscapeRoomSampler()

File: puzzles/escape_room/urdf/escape_room.urdf (robot description, URDF)
Before this commit: robot my_custom, 13 links, 12 joints
Links:
- removed link link_1_fixed_joint_1_handle_shaft
- removed link link_1_fixed_joint_2_handle_knob
- removed link link_1_fixed_joint_3_hinge
- removed link link_2_fixed_joint_1_handle_shaft
- removed link link_2_fixed_joint_2_handle_knob
- removed link link_2_fixed_joint_3_hinge
- removed link link_2_joint_0
- added link goal, mass 0.001; visual box size=0 0 0
- added link link_0_fixed_joint_3_hinge.001, mass 0.001; visual cylinder length=1.1 radius=0.05
- added link link_0_joint_1.001, mass 0.001; visual box size=0 0 0
- added link link_0_joint_2.001, mass 0.001; visual mesh filename=file:///home/userone/ba/puzzle-generator/puzzles/escape_roo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 scale=1.0 1.0 1.0
- added link link_1_fixed_joint_1_hinge, mass 0.001; visual cylinder length=1.1 radius=0.05
- added link link_1_fixed_joint_2_door_panel, mass 0.001; collision box size=2.0 0.2 1.0; visual box size=2.0 0.2 1.0
- added link link_1_fixed_joint_3_door_handle1, mass 0.001; collision box size=0.05 0.2 0.2; visual box size=0.05 0.2 0.2
- added link link_1_fixed_joint_4_door_handle2, mass 0.001; collision box size=0.05 0.2 0.2; visual box size=0.05 0.2 0.2
- added link link_2_fixed_joint_0_wall1, mass 0.001; collision box size=4.0 0.2 1.0; visual box size=4.0 0.2 1.0
- added link link_2_fixed_joint_0_wall2, mass 0.001; collision box size=4.0 0.2 1.0; visual box size=4.0 0.2 1.0
- added link link_2_fixed_joint_0_wall3, mass 0.001; collision box size=0.2 2.0 1.0; visual box size=0.2 2.0 1.0
- link link_0_joint_2: geometry collision mesh filename=file:///home/userone/ba/puzzle-generator/puzzles/escape_roo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 scale=1.0 1.0 1.0; visual mesh filename=file:///home/userone/ba/puzzle-generator/puzzles/escape_roo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 scale=1.0 1.0 1.0
- link link_1_joint_0: geometry collision cylinder length=1.0 radius=0.2; visual cylinder length=1.0 radius=0.2
Joints:
- removed joint link_1_fixed_joint_1_handle_shaft
- removed joint link_1_fixed_joint_2_handle_knob
- removed joint link_1_fixed_joint_3_hinge
- removed joint link_2_fixed_joint_1_handle_shaft
- removed joint link_2_fixed_joint_2_handle_knob
- removed joint link_2_fixed_joint_3_hinge
- removed joint link_2_joint_0
- added joint goal: type fixed, parent base_link, child goal, origin xyz=4.0 0 0.6 rpy=0 0 1.5708, limit effort=0 velocity=0
- added joint link_0_fixed_joint_3_hinge.001: type fixed, parent link_0_joint_2.001, child link_0_fixed_joint_3_hinge.001, origin xyz=0 0 0 rpy=0 0 0
- added joint link_0_joint_1.001: type fixed, parent goal, child link_0_joint_1.001, origin xyz=0 0 0 rpy=0 0 0, limit effort=0 velocity=0
- added joint link_0_joint_2.001: type fixed, parent link_0_joint_1.001, child link_0_joint_2.001, origin xyz=0 0 0 rpy=0 0 0, limit effort=0 velocity=0
- added joint link_1_fixed_joint_1_hinge: type fixed, parent link_1_joint_0, child link_1_fixed_joint_1_hinge, origin xyz=0 0 0 rpy=0 0 0
- added joint link_1_fixed_joint_2_door_panel: type fixed, parent link_1_joint_0, child link_1_fixed_joint_2_door_panel, origin xyz=1.0 0 0 rpy=0 0 0
- added joint link_1_fixed_joint_3_door_handle1: type fixed, parent link_1_joint_0, child link_1_fixed_joint_3_door_handle1, origin xyz=1.5 0.2 0 rpy=0 0 0
- added joint link_1_fixed_joint_4_door_handle2: type fixed, parent link_1_joint_0, child link_1_fixed_joint_4_door_handle2, origin xyz=1.5 -0.2 0 rpy=0 0 0
- added joint link_2_fixed_joint_0_wall1: type fixed, parent base_link, child link_2_fixed_joint_0_wall1, origin xyz=0 -1.4 0.6 rpy=0 0 0
- added joint link_2_fixed_joint_0_wall2: type fixed, parent base_link, child link_2_fixed_joint_0_wall2, origin xyz=0 1.4 0.6 rpy=0 0 0
- added joint link_2_fixed_joint_0_wall3: type fixed, parent base_link, child link_2_fixed_joint_0_wall3, origin xyz=-2.0 0 0.6 rpy=0 0 0
- joint link_1_joint_0: limit lower=-0.7854 upper=0.7854 effort=0 velocity=0 -> lower=0 upper=1.5708 effort=0 velocity=0; origin xyz=0 -5.0 0.6 rpy=0 0 0 -> xyz=2.0 -1.0 0.6 rpy=0 0 1.5708

Commit message: chore (minor): reduce joint bounds in escape_room

File: puzzles/escape_room/urdf/escape_room.urdf (robot description, URDF)
Before this commit: robot escape_room, 21 links, 20 joints
Links:
- link link_10_fixed_door_panel: geometry collision box size=3.199 0.199 0.999; visual box size=3.199 0.199 0.999
- link link_1_joint_0: geometry collision box size=3.499 0.349 0.249; visual box size=3.499 0.349 0.249
- link link_7_fixed_hinge: geometry visual cylinder length=0.274 radius=0.04325
Joints:
- joint link_0_joint_1: limit lower=-16.0 upper=16.0 effort=0 velocity=0 -> lower=-6.0 upper=6.0 effort=0 velocity=0
- joint link_0_joint_2: limit lower=-16.0 upper=16.0 effort=0 velocity=0 -> lower=-6.0 upper=6.0 effort=0 velocity=0
- joint link_10_fixed_door_panel: origin xyz=1.5 0 0 rpy=0 0 0 -> xyz=1.6 0 0 rpy=0 0 0
- joint link_11_fixed_door_handle1: origin xyz=2.25 0.2 0 rpy=0 0 0 -> xyz=2.4 0.2 0 rpy=0 0 0
- joint link_12_fixed_door_handle2: origin xyz=2.25 -0.2 0 rpy=0 0 0 -> xyz=2.4 -0.2 0 rpy=0 0 0
- joint link_1_joint_1: limit lower=-16.0 upper=16.0 effort=0 velocity=0 -> lower=-6.0 upper=6.0 effort=0 velocity=0
- joint link_1_joint_2: limit lower=-16.0 upper=16.0 effort=0 velocity=0 -> lower=-6.0 upper=6.0 effort=0 velocity=0
