Commit message: feat: support concave meshes in pybullet

File: puzzles/lockbox2017/urdf/lockbox2017.urdf (robot description, URDF)
Before this commit: robot lockbox2017, 3 links, 2 joints
Links:
- link link0: geometry collision box size=0.8 1.0 3.4; visual box size=0.8 1.0 3.4
- link link1: geometry collision mesh filename=file:///home/userone/ba/puzzle-generator/puzzles/lockbox201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 scale=1.0 1.0 1.0; visual mesh filename=file:///home/userone/ba/puzzle-generator/puzzles/lockbox201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 scale=2.0 2.0 0.5
Joints:
- joint link0: limit lower=0 upper=1.0 effort=0 velocity=0 -> lower=0 upper=2.0 effort=0 velocity=0; origin xyz=3.0 0 0.6 rpy=-1.5708 0 1.5708 -> xyz=2.0 0 0.6 rpy=-1.5708 0 -1.5708
- joint link1: limit lower=-6.28319 upper=6.28319 effort=0 velocity=0 -> lower=-3.14159 upper=3.14159 effort=0 velocity=0

Commit message: chore: add missing joints to lockbox2017

File: puzzles/lockbox2017/urdf/lockbox2017.urdf (robot description, URDF)
Before this commit: robot lockbox2017, 3 links, 2 joints
Links:
- added link link2, mass 0.001; collision mesh filename=file:///home/userone/ba/puzzle-generator/puzzles/lockbox201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 scale=1.0 1.0 1.0; visual mesh filename=file:///home/userone/ba/puzzle-generator/puzzles/lockbox201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 scale=2.0 2.0 0.5
- added link link3, mass 0.001; collision box size=0.8 1.0 3.6; visual box size=0.8 1.0 3.6
- added link link4, mass 0.001; collision box size=3.6 0.8 1.0; visual box size=3.6 0.8 1.0
- link link0: geometry collision box size=3.6 0.8 1.0; visual box size=3.6 0.8 1.0
- link link1: geometry collision box size=0.8 1.0 3.6; visual box size=0.8 1.0 3.6
Joints:
- added joint link2: type revolute, parent base_link, child link2, origin xyz=0 0 0.6 rpy=0 0 1.5708, axis 0 0 1.0, limit lower=-3.14159 upper=3.14159 effort=0 velocity=0
- added joint link3: type prismatic, parent base_link, child link3, origin xyz=0 2.0 0.6 rpy=-1.5708 0 0, axis 0 0 1.0, limit lower=0 upper=2.0 effort=0 velocity=0
- added joint link4: type revolute, parent base_link, child link4, origin xyz=-1.0 5.0 0.6 rpy=0 0 0, axis 0 0 1.0, limit lower=0 upper=1.5708 effort=0 velocity=0
- joint link0: limit lower=0 upper=2.0 effort=0 velocity=0 -> lower=0 upper=1.5708 effort=0 velocity=0; origin xyz=2.0 0 0.6 rpy=-1.5708 0 -1.5708 -> xyz=-6.0 -1.0 0.6 rpy=0 0 0; type prismatic -> revolute
- joint link1: limit lower=-3.14159 upper=3.14159 effort=0 velocity=0 -> lower=0 upper=2.0 effort=0 velocity=0; origin xyz=0 0 0.6 rpy=0 0 0 -> xyz=-4.0 0 0.6 rpy=-1.5708 0 -1.5708; type revolute -> prismatic

Commit message: feat: create_visual() can create cylinders

File: puzzles/lockbox2017/urdf/lockbox2017.urdf (robot description, URDF)
Before this commit: robot lockbox2017, 6 links, 5 joints
Links:
- link link2: geometry collision mesh filename=file:///home/userone/ba/puzzle-generator/puzzles/lockbox201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 scale=1.0 1.0 1.0; visual mesh filename=file:///home/userone/ba/puzzle-generator/puzzles/lockbox201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 scale=1.0 1.0 1.0

File: puzzles/my_custom/urdf/my_custom.urdf (robot description, URDF)
Before this commit: robot my_custom, 4 links, 3 joints
Links:
- link link2: geometry collision mesh filename=file:///home/userone/ba/puzzle-generator/puzzles/my_custom/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 scale=1.0 1.0 1.0; visual mesh filename=file:///home/userone/ba/puzzle-generator/puzzles/my_custom/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 scale=1.0 1.0 1.0

Commit message: chore: use new door objects for lockbox2017

File: puzzles/lockbox2017/urdf/lockbox2017.urdf (robot description, URDF)
Before this commit: robot lockbox2017, 6 links, 5 joints
Links:
- removed link link_0
- removed link link_4
- added link link_door_0, mass 0.001; collision box size=0.2 0.05 0.2; collision box size=2.0 0.2 2.0
- added link link_door_4, mass 0.001; collision box size=0.2 0.05 0.2; collision box size=4.0 0.2 2.0
Joints:
- removed joint link_0
- removed joint link_4
- added joint link_door_0: type revolute, parent base_link, child link_door_0, origin xyz=-6.0 -1.0 0.6 rpy=0 0 0, axis 0 0 1.0, limit lower=0 upper=1.5708 effort=0 velocity=0
- added joint link_door_4: type revolute, parent base_link, child link_door_4, origin xyz=-2.0 4.0 1.1 rpy=0 0 0, axis 0 0 1.0, limit lower=0 upper=1.5708 effort=0 velocity=0
- joint link_2: limit lower=-3.14159 upper=3.14159 effort=0 velocity=0 -> lower=0 upper=1.5708 effort=0 velocity=0

File: puzzles/my_custom/urdf/my_custom.urdf (robot description, URDF)
Before this commit: robot my_custom, 6 links, 5 joints
Links:
- link link_door_3: geometry collision box size=0.2 0.05 0.2; collision box size=2.0 0.2 4.0
- link link_door_4: geometry collision box size=0.05 0.2 0.2; collision box size=0.05 0.2 0.2
Joints:
- joint link_door_4: limit lower=0 upper=1.5708 effort=0 velocity=0 -> lower=-1.5708 upper=0.7854 effort=0 velocity=0

Commit message: feat (minor): manually add handle to slider through child visuals

File: puzzles/lockbox2017/urdf/lockbox2017.urdf (robot description, URDF)
Before this commit: robot lockbox2017, 6 links, 5 joints
Links:
- link link_1: geometry collision box size=0.2 0.2 0.05; collision box size=0.8 1.0 3.6
- link link_3: geometry collision box size=0.2 0.2 0.05; collision box size=0.8 1.0 3.6

Commit message: feat: remove the feature of adding multiple visual/collision objects to one link create multiple links instead

File: puzzles/lockbox2017/urdf/lockbox2017.urdf (robot description, URDF)
Before this commit: robot lockbox2017, 6 links, 5 joints
Links:
- added link link_door_handle_1, mass 0.001; collision box size=0.2 0.05 0.2; visual box size=0.2 0.05 0.2
- added link link_door_handle_5, mass 0.001; collision box size=0.2 0.05 0.2; visual box size=0.2 0.05 0.2
- added link link_door_panel_1, mass 0.001; collision box size=2.0 0.2 2.0; visual box size=2.0 0.2 2.0
- added link link_door_panel_5, mass 0.001; collision box size=4.0 0.2 2.0; visual box size=4.0 0.2 2.0
- added link link_handle_2, mass 0.001; collision box size=0.2 0.2 0.05; visual box size=0.2 0.2 0.05
- added link link_handle_4, mass 0.001; collision box size=0.2 0.2 0.05; visual box size=0.2 0.2 0.05
- link link_1: geometry collision box size=0.8 1.0 3.6; visual box size=0.8 1.0 3.6
- link link_3: geometry collision box size=0.8 1.0 3.6; visual box size=0.8 1.0 3.6
- link link_door_0: geometry collision cylinder length=2.0 radius=0.2; visual cylinder length=2.0 radius=0.2
- link link_door_4: geometry collision cylinder length=2.0 radius=0.2; visual cylinder length=2.0 radius=0.2
Joints:
- added joint link_door_handle_1: type fixed, parent link_door_0, child link_door_handle_1, origin xyz=1.5 0 1.1 rpy=0 0 0
- added joint link_door_handle_5: type fixed, parent link_door_4, child link_door_handle_5, origin xyz=3.0 0 1.1 rpy=0 0 0
- added joint link_door_panel_1: type fixed, parent link_door_0, child link_door_panel_1, origin xyz=1.0 0 0 rpy=0 0 0
- added joint link_door_panel_5: type fixed, parent link_door_4, child link_door_panel_5, origin xyz=2.0 0 0 rpy=0 0 0
- added joint link_handle_2: type fixed, parent link_1, child link_handle_2, origin xyz=0 -0.6 0 rpy=0 0 0
- added joint link_handle_4: type fixed, parent link_3, child link_handle_4, origin xyz=0 -0.6 0 rpy=0 0 0

File: puzzles/my_custom/urdf/my_custom.urdf (robot description, URDF)
Before this commit: robot my_custom, 6 links, 5 joints
Links:
- added link link_door_handle1_5, mass 0.001; collision box size=0.05 0.2 0.2; visual box size=0.05 0.2 0.2
- added link link_door_handle2_5, mass 0.001; collision box size=0.05 0.2 0.2; visual box size=0.05 0.2 0.2
- added link link_door_handle_4, mass 0.001; collision box size=0.2 0.05 0.2; visual box size=0.2 0.05 0.2
- added link link_door_panel_4, mass 0.001; collision box size=2.0 0.2 4.0; visual box size=2.0 0.2 4.0
- added link link_door_panel_5, mass 0.001; collision box size=2.0 0.2 4.0; visual box size=2.0 0.2 4.0
- link link_0: geometry collision cylinder length=2.0 radius=0.5; visual cylinder length=2.0 radius=0.5
- link link_door_3: geometry collision cylinder length=4.0 radius=0.2; visual cylinder length=4.0 radius=0.2
- link link_door_4: geometry collision cylinder length=4.0 radius=0.2; visual cylinder length=4.0 radius=0.2
Joints:
- added joint link_door_handle1_5: type fixed, parent link_door_4, child link_door_handle1_5, origin xyz=1.5 0.2 0 rpy=0 0 0
- added joint link_door_handle2_5: type fixed, parent link_door_4, child link_door_handle2_5, origin xyz=1.5 -0.2 0 rpy=0 0 0
- added joint link_door_handle_4: type fixed, parent link_door_3, child link_door_handle_4, origin xyz=1.5 0 2.1 rpy=0 0 0
- added joint link_door_panel_4: type fixed, parent link_door_3, child link_door_panel_4, origin xyz=1.0 0 0 rpy=0 0 0
- added joint link_door_panel_5: type fixed, parent link_door_4, child link_door_panel_5, origin xyz=1.0 0 0 rpy=0 0 0

Commit message: fix: scaling of meshes in create_visual() remove bpy.ops.object.transform_apply(location=False, rotation=False, scale=True)

File: puzzles/lockbox2017/urdf/lockbox2017.urdf (robot description, URDF)
Before this commit: robot lockbox2017, 23 links, 22 joints
Links:
- link link_2_joint_0: geometry collision mesh filename=file:///home/userone/ba/puzzle-generator/puzzles/lockbox201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 scale=1.0 1.0 1.0; visual mesh filename=file:///home/userone/ba/puzzle-generator/puzzles/lockbox201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 scale=4.0 4.0 1.0

File: puzzles/lockbox_random/urdf/lockbox_random.urdf (robot description, URDF)
Before this commit: robot lockbox_random, 21 links, 20 joints
Links:
- link link_1_joint_0: geometry collision mesh filename=file:///home/userone/ba/puzzle-generator/puzzles/lockbox_ra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 scale=1.0 1.0 1.0; visual mesh filename=file:///home/userone/ba/puzzle-generator/puzzles/lockbox_ra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 scale=3.0 3.0 1.0
- link link_3_joint_0: geometry collision mesh filename=file:///home/userone/ba/puzzle-generator/puzzles/lockbox_ra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 scale=1.0 1.0 1.0; visual mesh filename=file:///home/userone/ba/puzzle-generator/puzzles/lockbox_ra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 scale=3.0 3.0 1.0

Commit message: fix: collision mesh offset fix: create_collision() when visual_obj is None error feat: create_collision() returns collision object if visual_obj is not None

File: puzzles/lockbox2017/urdf/lockbox2017.urdf (robot description, URDF)
Before this commit: robot lockbox2017, 23 links, 22 joints
Links:
- link link_2_joint_0: geometry collision mesh filename=file:///home/userone/ba/puzzle-generator/puzzles/lockbox201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 scale=1.0 1.0 1.0; visual mesh filename=file:///home/userone/ba/puzzle-generator/puzzles/lockbox201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 scale=1.0 1.0 1.0

File: puzzles/lockbox_random/urdf/lockbox_random.urdf (robot description, URDF)
Before this commit: robot lockbox_random, 21 links, 20 joints
Links:
- link link_1_joint_0: geometry collision mesh filename=file:///home/userone/ba/puzzle-generator/puzzles/lockbox_ra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 scale=1.0 1.0 1.0; visual mesh filename=file:///home/userone/ba/puzzle-generator/puzzles/lockbox_ra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 scale=1.0 1.0 1.0
- link link_3_joint_0: geometry collision mesh filename=file:///home/userone/ba/puzzle-generator/puzzles/lockbox_ra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 scale=1.0 1.0 1.0; visual mesh filename=file:///home/userone/ba/puzzle-generator/puzzles/lockbox_ra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 scale=1.0 1.0 1.0

File: puzzles/my_custom/urdf/my_custom.urdf (robot description, URDF)
Before this commit: robot my_custom, 13 links, 12 joints
Links:
- link link_0_joint_2: geometry collision mesh filename=file:///home/userone/ba/puzzle-generator/puzzles/my_custom/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 scale=1.0 1.0 1.0; visual mesh filename=file:///home/userone/ba/puzzle-generator/puzzles/my_custom/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 scale=1.0 1.0 1.0
- link link_1_joint_0: geometry collision mesh filename=file:///home/userone/ba/puzzle-generator/puzzles/my_custom/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 scale=1.0 1.0 1.0; visual mesh filename=file:///home/userone/ba/puzzle-generator/puzzles/my_custom/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 scale=1.0 1.0 1.0
- link link_2_joint_0: geometry collision mesh filename=file:///home/userone/ba/puzzle-generator/puzzles/my_custom/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 scale=1.0 1.0 1.0; visual mesh filename=file:///home/userone/ba/puzzle-generator/puzzles/my_custom/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 scale=1.0 1.0 1.0

Commit message: chore (minor): smaller sliders in lockbox2017

File: puzzles/lockbox2017/urdf/lockbox2017.urdf (robot description, URDF)
Before this commit: robot lockbox2017, 23 links, 22 joints
Links:
- link link_1_joint_0: geometry collision box size=2.999 0.499 0.999; visual box size=2.999 0.499 0.999
- link link_3_joint_0: geometry collision box size=2.999 0.499 0.999; visual box size=2.999 0.499 0.999
