Commit message: refactor (minor): shuffle() instead of random() < 0.5 in GridWorldSampler

File: puzzles/grid_world/urdf/grid_world.urdf (robot description, URDF)
Before this commit: robot grid_world, 19 links, 18 joints
Links:
- removed link link_10_fixed_handle_knob
- removed link link_5_fixed_hinge
- removed link link_6_fixed_handle_shaft
- removed link link_7_fixed_handle_knob
- removed link link_9_fixed_handle_shaft
- added link link_11_fixed_hinge, mass 0.001; visual cylinder length=0.989 radius=0.112
- added link link_5_fixed_handle_shaft, mass 0.001; collision box size=0.199 0.199 0.999; visual box size=0.199 0.199 0.999
- added link link_6_fixed_handle_knob, mass 0.001; collision box size=0.049 0.049 0.199; visual box size=0.049 0.049 0.199
- added link link_8_fixed_handle_shaft, mass 0.001; collision box size=0.199 0.199 0.999; visual box size=0.199 0.199 0.999
- added link link_9_fixed_handle_knob, mass 0.001; collision box size=0.049 0.049 0.199; visual box size=0.049 0.049 0.199
- link link_12_fixed_handle_shaft: geometry collision cylinder length=0.999 radius=0.0995; visual cylinder length=0.999 radius=0.0995
- link link_1_joint_0: geometry collision box size=1.899 0.899 0.899; visual box size=1.899 0.899 0.899
- link link_3_joint_0: geometry collision box size=2.899 0.899 0.899; visual box size=2.899 0.899 0.899
Joints:
- removed joint link_10_fixed_handle_knob
- removed joint link_5_fixed_hinge
- removed joint link_6_fixed_handle_shaft
- removed joint link_7_fixed_handle_knob
- removed joint link_9_fixed_handle_shaft
- added joint link_11_fixed_hinge: type fixed, parent link_3_joint_0, child link_11_fixed_hinge, origin xyz=0 0 0 rpy=0 0 0
- added joint link_5_fixed_handle_shaft: type fixed, parent link_1_joint_0, child link_5_fixed_handle_shaft, origin xyz=0 0 0.95 rpy=0 0 0
- added joint link_6_fixed_handle_knob: type fixed, parent link_5_fixed_handle_shaft, child link_6_fixed_handle_knob, origin xyz=0 0 0.6 rpy=0 0 0
- added joint link_8_fixed_handle_shaft: type fixed, parent link_2_joint_0, child link_8_fixed_handle_shaft, origin xyz=0 0 0.95 rpy=0 0 0
- added joint link_9_fixed_handle_knob: type fixed, parent link_8_fixed_handle_shaft, child link_9_fixed_handle_knob, origin xyz=0 0 0.6 rpy=0 0 0
- joint link_12_fixed_handle_shaft: origin xyz=0 0 0.95 rpy=0 0 0 -> xyz=1.0875 0 0.95 rpy=0 0 0
- joint link_1_joint_0: axis 0 0 1.0 -> 1.0 0 0; limit lower=-1.5708 upper=0 effort=0 velocity=0 -> lower=0 upper=1.0 effort=0 velocity=0; origin xyz=-2.5 -0.5 0.55 rpy=0 0 0 -> xyz=1.0 1.5 0.55 rpy=0 0 0; type revolute -> prismatic
- joint link_2_joint_0: origin xyz=1.0 1.5 0.55 rpy=0 0 0 -> xyz=-2.0 -0.5 0.55 rpy=0 0 3.14159
- joint link_3_joint_0: axis 1.0 0 0 -> 0 0 1.0; limit lower=0 upper=1.0 effort=0 velocity=0 -> lower=-1.5708 upper=0 effort=0 velocity=0; origin xyz=-1.5 -2.0 0.55 rpy=0 0 -1.5708 -> xyz=2.5 0.5 0.55 rpy=0 0 1.5708; type prismatic -> revolute

Commit message: feat (minor): branching_per_revolute_joint in GridWorldSampler

File: puzzles/grid_world/urdf/grid_world.urdf (robot description, URDF)
Before this commit: robot grid_world, 19 links, 18 joints
Links:
- removed link link_11_fixed_hinge
- removed link link_8_fixed_handle_shaft
- removed link link_9_fixed_handle_knob
- added link link_10_fixed_handle_knob, mass 0.001; collision box size=0.049 0.049 0.199; visual box size=0.049 0.049 0.199
- added link link_15_fixed_handle_shaft, mass 0.001; collision box size=0.199 0.199 0.999; visual box size=0.199 0.199 0.999
- added link link_16_fixed_handle_knob, mass 0.001; collision box size=0.049 0.049 0.199; visual box size=0.049 0.049 0.199
- added link link_18_fixed_handle_shaft, mass 0.001; collision box size=0.199 0.199 0.999; visual box size=0.199 0.199 0.999
- added link link_19_fixed_handle_knob, mass 0.001; collision box size=0.049 0.049 0.199; visual box size=0.049 0.049 0.199
- added link link_4_joint_0, mass 0.001; collision box size=1.899 0.899 0.899; visual box size=1.899 0.899 0.899
- added link link_5_joint_0, mass 0.001; collision box size=1.899 0.899 0.899; visual box size=1.899 0.899 0.899
- added link link_8_fixed_hinge, mass 0.001; visual cylinder length=0.989 radius=0.112
- added link link_9_fixed_handle_shaft, mass 0.001; collision cylinder length=0.999 radius=0.0995; visual cylinder length=0.999 radius=0.0995
- link link_12_fixed_handle_shaft: geometry collision box size=0.199 0.199 0.999; visual box size=0.199 0.199 0.999
- link link_2_joint_0: geometry collision box size=2.899 0.899 0.899; visual box size=2.899 0.899 0.899
- link link_3_joint_0: geometry collision box size=1.899 0.899 0.899; visual box size=1.899 0.899 0.899
Joints:
- removed joint link_11_fixed_hinge
- removed joint link_8_fixed_handle_shaft
- removed joint link_9_fixed_handle_knob
- added joint link_10_fixed_handle_knob: type fixed, parent link_9_fixed_handle_shaft, child link_10_fixed_handle_knob, origin xyz=0 0 0.6 rpy=0 0 0
- added joint link_15_fixed_handle_shaft: type fixed, parent link_4_joint_0, child link_15_fixed_handle_shaft, origin xyz=0 0 0.95 rpy=0 0 0
- added joint link_16_fixed_handle_knob: type fixed, parent link_15_fixed_handle_shaft, child link_16_fixed_handle_knob, origin xyz=0 0 0.6 rpy=0 0 0
- added joint link_18_fixed_handle_shaft: type fixed, parent link_5_joint_0, child link_18_fixed_handle_shaft, origin xyz=0 0 0.95 rpy=0 0 0
- added joint link_19_fixed_handle_knob: type fixed, parent link_18_fixed_handle_shaft, child link_19_fixed_handle_knob, origin xyz=0 0 0.6 rpy=0 0 0
- added joint link_4_joint_0: type prismatic, parent base_link, child link_4_joint_0, origin xyz=0 -0.5 0.55 rpy=0 0 0, axis 1.0 0 0, limit lower=0 upper=1.0 effort=0 velocity=0
- added joint link_5_joint_0: type prismatic, parent base_link, child link_5_joint_0, origin xyz=-2.5 2.0 0.55 rpy=0 0 1.5708, axis 1.0 0 0, limit lower=0 upper=1.0 effort=0 velocity=0
- added joint link_8_fixed_hinge: type fixed, parent link_2_joint_0, child link_8_fixed_hinge, origin xyz=0 0 0 rpy=0 0 0
- added joint link_9_fixed_handle_shaft: type fixed, parent link_2_joint_0, child link_9_fixed_handle_shaft, origin xyz=1.0875 0 0.95 rpy=0 0 0
- joint link_12_fixed_handle_shaft: origin xyz=1.0875 0 0.95 rpy=0 0 0 -> xyz=0 0 0.95 rpy=0 0 0
- joint link_1_joint_0: origin xyz=1.0 1.5 0.55 rpy=0 0 0 -> xyz=-1.0 1.5 0.55 rpy=0 0 3.14159
- joint link_2_joint_0: axis 1.0 0 0 -> 0 0 1.0; limit lower=0 upper=1.0 effort=0 velocity=0 -> lower=-1.5708 upper=0 effort=0 velocity=0; origin xyz=-2.0 -0.5 0.55 rpy=0 0 3.14159 -> xyz=-2.5 -0.5 0.55 rpy=0 0 0; type prismatic -> revolute
- joint link_3_joint_0: axis 0 0 1.0 -> 1.0 0 0; limit lower=-1.5708 upper=0 effort=0 velocity=0 -> lower=0 upper=1.0 effort=0 velocity=0; origin xyz=2.5 0.5 0.55 rpy=0 0 1.5708 -> xyz=1.0 1.5 0.55 rpy=0 0 0; type revolute -> prismatic

File: puzzles/simple_sliders/urdf/simple_sliders.urdf (robot description, URDF)
Before this commit: robot simple_sliders, 6 links, 5 joints
Links:
- added link link_10_fixed_handle_shaft, mass 0.001; collision box size=0.199 0.199 0.999; visual box size=0.199 0.199 0.999
- added link link_11_fixed_handle_knob, mass 0.001; collision box size=0.049 0.049 0.199; visual box size=0.049 0.049 0.199
- added link link_1_fixed_handle_shaft, mass 0.001; collision box size=0.199 0.199 0.999; visual box size=0.199 0.199 0.999
- added link link_1_fixed_handle_shaft.001, mass 0.001; visual box size=0.199 0.199 0.999
- added link link_2_fixed_handle_knob, mass 0.001; collision box size=0.049 0.049 0.199; visual box size=0.049 0.049 0.199
- added link link_2_fixed_handle_knob.001, mass 0.001; visual box size=0.049 0.049 0.199
- added link link_4_fixed_handle_shaft, mass 0.001; collision box size=0.199 0.199 0.999; visual box size=0.199 0.199 0.999
- added link link_5_fixed_handle_knob, mass 0.001; collision box size=0.049 0.049 0.199; visual box size=0.049 0.049 0.199
- added link link_7_fixed_handle_shaft, mass 0.001; collision box size=0.199 0.199 0.999; visual box size=0.199 0.199 0.999
- added link link_8_fixed_handle_knob, mass 0.001; collision box size=0.049 0.049 0.199; visual box size=0.049 0.049 0.199
Joints:
- added joint link_10_fixed_handle_shaft: type fixed, parent link_3_joint_0, child link_10_fixed_handle_shaft, origin xyz=0 0 0.6 rpy=0 0 0
- added joint link_11_fixed_handle_knob: type fixed, parent link_10_fixed_handle_shaft, child link_11_fixed_handle_knob, origin xyz=0 0 0.6 rpy=0 0 0
- added joint link_1_fixed_handle_shaft: type fixed, parent link_0_joint_0, child link_1_fixed_handle_shaft, origin xyz=0 0 0.6 rpy=0 0 0
- added joint link_1_fixed_handle_shaft.001: type fixed, parent goal, child link_1_fixed_handle_shaft.001, origin xyz=0 0 0.6 rpy=0 0 0
- added joint link_2_fixed_handle_knob: type fixed, parent link_1_fixed_handle_shaft, child link_2_fixed_handle_knob, origin xyz=0 0 0.6 rpy=0 0 0
- added joint link_2_fixed_handle_knob.001: type fixed, parent link_1_fixed_handle_shaft.001, child link_2_fixed_handle_knob.001, origin xyz=0 0 0.6 rpy=0 0 0
- added joint link_4_fixed_handle_shaft: type fixed, parent link_1_joint_0, child link_4_fixed_handle_shaft, origin xyz=0 0 0.6 rpy=0 0 0
- added joint link_5_fixed_handle_knob: type fixed, parent link_4_fixed_handle_shaft, child link_5_fixed_handle_knob, origin xyz=0 0 0.6 rpy=0 0 0
- added joint link_7_fixed_handle_shaft: type fixed, parent link_2_joint_0, child link_7_fixed_handle_shaft, origin xyz=0 0 0.6 rpy=0 0 0
- added joint link_8_fixed_handle_knob: type fixed, parent link_7_fixed_handle_shaft, child link_8_fixed_handle_knob, origin xyz=0 0 0.6 rpy=0 0 0
