Commit message: chore: replace epsilon with slider_length, slider_width in lockbox_random

File: puzzles/lockbox_random/urdf/lockbox_random.urdf (robot description, URDF)
Before this commit: robot lockbox_random, 21 links, 20 joints
Links:
- link goal: geometry visual box size=0.999 0.199 1.399
- link link_0_joint_0: geometry collision box size=0.999 0.199 1.399; visual box size=0.999 0.199 1.399
- link link_2_joint_0: geometry collision box size=0.999 0.199 1.399; visual box size=0.999 0.199 1.399
- link link_4_joint_0: geometry collision box size=0.999 0.199 1.399; visual box size=0.999 0.199 1.399

Commit message: refactor: LockboxRandomSampler * add radius_interval * add get_rotation dict * make first slider direction random

File: puzzles/lockbox_random/urdf/lockbox_random.urdf (robot description, URDF)
Before this commit: robot lockbox_random, 22 links, 21 joints
Links:
- link link_fixed_12_hinge: geometry visual cylinder length=1.099 radius=0.11261
- link link_fixed_5_hinge: geometry visual cylinder length=1.099 radius=0.09437
Joints:
- joint goal: origin xyz=-1.0 0.5 0.5 rpy=0 0 0 -> xyz=-1.0 0 0.5 rpy=0 0 3.14159
- joint link_0_joint_0: origin xyz=-2.0 0.5 0.5 rpy=0 0 0 -> xyz=0 0 0.5 rpy=0 0 3.14159
- joint link_1_joint_0: origin xyz=0.5 0.5 0.5 rpy=0 0 1.5708 -> xyz=-2.51783 0 0.5 rpy=0 0 3.14159
- joint link_2_joint_0: origin xyz=0.5 2.0 0.5 rpy=0 0 1.5708 -> xyz=-4.03566 0 0.5 rpy=0 0 3.14159
- joint link_3_joint_0: origin xyz=0.5 4.5 0.5 rpy=0 0 3.14159 -> xyz=-6.84553 0 0.5 rpy=0 0 3.14159
- joint link_4_joint_0: origin xyz=-1.0 4.5 0.5 rpy=0 0 3.14159 -> xyz=-8.6554 0 0.5 rpy=0 0 3.14159
- joint link_fixed_13_handle_shaft: origin xyz=0 1.125 1.0 rpy=0 0 0 -> xyz=0 1.3574 1.0 rpy=0 0 0
- joint link_fixed_6_handle_shaft: origin xyz=0 1.125 1.0 rpy=0 0 0 -> xyz=0 1.13838 1.0 rpy=0 0 0
