Commit message: feat: add move_twice puzzle

File: puzzles/move_twice/urdf/move_twice.urdf (robot description, URDF)
Before this commit: robot my_custom, 13 links, 12 joints
Links:
- removed link link_1_fixed_joint_1_handle_shaft
- removed link link_1_fixed_joint_2_handle_knob
- removed link link_1_fixed_joint_3_hinge
- removed link link_2_fixed_joint_1_handle_shaft
- removed link link_2_fixed_joint_2_handle_knob
- removed link link_2_fixed_joint_3_hinge
- removed link link_2_joint_0
- added link goal, mass 0.001
- added link link_0_fixed_joint_3_hinge.001, mass 0.001; visual cylinder length=1.1 radius=0.05
- added link link_0_joint_1.001, mass 0.001
- added link link_0_joint_2.001, mass 0.001; visual mesh filename=file:///home/userone/ba/puzzle-generator/puzzles/move_twice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 scale=1.0 1.0 1.0
- added link link_1_fixed_joint_0_wall_back, mass 0.001; collision box size=0.2 6.0 1.0; visual box size=0.2 6.0 1.0
- added link link_1_fixed_joint_0_wall_left, mass 0.001; collision box size=4.0 0.2 1.0; visual box size=4.0 0.2 1.0
- added link link_1_fixed_joint_0_wall_mid, mass 0.001; collision box size=4.0 0.2 1.0; visual box size=4.0 0.2 1.0
- added link link_1_fixed_joint_0_wall_right, mass 0.001; collision box size=4.0 0.2 1.0; visual box size=4.0 0.2 1.0
- link link_0_joint_2: geometry collision mesh filename=file:///home/userone/ba/puzzle-generator/puzzles/move_twice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 scale=1.0 1.0 1.0; visual mesh filename=file:///home/userone/ba/puzzle-generator/puzzles/move_twice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 scale=1.0 1.0 1.0
- link link_1_joint_0: geometry collision box size=0.2 6.0 1.0; visual box size=0.2 6.0 1.0
Joints:
- removed joint link_1_fixed_joint_1_handle_shaft
- removed joint link_1_fixed_joint_2_handle_knob
- removed joint link_1_fixed_joint_3_hinge
- removed joint link_2_fixed_joint_1_handle_shaft
- removed joint link_2_fixed_joint_2_handle_knob
- removed joint link_2_fixed_joint_3_hinge
- removed joint link_2_joint_0
- added joint goal: type fixed, parent base_link, child goal, origin xyz=0 3.0 0.6 rpy=0 0 1.5708, limit effort=0 velocity=0
- added joint link_0_fixed_joint_3_hinge.001: type fixed, parent link_0_joint_2.001, child link_0_fixed_joint_3_hinge.001, origin xyz=0 0 0 rpy=0 0 0
- added joint link_0_joint_1.001: type fixed, parent goal, child link_0_joint_1.001, origin xyz=0 0 0 rpy=0 0 0, limit effort=0 velocity=0
- added joint link_0_joint_2.001: type fixed, parent link_0_joint_1.001, child link_0_joint_2.001, origin xyz=0 0 0 rpy=0 0 0, limit effort=0 velocity=0
- added joint link_1_fixed_joint_0_wall_back: type fixed, parent base_link, child link_1_fixed_joint_0_wall_back, origin xyz=-2.1 1.5 0.6 rpy=0 0 0
- added joint link_1_fixed_joint_0_wall_left: type fixed, parent base_link, child link_1_fixed_joint_0_wall_left, origin xyz=0 -1.4 0.6 rpy=0 0 0
- added joint link_1_fixed_joint_0_wall_mid: type fixed, parent base_link, child link_1_fixed_joint_0_wall_mid, origin xyz=0 1.5 0.6 rpy=0 0 0
- added joint link_1_fixed_joint_0_wall_right: type fixed, parent base_link, child link_1_fixed_joint_0_wall_right, origin xyz=0 4.4 0.6 rpy=0 0 0
- joint link_1_joint_0: axis 0 0 1.0 -> 0 1.0 0; limit lower=-0.7854 upper=0.7854 effort=0 velocity=0 -> lower=-2.0 upper=2.0 effort=0 velocity=0; origin xyz=0 -5.0 0.6 rpy=0 0 0 -> xyz=2.1 1.5 0.6 rpy=0 0 0; type revolute -> prismatic

Commit message: feat: random goal position in move_twice

File: puzzles/move_twice/urdf/move_twice.urdf (robot description, URDF)
Before this commit: robot move_twice, 14 links, 13 joints
Joints:
- joint goal: origin xyz=0 3.0 0.6 rpy=0 0 1.5708 -> xyz=1.03327 3.36114 0.6 rpy=0 0 -0.49906

Commit message: fix (minor): increase link_shrink

File: puzzles/move_twice/urdf/move_twice.urdf (robot description, URDF)
Before this commit: robot move_twice, 13 links, 12 joints
Links:
- link link_0_joint_0.001: geometry visual mesh filename=file:///home/userone/ba/puzzle-generator/puzzles/move_twice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 scale=0.995 0.995 0.995
- link link_1_joint_0: geometry collision box size=0.195 5.995 0.995; visual box size=0.195 5.995 0.995
- link link_fixed_0_floor: geometry collision box size=31.995 31.995 0.195; visual box size=31.995 31.995 0.195
- link link_fixed_4_wall_left: geometry collision box size=3.995 0.195 0.995; visual box size=3.995 0.195 0.995
- link link_fixed_5_wall_right: geometry collision box size=3.995 0.195 0.995; visual box size=3.995 0.195 0.995
- link link_fixed_6_wall_mid: geometry collision box size=3.995 0.195 0.995; visual box size=3.995 0.195 0.995
- link link_fixed_7_wall_back: geometry collision box size=0.195 5.995 0.995; visual box size=0.195 5.995 0.995
